File: KICAD/Drivers_Command.sch (KiCad schematic (older format))
At the start: 12 parts

Commit message: merge program breaker nicolas
Connections:
- net at U?.10 (S2), U?.11 (S1): now also U?.11
Other:
- note added: "Pull-downs MOS parallèles"
- note added: "Pull-ups MOS séries"
- note added: "Rework needed"
- moved on the sheet: R?
Changed lines of the file:
@@
 	1    0    0    -1
 $EndComp
-Text HLabel 8200 3450 2    50   Output ~ 0
+Text HLabel 8400 3250 2    50   Output ~ 0
 Driver_LS
 $Comp
 L power:GND #PWR?
 U 1 1 61156299
-P 8700 4650
-F 0 "#PWR?" H 8700 4400 50  0001 C CNN
-F 1 "GND" H 8705 4477 50  0000 C CNN
-F 2 "" H 8700 4650 50  0001 C CNN
-F 3 "" H 8700 4650 50  0001 C CNN
-	1    8700 4650
+P 8900 4650
+F 0 "#PWR?" H 8900 4400 50  0001 C CNN
+F 1 "GND" H 8905 4477 50  0000 C CNN
+F 2 "" H 8900 4650 50  0001 C CNN
+F 3 "" H 8900 4650 50  0001 C CNN
+	1    8900 4650
 	1    0    0    -1
 $EndComp
@@
 L Device:R R?
 U 1 1 61146E6D
-P 8050 4300
-F 0 "R?" H 8120 4346 50  0000 L CNN
-F 1 "R" H 8120 4255 50  0000 L CNN
-F 2 "" V 7980 4300 50  0001 C CNN
-F 3 "~" H 8050 4300 50  0001 C CNN
-	1    8050 4300
+P 8250 4450
+F 0 "R?" H 8320 4496 50  0000 L CNN
+F 1 "R" H 8320 4405 50  0000 L CNN
+F 2 "" V 8180 4450 50  0001 C CNN
+F 3 "~" H 8250 4450 50  0001 C CNN
+	1    8250 4450
 	1    0    0    -1
 $EndComp
@@
 L Device:R R?
 U 1 1 611408F1
-P 8700 4300
-F 0 "R?" H 8770 4346 50  0000 L CNN
-F 1 "R" H 8770 4255 50  0000 L CNN
-F 2 "" V 8630 4300 50  0001 C CNN
-F 3 "~" H 8700 4300 50  0001 C CNN
-	1    8700 4300
+P 8900 4450
+F 0 "R?" H 8970 4496 50  0000 L CNN
+F 1 "R" H 8970 4405 50  0000 L CNN
+F 2 "" V 8830 4450 50  0001 C CNN
+F 3 "~" H 8900 4450 50  0001 C CNN
+	1    8900 4450
 	1    0    0    -1
 $EndComp
@@
 L power:GND #PWR?
 U 1 1 610F5D5C
-P 8050 4650
-F 0 "#PWR?" H 8050 4400 50  0001 C CNN
-F 1 "GND" H 8055 4477 50  0000 C CNN
-F 2 "" H 8050 4650 50  0001 C CNN
-F 3 "" H 8050 4650 50  0001 C CNN
-	1    8050 4650
+P 8250 4650
+F 0 "#PWR?" H 8250 4400 50  0001 C CNN
+F 1 "GND" H 8255 4477 50  0000 C CNN
+F 2 "" H 8250 4650 50  0001 C CNN
+F 3 "" H 8250 4650 50  0001 C CNN
+	1    8250 4650
 	1    0    0    -1
 $EndComp
@@
 Wire Wire Line
 	6750 4350 6750 4400
-Text HLabel 8175 3850 2    50   Output ~ 0
+Text HLabel 8375 4050 2    50   Output ~ 0
 Driver_RP
-Text HLabel 8800 3550 2    50   Output ~ 0
+Text HLabel 9000 3350 2    50   Output ~ 0
 Driver_RS
-Text HLabel 8775 3750 2    50   Output ~ 0
+Text HLabel 8975 3950 2    50   Output ~ 0
 Driver_LP
 Text HLabel 5700 3450 0    50   Input ~ 0
@@
 L Device:R R?
 U 1 1 6114968D
-P 8050 3050
-F 0 "R?" H 8120 3096 50  0000 L CNN
-F 1 "R" H 8120 3005 50  0000 L CNN
-F 2 "" V 7980 3050 50  0001 C CNN
-F 3 "~" H 8050 3050 50  0001 C CNN
-	1    8050 3050
+P 8250 2850
+F 0 "R?" H 8320 2896 50  0000 L CNN
+F 1 "R" H 8320 2805 50  0000 L CNN
+F 2 "" V 8180 2850 50  0001 C CNN
+F 3 "~" H 8250 2850 50  0001 C CNN
+	1    8250 2850
 	1    0    0    -1
 $EndComp
@@
 L Device:R R?
 U 1 1 6114A712
-P 8700 3050
-F 0 "R?" H 8770 3096 50  0000 L CNN
-F 1 "R" H 8770 3005 50  0000 L CNN
-F 2 "" V 8630 3050 50  0001 C CNN
-F 3 "~" H 8700 3050 50  0001 C CNN
-	1    8700 3050
-	1    0    0    -1
-$EndComp
-Wire Wire Line
-	8050 3200 8050 3450
-Connection ~ 8050 3450
-Wire Wire Line
-	8700 3200 8700 3550
-Wire Wire Line
-	8050 3450 8200 3450
-Wire Wire Line
-	8700 3550 8800 3550
-Connection ~ 8700 3550
+P 8900 2850
+F 0 "R?" H 8970 2896 50  0000 L CNN
+F 1 "R" H 8970 2805 50  0000 L CNN
+F 2 "" V 8830 2850 50  0001 C CNN
+F 3 "~" H 8900 2850 50  0001 C CNN
+	1    8900 2850
+	1    0    0    -1
+$EndComp
+Wire Wire Line
+	8250 3000 8250 3250
+Connection ~ 8250 3250
+Wire Wire Line
+	8900 3000 8900 3350
+Wire Wire Line
+	8250 3250 8400 3250
+Wire Wire Line
+	8900 3350 9000 3350
 $Comp
 L power:VCC #PWR?
 U 1 1 611540C5
-P 8050 2850
-F 0 "#PWR?" H 8050 2700 50  0001 C CNN
-F 1 "VCC" H 8065 3023 50  0000 C CNN
-F 2 "" H 8050 2850 50  0001 C CNN
-F 3 "" H 8050 2850 50  0001 C CNN
-	1    8050 2850
+P 8250 2650
+F 0 "#PWR?" H 8250 2500 50  0001 C CNN
+F 1 "VCC" H 8265 2823 50  0000 C CNN
+F 2 "" H 8250 2650 50  0001 C CNN
+F 3 "" H 8250 2650 50  0001 C CNN
+	1    8250 2650
 	1    0    0    -1
 $EndComp
@@
 L power:VCC #PWR?
 U 1 1 61154F00
-P 8700 2850
-F 0 "#PWR?" H 8700 2700 50  0001 C CNN
-F 1 "VCC" H 8715 3023 50  0000 C CNN
-F 2 "" H 8700 2850 50  0001 C CNN
-F 3 "" H 8700 2850 50  0001 C CNN
-	1    8700 2850
-	1    0    0    -1
-$EndComp
-Wire Wire Line
-	8700 2850 8700 2900
-Wire Wire Line
-	8050 2850 8050 2900
+P 8900 2650
+F 0 "#PWR?" H 8900 2500 50  0001 C CNN
+F 1 "VCC" H 8915 2823 50  0000 C CNN
+F 2 "" H 8900 2650 50  0001 C CNN
+F 3 "" H 8900 2650 50  0001 C CNN
+	1    8900 2650
+	1    0    0    -1
+$EndComp
+Wire Wire Line
+	8900 2650 8900 2700
+Wire Wire Line
+	8250 2650 8250 2700
 Wire Wire Line
 	2600 3300 2600 3550
@@
 	4150 3300 4250 3300
 Wire Wire Line
-	7350 3550 8700 3550
-Wire Wire Line
-	7350 3450 8050 3450
-Wire Wire Line
-	7350 3850 8050 3850
-Wire Wire Line
-	8050 4450 8050 4650
-Wire Wire Line
-	8700 4450 8700 4650
-Wire Wire Line
-	7350 3750 8700 3750
-Wire Wire Line
-	8700 3750 8700 4150
-Connection ~ 8700 3750
-Wire Wire Line
-	8700 3750 8775 3750
-Wire Wire Line
-	8050 4150 8050 3850
-Connection ~ 8050 3850
-Wire Wire Line
-	8050 3850 8175 3850
+	8250 4600 8250 4650
+Wire Wire Line
+	8900 4600 8900 4650
+Wire Wire Line
+	8900 3950 8900 4300
+Connection ~ 8900 3950
+Wire Wire Line
+	8900 3950 8975 3950
+Wire Wire Line
+	8250 4300 8250 4050
+Connection ~ 8250 4050
+Wire Wire Line
+	8250 4050 8375 4050
 NoConn ~ 7350 4050
 NoConn ~ 7350 4150
@@
 Wire Wire Line
 	5700 3750 6350 3750
-Wire Wire Line
-	4950 3200 6300 3200
 Wire Notes Line
 	5800 2550 7650 2550
 Wire Notes Line
+	7650 5000 5800 5000
+Wire Notes Line
+	5800 2550 5800 5000
+Wire Notes Line
+	4950 2550 4950 3900
+Wire Notes Line
+	4950 3900 2350 3900
+Wire Notes Line
+	2350 3900 2350 2550
+Wire Notes Line
+	2350 2550 4950 2550
+Wire Wire Line
+	2250 3100 2600 3100
+Wire Wire Line
+	2250 3300 2600 3300
+Text Notes 4000 5750 0    394  ~ 79
+Rework needed
+Wire Wire Line
+	4850 3200 6300 3200
+Text HLabel 8975 3950 2    50   Output ~ 0
+Driver_LP
+Wire Wire Line
+	7350 3750 7850 3750
+Wire Wire Line
+	7850 3950 8900 3950
+Wire Notes Line
 	7650 2550 7650 5000
-Wire Notes Line
-	7650 5000 5800 5000
-Wire Notes Line
-	5800 2550 5800 5000
-Wire Notes Line
-	4950 2550 4950 3900
-Wire Notes Line
-	4950 3900 2350 3900
-Wire Notes Line
-	2350 3900 2350 2550
-Wire Notes Line
-	2350 2550 4950 2550
-Wire Wire Line
-	2250 3100 2600 3100
-Wire Wire Line
-	2250 3300 2600 3300
-Wire Notes Line
-	7800 3650 9300 3650
-Wire Notes Line
-	9300 2550 7800 2550
-Wire Notes Line
-	7800 5000 9300 5000
-Wire Notes Line
-	7800 2550 7800 5000
-Wire Notes Line
-	9300 2550 9300 5000
+Wire Wire Line
+	7350 3850 7750 3850
+Wire Wire Line
+	7750 4050 8250 4050
+Wire Wire Line
+	7750 3850 7750 4050
+Wire Wire Line
+	7850 3750 7850 3950
+Wire Wire Line
+	7750 3250 8250 3250
+Wire Wire Line
+	8900 3350 7850 3350
+Wire Wire Line
+	7850 3350 7850 3550
+Connection ~ 8900 3350
+Wire Wire Line
+	7350 3450 7750 3450
+Wire Wire Line
+	7750 3450 7750 3250
+Wire Wire Line
+	7350 3550 7850 3550
+Wire Notes Line
+	9500 3550 8050 3550
+Wire Notes Line
+	8050 3750 9500 3750
+Text Notes 8650 2350 0    50   ~ 0
+Pull-ups MOS séries
+Wire Notes Line
+	9500 2200 8050 2200
+Wire Notes Line
+	8050 2200 8050 3550
+Wire Notes Line
+	9500 2200 9500 3550
+Wire Notes Line
+	8050 5100 9500 5100
+Wire Notes Line
+	9500 3750 9500 5100
+Wire Notes Line
+	8050 3750 8050 5100
+Text Notes 8400 5050 0    50   ~ 0
+Pull-downs MOS parallèles
 $EndSCHEMATC

Commit message: minors edits + 7v rail
Parts:
- removed R?: R, symbol Device:R
Connections:
- net GND: now also U?.4 (C), U?.9 (S3)
- net VCC renamed +7V
Other:
- moved on the sheet: U?A, U?B, U?C, U?D

Commit message: a ton of new stuff. V0.8
Parts:
- added C?: 100n, symbol Device:C
Connections:
- net +7V: no longer C?.1, U?.14 (VDD)
- net GND: now also C?.2
- new net VCC: C?.1, C?.1, U?.14 (VDD)
Other:
- note added: "SWITCH POWER MOS ICI"
- note removed: "Rework needed"
Changed lines of the file:
@@
 $Descr A4 11693 8268
 encoding utf-8
-Sheet 13 15
+Sheet 13 16
 Title "SESAME"
 Date "2021-08-04"
@@
 $EndComp
 $Comp
-L power:GND #PWR?
+L power:GND #PWR0166
 U 1 1 610E393A
 P 1300 7500
-F 0 "#PWR?" H 1300 7250 50  0001 C CNN
+F 0 "#PWR0166" H 1300 7250 50  0001 C CNN
 F 1 "GND" H 1305 7327 50  0000 C CNN
 F 2 "" H 1300 7500 50  0001 C CNN
@@
 Driver_LS
 $Comp
-L power:GND #PWR?
+L power:GND #PWR0167
 U 1 1 61156299
 P 8900 4650
-F 0 "#PWR?" H 8900 4400 50  0001 C CNN
+F 0 "#PWR0167" H 8900 4400 50  0001 C CNN
 F 1 "GND" H 8905 4477 50  0000 C CNN
 F 2 "" H 8900 4650 50  0001 C CNN
@@
 $EndComp
 $Comp
-L power:GND #PWR?
+L power:GND #PWR0168
 U 1 1 610F5D5C
 P 8250 4650
-F 0 "#PWR?" H 8250 4400 50  0001 C CNN
+F 0 "#PWR0168" H 8250 4400 50  0001 C CNN
 F 1 "GND" H 8255 4477 50  0000 C CNN
 F 2 "" H 8250 4650 50  0001 C CNN
@@
 	6800 4450 6800 4400
 $Comp
-L power:GND #PWR?
+L power:GND #PWR0169
 U 1 1 610EA813
 P 6800 4450
-F 0 "#PWR?" H 6800 4200 50  0001 C CNN
+F 0 "#PWR0169" H 6800 4200 50  0001 C CNN
 F 1 "GND" H 6805 4277 50  0000 C CNN
 F 2 "" H 6800 4450 50  0001 C CNN
@@
 	6250 4150 6350 4150
 $Comp
-L power:GND #PWR?
+L power:GND #PWR0170
 U 1 1 61122542
 P 6250 4450
-F 0 "#PWR?" H 6250 4200 50  0001 C CNN
+F 0 "#PWR0170" H 6250 4200 50  0001 C CNN
 F 1 "GND" H 6255 4277 50  0000 C CNN
 F 2 "" H 6250 4450 50  0001 C CNN
@@
 Wire Wire Line
 	2250 3250 2600 3250
-Text Notes 3050 4250 0    100  ~ 20
-Rework needed
 Wire Wire Line
 	4850 3150 6300 3150
@@
 	6300 3150 6300 3250
 $Comp
-L power:GND #PWR?
+L power:GND #PWR0171
 U 1 1 612292EA
 P 6100 3350
-F 0 "#PWR?" H 6100 3100 50  0001 C CNN
+F 0 "#PWR0171" H 6100 3100 50  0001 C CNN
 F 1 "GND" H 6105 3177 50  0000 C CNN
 F 2 "" H 6100 3350 50  0001 C CNN
@@
 Connection ~ 6250 4150
 $Comp
-L Sesame:+7V #PWR?
-U 1 1 612704FB
-P 1300 6500
-F 0 "#PWR?" H 1300 6350 50  0001 C CNN
-F 1 "+7V" H 1315 6673 50  0000 C CNN
-F 2 "" H 1300 6500 50  0001 C CNN
-F 3 "" H 1300 6500 50  0001 C CNN
-	1    1300 6500
-	1    0    0    -1
-$EndComp
-Connection ~ 1300 6500
-$Comp
-L Sesame:+7V #PWR?
+L Sesame:+7V #PWR0172
 U 1 1 61274E3B
 P 6950 2900
-F 0 "#PWR?" H 6950 2750 50  0001 C CNN
+F 0 "#PWR0172" H 6950 2750 50  0001 C CNN
 F 1 "+7V" H 6965 3073 50  0000 C CNN
 F 2 "" H 6950 2900 50  0001 C CNN
@@
 $EndComp
 $Comp
-L Sesame:+7V #PWR?
+L Sesame:+7V #PWR0173
 U 1 1 61278908
 P 8250 2650
-F 0 "#PWR?" H 8250 2500 50  0001 C CNN
+F 0 "#PWR0173" H 8250 2500 50  0001 C CNN
 F 1 "+7V" H 8265 2823 50  0000 C CNN
 F 2 "" H 8250 2650 50  0001 C CNN
@@
 $EndComp
 $Comp
-L Sesame:+7V #PWR?
+L Sesame:+7V #PWR0174
 U 1 1 6127D6D0
 P 8900 2650
-F 0 "#PWR?" H 8900 2500 50  0001 C CNN
+F 0 "#PWR0174" H 8900 2500 50  0001 C CNN
 F 1 "+7V" H 8915 2823 50  0000 C CNN
 F 2 "" H 8900 2650 50  0001 C CNN
@@
 	1    0    0    -1
 $EndComp
+$Comp
+L power:VCC #PWR0175
+U 1 1 615841AD
+P 1300 6500
+F 0 "#PWR0175" H 1300 6350 50  0001 C CNN
+F 1 "VCC" H 1315 6673 50  0000 C CNN
+F 2 "" H 1300 6500 50  0001 C CNN
+F 3 "" H 1300 6500 50  0001 C CNN
+	1    1300 6500
+	1    0    0    -1
+$EndComp
+Connection ~ 1300 6500
+$Comp
+L power:GND #PWR?
+U 1 1 61587C63
+P 2200 7050
+AR Path="/60F421D1/61587C63" Ref="#PWR?"  Part="1"
+AR Path="/60F4EAD9/61587C63" Ref="#PWR0176"  Part="1"
+F 0 "#PWR0176" H 2200 6800 50  0001 C CNN
+F 1 "GND" H 2205 6877 50  0000 C CNN
+F 2 "" H 2200 7050 50  0001 C CNN
+F 3 "" H 2200 7050 50  0001 C CNN
+	1    2200 7050
+	1    0    0    -1
+$EndComp
+$Comp
+L Device:C C?
+U 1 1 61587C69
+P 2200 6900
+AR Path="/60F421D1/61587C69" Ref="C?"  Part="1"
+AR Path="/60F4EAD9/61587C69" Ref="C?"  Part="1"
+F 0 "C?" H 2315 6946 50  0000 L CNN
+F 1 "100n" H 2315 6855 50  0000 L CNN
+F 2 "" H 2238 6750 50  0001 C CNN
+F 3 "~" H 2200 6900 50  0001 C CNN
+	1    2200 6900
+	1    0    0    -1
+$EndComp
+$Comp
+L power:VCC #PWR?
+U 1 1 61587C6F
+P 2200 6750
+AR Path="/60F421D1/61587C6F" Ref="#PWR?"  Part="1"
+AR Path="/60F4EAD9/61587C6F" Ref="#PWR0177"  Part="1"
+F 0 "#PWR0177" H 2200 6600 50  0001 C CNN
+F 1 "VCC" H 2215 6923 50  0000 C CNN
+F 2 "" H 2200 6750 50  0001 C CNN
+F 3 "" H 2200 6750 50  0001 C CNN
+	1    2200 6750
+	1    0    0    -1
+$EndComp
+Text Notes 3100 4400 0    100  ~ 0
+SWITCH POWER MOS ICI
 $EndSCHEMATC
