File: KICAD/Drivers_Command.sch (KiCad schematic (older format))
At the start: 24 parts, among them U4 CD4053BM96, U5 CD4053BM96, U6 4011

Commit message: review w/ jmt
Parts:
- removed C?: 100n, symbol Device:C
- removed R?: 1k, Resistor_SMD:R_0805_2012Metric_Pad1.15x1.40mm_HandSolder, symbol Device:R
- C13, C15, C16: renamed from C?; footprint Capacitor_SMD:C_0805_2012Metric_Pad1.15x1.40mm_HandSolder -> (none)
- R29, R30, R31, R32, R33, R34, R35, R36: renamed from R?; footprint Resistor_SMD:R_0805_2012Metric_Pad1.15x1.40mm_HandSolder -> (none)
- U5: renamed from U4; footprint Package_SO:SO-16_3.9x9.9mm_P1.27mm -> (none)
- U6: renamed from U5; footprint Package_SO:SO-16_3.9x9.9mm_P1.27mm -> (none)
- gave numbers to parts that had none: 8
- renumbered U6 to U4
Connections:
- net ~Enable_Softstart is gone; now on net ~Enable: U5.11 (S1), U6.6 (INH)
Other:
- note removed: "au plus vite (juste apres le triangle)\nenv 0.1ms"

Commit message: edit footprints by jmt
Parts:
- C13, C15, C16: footprint (none) -> Capacitor_SMD:C_0805_2012Metric_Pad1.15x1.40mm_HandSolder
- R29, R30, R31, R32, R33, R34, R35, R36: footprint (none) -> Resistor_SMD:R_0805_2012Metric_Pad1.15x1.40mm_HandSolder
- TP10, TP11: footprint (none) -> TestPoint:TestPoint_THTPad_D2.0mm_Drill1.0mm
- TP12, TP13, TP14, TP15, TP16, TP17: footprint (none) -> TestPoint:TestPoint_Loop_D1.80mm_Drill1.0mm_Beaded
- U4: footprint (none) -> Package_SO:SOIC-14_3.9x8.7mm_P1.27mm
- U5, U6: footprint (none) -> Package_SO:SOIC-16_4.55x10.3mm_P1.27mm
Changed lines of the file:
@@
 F 0 "U4" H 1530 7046 50  0000 L CNN
 F 1 "4011" H 1530 6955 50  0000 L CNN
-F 2 "" H 1300 7000 50  0001 C CNN
+F 2 "Package_SO:SOIC-14_3.9x8.7mm_P1.27mm" H 1300 7000 50  0001 C CNN
 F 3 "http://www.intersil.com/content/dam/Intersil/documents/cd40/cd4011bms-12bms-23bms.pdf" H 1300 7000 50  0001 C CNN
 	5    1300 7000
@@
 F 0 "C13" H 600 7050 50  0000 L CNN
 F 1 "100n" H 550 6950 50  0000 L CNN
-F 2 "" H 888 6850 50  0001 C CNN
+F 2 "Capacitor_SMD:C_0805_2012Metric_Pad1.15x1.40mm_HandSolder" H 888 6850 50  0001 C CNN
 F 3 "~" H 850 7000 50  0001 C CNN
 	1    850  7000
@@
 F 0 "C15" H 2215 7046 50  0000 L CNN
 F 1 "100n" H 2215 6955 50  0000 L CNN
-F 2 "" H 2138 6850 50  0001 C CNN
+F 2 "Capacitor_SMD:C_0805_2012Metric_Pad1.15x1.40mm_HandSolder" H 2138 6850 50  0001 C CNN
 F 3 "~" H 2100 7000 50  0001 C CNN
 	1    2100 7000
@@
 F 0 "U6" H 7800 4250 50  0000 C CNN
 F 1 "CD4053BM96" H 7800 4150 50  0000 C CNN
-F 2 "" H 7500 2650 50  0001 L CNN
+F 2 "Package_SO:SOIC-16_4.55x10.3mm_P1.27mm" H 7500 2650 50  0001 L CNN
 F 3 "" H 7330 3600 50  0001 C CNN
 	1    7350 3400
@@
 F 0 "U4" H 4000 1400 50  0000 C CNN
 F 1 "4011" H 4000 1300 50  0000 C CNN
-F 2 "" H 4000 1650 50  0001 C CNN
+F 2 "Package_SO:SOIC-14_3.9x8.7mm_P1.27mm" H 4000 1650 50  0001 C CNN
 F 3 "http://www.intersil.com/content/dam/Intersil/documents/cd40/cd4011bms-12bms-23bms.pdf" H 4000 1650 50  0001 C CNN
 	2    4000 1650
@@
 F 0 "U4" H 4800 1200 50  0000 C CNN
 F 1 "4011" H 4800 1100 50  0000 C CNN
-F 2 "" H 4800 1400 50  0001 C CNN
+F 2 "Package_SO:SOIC-14_3.9x8.7mm_P1.27mm" H 4800 1400 50  0001 C CNN
 F 3 "http://www.intersil.com/content/dam/Intersil/documents/cd40/cd4011bms-12bms-23bms.pdf" H 4800 1400 50  0001 C CNN
 	4    4800 1400
@@
 F 0 "U4" H 3200 1175 50  0000 C CNN
 F 1 "4011" H 3200 1100 50  0000 C CNN
-F 2 "" H 3200 1400 50  0001 C CNN
+F 2 "Package_SO:SOIC-14_3.9x8.7mm_P1.27mm" H 3200 1400 50  0001 C CNN
 F 3 "http://www.intersil.com/content/dam/Intersil/documents/cd40/cd4011bms-12bms-23bms.pdf" H 3200 1400 50  0001 C CNN
 	3    3200 1400
@@
 F 0 "U4" H 4000 1475 50  0000 C CNN
 F 1 "4011" H 4000 1384 50  0000 C CNN
-F 2 "" H 4000 1150 50  0001 C CNN
+F 2 "Package_SO:SOIC-14_3.9x8.7mm_P1.27mm" H 4000 1150 50  0001 C CNN
 F 3 "http://www.intersil.com/content/dam/Intersil/documents/cd40/cd4011bms-12bms-23bms.pdf" H 4000 1150 50  0001 C CNN
 	1    4000 1150
@@
 F 0 "C16" H 2815 7046 50  0000 L CNN
 F 1 "100n" H 2815 6955 50  0000 L CNN
-F 2 "" H 2738 6850 50  0001 C CNN
+F 2 "Capacitor_SMD:C_0805_2012Metric_Pad1.15x1.40mm_HandSolder" H 2738 6850 50  0001 C CNN
 F 3 "~" H 2700 7000 50  0001 C CNN
 	1    2700 7000
@@
 F 0 "R31" H 8870 4046 50  0000 L CNN
 F 1 "10k" H 8870 3955 50  0000 L CNN
-F 2 "" V 8730 4000 50  0001 C CNN
+F 2 "Resistor_SMD:R_0805_2012Metric_Pad1.15x1.40mm_HandSolder" V 8730 4000 50  0001 C CNN
 F 3 "~" H 8800 4000 50  0001 C CNN
 	1    8800 4000
@@
 F 0 "R35" H 9520 4046 50  0000 L CNN
 F 1 "10k" H 9520 3955 50  0000 L CNN
-F 2 "" V 9380 4000 50  0001 C CNN
+F 2 "Resistor_SMD:R_0805_2012Metric_Pad1.15x1.40mm_HandSolder" V 9380 4000 50  0001 C CNN
 F 3 "~" H 9450 4000 50  0001 C CNN
 	1    9450 4000
@@
 F 0 "R33" H 8920 2896 50  0000 L CNN
 F 1 "NC" H 8920 2805 50  0000 L CNN
-F 2 "" V 8780 2850 50  0001 C CNN
+F 2 "Resistor_SMD:R_0805_2012Metric_Pad1.15x1.40mm_HandSolder" V 8780 2850 50  0001 C CNN
 F 3 "~" H 8850 2850 50  0001 C CNN
 	1    8850 2850
@@
 F 0 "R29" V 6807 2750 50  0000 C CNN
 F 1 "10k" V 6716 2750 50  0000 C CNN
-F 2 "" V 6530 2750 50  0001 C CNN
+F 2 "Resistor_SMD:R_0805_2012Metric_Pad1.15x1.40mm_HandSolder" V 6530 2750 50  0001 C CNN
 F 3 "~" H 6600 2750 50  0001 C CNN
 	1    6600 2750
@@
 F 0 "U5" H 4700 4250 50  0000 C CNN
 F 1 "CD4053BM96" H 4700 4150 50  0000 C CNN
-F 2 "" H 4400 2650 50  0001 L CNN
+F 2 "Package_SO:SOIC-16_4.55x10.3mm_P1.27mm" H 4400 2650 50  0001 L CNN
 F 3 "" H 4230 3600 50  0001 C CNN
 	1    4250 3400
@@
 F 0 "R30" V 6500 3200 50  0000 C CNN
 F 1 "10k" V 6400 3200 50  0000 C CNN
-F 2 "" V 6530 3200 50  0001 C CNN
+F 2 "Resistor_SMD:R_0805_2012Metric_Pad1.15x1.40mm_HandSolder" V 6530 3200 50  0001 C CNN
 F 3 "~" H 6600 3200 50  0001 C CNN
 	1    6600 3200
@@
 F 0 "R32" H 8870 5446 50  0000 L CNN
 F 1 "10k" H 8870 5355 50  0000 L CNN
-F 2 "" V 8730 5400 50  0001 C CNN
+F 2 "Resistor_SMD:R_0805_2012Metric_Pad1.15x1.40mm_HandSolder" V 8730 5400 50  0001 C CNN
 F 3 "~" H 8800 5400 50  0001 C CNN
 	1    8800 5400
@@
 F 0 "R36" H 9520 5446 50  0000 L CNN
 F 1 "10k" H 9520 5355 50  0000 L CNN
-F 2 "" V 9380 5400 50  0001 C CNN
+F 2 "Resistor_SMD:R_0805_2012Metric_Pad1.15x1.40mm_HandSolder" V 9380 5400 50  0001 C CNN
 F 3 "~" H 9450 5400 50  0001 C CNN
 	1    9450 5400
@@
 F 0 "R34" H 9170 2896 50  0000 L CNN
 F 1 "NC" H 9170 2805 50  0000 L CNN
-F 2 "" V 9030 2850 50  0001 C CNN
+F 2 "Resistor_SMD:R_0805_2012Metric_Pad1.15x1.40mm_HandSolder" V 9030 2850 50  0001 C CNN
 F 3 "~" H 9100 2850 50  0001 C CNN
 	1    9100 2850
@@
 F 0 "TP14" H 10250 3750 50  0000 L CNN
 F 1 "TP_POP" H 10300 3850 50  0000 C CNN
-F 2 "" H 10500 3500 50  0001 C CNN
+F 2 "TestPoint:TestPoint_Loop_D1.80mm_Drill1.0mm_Beaded" H 10500 3500 50  0001 C CNN
 F 3 "~" H 10500 3500 50  0001 C CNN
 	1    10300 3500
@@
 F 0 "TP15" H 10250 3850 50  0000 L CNN
 F 1 "TP_POP" H 10300 3950 50  0000 C CNN
-F 2 "" H 10500 3600 50  0001 C CNN
+F 2 "TestPoint:TestPoint_Loop_D1.80mm_Drill1.0mm_Beaded" H 10500 3600 50  0001 C CNN
 F 3 "~" H 10500 3600 50  0001 C CNN
 	1    10300 3600
@@
 F 0 "TP17" H 10250 5250 50  0000 L CNN
 F 1 "TP_POP" H 10300 5350 50  0000 C CNN
-F 2 "" H 10500 5000 50  0001 C CNN
+F 2 "TestPoint:TestPoint_Loop_D1.80mm_Drill1.0mm_Beaded" H 10500 5000 50  0001 C CNN
 F 3 "~" H 10500 5000 50  0001 C CNN
 	1    10300 5000
@@
 F 0 "TP16" H 10250 5150 50  0000 L CNN
 F 1 "TP_POP" H 10300 5250 50  0000 C CNN
-F 2 "" H 10500 4900 50  0001 C CNN
+F 2 "TestPoint:TestPoint_Loop_D1.80mm_Drill1.0mm_Beaded" H 10500 4900 50  0001 C CNN
 F 3 "~" H 10500 4900 50  0001 C CNN
 	1    10300 4900
@@
 F 0 "TP12" H 6000 1650 50  0000 L CNN
 F 1 "TP_POP" H 6050 1750 50  0000 C CNN
-F 2 "" H 6250 1400 50  0001 C CNN
+F 2 "TestPoint:TestPoint_Loop_D1.80mm_Drill1.0mm_Beaded" H 6250 1400 50  0001 C CNN
 F 3 "~" H 6250 1400 50  0001 C CNN
 	1    6050 1400
@@
 F 0 "TP13" H 8200 6100 50  0000 L CNN
 F 1 "TP_POP" H 8250 6200 50  0000 C CNN
-F 2 "" H 8450 5850 50  0001 C CNN
+F 2 "TestPoint:TestPoint_Loop_D1.80mm_Drill1.0mm_Beaded" H 8450 5850 50  0001 C CNN
 F 3 "~" H 8450 5850 50  0001 C CNN
 	1    8250 5850
@@
 F 0 "TP11" H 5850 4050 50  0000 L CNN
 F 1 "TP_NOP" H 5900 4150 50  0000 C CNN
-F 2 "" H 6100 3800 50  0001 C CNN
+F 2 "TestPoint:TestPoint_THTPad_D2.0mm_Drill1.0mm" H 6100 3800 50  0001 C CNN
 F 3 "~" H 6100 3800 50  0001 C CNN
 	1    5900 3800
@@
 F 0 "TP10" H 5850 3850 50  0000 L CNN
 F 1 "TP_NOP" H 5900 3950 50  0000 C CNN
-F 2 "" H 6100 3600 50  0001 C CNN
+F 2 "TestPoint:TestPoint_THTPad_D2.0mm_Drill1.0mm" H 6100 3600 50  0001 C CNN
 F 3 "~" H 6100 3600 50  0001 C CNN
 	1    5900 3600

Commit message: added footprint for sepic coil + no more errors in netlist
Parts:
- C13, C15, C16: footprint Capacitor_SMD:C_0805_2012Metric_Pad1.15x1.40mm_HandSolder -> Sesame_footprint:C_0805_2012Metric_Pad1.18x1.45mm_HandSolder
- R29, R30, R31, R32, R33, R34, R35, R36: footprint Resistor_SMD:R_0805_2012Metric_Pad1.15x1.40mm_HandSolder -> Sesame_footprint:R_0805_2012Metric_Pad1.20x1.40mm_HandSolder
Changed lines of the file:
@@
 F 0 "C13" H 600 7050 50  0000 L CNN
 F 1 "100n" H 550 6950 50  0000 L CNN
-F 2 "Capacitor_SMD:C_0805_2012Metric_Pad1.15x1.40mm_HandSolder" H 888 6850 50  0001 C CNN
+F 2 "Sesame_footprint:C_0805_2012Metric_Pad1.18x1.45mm_HandSolder" H 888 6850 50  0001 C CNN
 F 3 "~" H 850 7000 50  0001 C CNN
 	1    850  7000
@@
 F 0 "C15" H 2215 7046 50  0000 L CNN
 F 1 "100n" H 2215 6955 50  0000 L CNN
-F 2 "Capacitor_SMD:C_0805_2012Metric_Pad1.15x1.40mm_HandSolder" H 2138 6850 50  0001 C CNN
+F 2 "Sesame_footprint:C_0805_2012Metric_Pad1.18x1.45mm_HandSolder" H 2138 6850 50  0001 C CNN
 F 3 "~" H 2100 7000 50  0001 C CNN
 	1    2100 7000
@@
 F 0 "C16" H 2815 7046 50  0000 L CNN
 F 1 "100n" H 2815 6955 50  0000 L CNN
-F 2 "Capacitor_SMD:C_0805_2012Metric_Pad1.15x1.40mm_HandSolder" H 2738 6850 50  0001 C CNN
+F 2 "Sesame_footprint:C_0805_2012Metric_Pad1.18x1.45mm_HandSolder" H 2738 6850 50  0001 C CNN
 F 3 "~" H 2700 7000 50  0001 C CNN
 	1    2700 7000
@@
 F 0 "R31" H 8870 4046 50  0000 L CNN
 F 1 "10k" H 8870 3955 50  0000 L CNN
-F 2 "Resistor_SMD:R_0805_2012Metric_Pad1.15x1.40mm_HandSolder" V 8730 4000 50  0001 C CNN
+F 2 "Sesame_footprint:R_0805_2012Metric_Pad1.20x1.40mm_HandSolder" V 8730 4000 50  0001 C CNN
 F 3 "~" H 8800 4000 50  0001 C CNN
 	1    8800 4000
@@
 F 0 "R35" H 9520 4046 50  0000 L CNN
 F 1 "10k" H 9520 3955 50  0000 L CNN
-F 2 "Resistor_SMD:R_0805_2012Metric_Pad1.15x1.40mm_HandSolder" V 9380 4000 50  0001 C CNN
+F 2 "Sesame_footprint:R_0805_2012Metric_Pad1.20x1.40mm_HandSolder" V 9380 4000 50  0001 C CNN
 F 3 "~" H 9450 4000 50  0001 C CNN
 	1    9450 4000
@@
 F 0 "R33" H 8920 2896 50  0000 L CNN
 F 1 "NC" H 8920 2805 50  0000 L CNN
-F 2 "Resistor_SMD:R_0805_2012Metric_Pad1.15x1.40mm_HandSolder" V 8780 2850 50  0001 C CNN
+F 2 "Sesame_footprint:R_0805_2012Metric_Pad1.20x1.40mm_HandSolder" V 8780 2850 50  0001 C CNN
 F 3 "~" H 8850 2850 50  0001 C CNN
 	1    8850 2850
@@
 F 0 "R29" V 6807 2750 50  0000 C CNN
 F 1 "10k" V 6716 2750 50  0000 C CNN
-F 2 "Resistor_SMD:R_0805_2012Metric_Pad1.15x1.40mm_HandSolder" V 6530 2750 50  0001 C CNN
+F 2 "Sesame_footprint:R_0805_2012Metric_Pad1.20x1.40mm_HandSolder" V 6530 2750 50  0001 C CNN
 F 3 "~" H 6600 2750 50  0001 C CNN
 	1    6600 2750
@@
 F 0 "R30" V 6500 3200 50  0000 C CNN
 F 1 "10k" V 6400 3200 50  0000 C CNN
-F 2 "Resistor_SMD:R_0805_2012Metric_Pad1.15x1.40mm_HandSolder" V 6530 3200 50  0001 C CNN
+F 2 "Sesame_footprint:R_0805_2012Metric_Pad1.20x1.40mm_HandSolder" V 6530 3200 50  0001 C CNN
 F 3 "~" H 6600 3200 50  0001 C CNN
 	1    6600 3200
@@
 F 0 "R32" H 8870 5446 50  0000 L CNN
 F 1 "10k" H 8870 5355 50  0000 L CNN
-F 2 "Resistor_SMD:R_0805_2012Metric_Pad1.15x1.40mm_HandSolder" V 8730 5400 50  0001 C CNN
+F 2 "Sesame_footprint:R_0805_2012Metric_Pad1.20x1.40mm_HandSolder" V 8730 5400 50  0001 C CNN
 F 3 "~" H 8800 5400 50  0001 C CNN
 	1    8800 5400
@@
 F 0 "R36" H 9520 5446 50  0000 L CNN
 F 1 "10k" H 9520 5355 50  0000 L CNN
-F 2 "Resistor_SMD:R_0805_2012Metric_Pad1.15x1.40mm_HandSolder" V 9380 5400 50  0001 C CNN
+F 2 "Sesame_footprint:R_0805_2012Metric_Pad1.20x1.40mm_HandSolder" V 9380 5400 50  0001 C CNN
 F 3 "~" H 9450 5400 50  0001 C CNN
 	1    9450 5400
@@
 F 0 "R34" H 9170 2896 50  0000 L CNN
 F 1 "NC" H 9170 2805 50  0000 L CNN
-F 2 "Resistor_SMD:R_0805_2012Metric_Pad1.15x1.40mm_HandSolder" V 9030 2850 50  0001 C CNN
+F 2 "Sesame_footprint:R_0805_2012Metric_Pad1.20x1.40mm_HandSolder" V 9030 2850 50  0001 C CNN
 F 3 "~" H 9100 2850 50  0001 C CNN
 	1    9100 2850

Commit message: 200 conn. remaining
Parts:
- U5, U6: footprint Package_SO:SOIC-16_4.55x10.3mm_P1.27mm -> Package_SO:SOIC-16_3.9x9.9mm_P1.27mm
Changed lines of the file:
@@
 F 0 "U6" H 7800 4250 50  0000 C CNN
 F 1 "CD4053BM96" H 7800 4150 50  0000 C CNN
-F 2 "Package_SO:SOIC-16_4.55x10.3mm_P1.27mm" H 7500 2650 50  0001 L CNN
+F 2 "Package_SO:SOIC-16_3.9x9.9mm_P1.27mm" H 7500 2650 50  0001 L CNN
 F 3 "" H 7330 3600 50  0001 C CNN
 	1    7350 3400
@@
 F 0 "U5" H 4700 4250 50  0000 C CNN
 F 1 "CD4053BM96" H 4700 4150 50  0000 C CNN
-F 2 "Package_SO:SOIC-16_4.55x10.3mm_P1.27mm" H 4400 2650 50  0001 L CNN
+F 2 "Package_SO:SOIC-16_3.9x9.9mm_P1.27mm" H 4400 2650 50  0001 L CNN
 F 3 "" H 4230 3600 50  0001 C CNN
 	1    4250 3400

Commit message: lil cleanup on the main schematic sheet
Parts:
- C13, C15, C16: symbol Device:C -> sesame-fonctionnel-rescue:C-Device
- R29, R30, R31, R32, R33, R34, R35, R36: symbol Device:R -> sesame-fonctionnel-rescue:R-Device
- TP10, TP11, TP12, TP13, TP14, TP15, TP16, TP17: symbol Connector:TestPoint -> sesame-fonctionnel-rescue:TestPoint-Connector
- U4: symbol 4xxx:4011 -> sesame-fonctionnel-rescue:4011-4xxx
Changed lines of the file:
@@
 	850  6500 850  6850
 $Comp
-L 4xxx:4011 U4
+L sesame-fonctionnel-rescue:4011-4xxx U4
 U 5 1 610DDCAD
 P 1300 7000
@@
 $EndComp
 $Comp
-L power:GND #PWR038
+L sesame-fonctionnel-rescue:GND-power #PWR038
 U 1 1 610E393A
 P 1300 7500
@@
 Connection ~ 1300 7500
 $Comp
-L Device:C C13
+L sesame-fonctionnel-rescue:C-Device C13
 U 1 1 610C6593
 P 850 7000
@@
 $EndComp
 $Comp
-L power:GND #PWR056
+L sesame-fonctionnel-rescue:GND-power #PWR056
 U 1 1 61156299
 P 9450 4200
@@
 $EndComp
 $Comp
-L power:GND #PWR053
+L sesame-fonctionnel-rescue:GND-power #PWR053
 U 1 1 610F5D5C
 P 8800 4200
@@
 	7300 4200 7300 4150
 $Comp
-L power:GND #PWR051
+L sesame-fonctionnel-rescue:GND-power #PWR051
 U 1 1 610EA813
 P 7300 4200
@@
 Pull-down MOS in parallel
 $Comp
-L power:GND #PWR049
+L sesame-fonctionnel-rescue:GND-power #PWR049
 U 1 1 612292EA
 P 6400 2800
@@
 	6850 3200 6750 3200
 $Comp
-L power:VCC #PWR037
+L sesame-fonctionnel-rescue:VCC-power #PWR037
 U 1 1 615841AD
 P 1300 6500
@@
 $EndComp
 $Comp
-L power:GND #PWR?
+L sesame-fonctionnel-rescue:GND-power #PWR?
 U 1 1 61587C63
 P 2100 7150
@@
 $EndComp
 $Comp
-L Device:C C?
+L sesame-fonctionnel-rescue:C-Device C?
 U 1 1 61587C69
 P 2100 7000
@@
 $EndComp
 $Comp
-L power:VCC #PWR?
+L sesame-fonctionnel-rescue:VCC-power #PWR?
 U 1 1 61587C6F
 P 2100 6850
@@
 $EndComp
 $Comp
-L 4xxx:4011 U4
+L sesame-fonctionnel-rescue:4011-4xxx U4
 U 2 1 6119334A
 P 4000 1650
@@
 $EndComp
 $Comp
-L 4xxx:4011 U4
+L sesame-fonctionnel-rescue:4011-4xxx U4
 U 4 1 6119F84F
 P 4800 1400
@@
 $EndComp
 $Comp
-L 4xxx:4011 U4
+L sesame-fonctionnel-rescue:4011-4xxx U4
 U 3 1 61192492
 P 3200 1400
@@
 $EndComp
 $Comp
-L 4xxx:4011 U4
+L sesame-fonctionnel-rescue:4011-4xxx U4
 U 1 1 61194533
 P 4000 1150
@@
 $EndComp
 $Comp
-L power:GND #PWR?
+L sesame-fonctionnel-rescue:GND-power #PWR?
 U 1 1 6143955C
 P 2700 7150
@@
 $EndComp
 $Comp
-L Device:C C?
+L sesame-fonctionnel-rescue:C-Device C?
 U 1 1 61439562
 P 2700 7000
@@
 $EndComp
 $Comp
-L power:VCC #PWR?
+L sesame-fonctionnel-rescue:VCC-power #PWR?
 U 1 1 61439568
 P 2700 6850
@@
 XOR Gate
 $Comp
-L power:GND #PWR054
+L sesame-fonctionnel-rescue:GND-power #PWR054
 U 1 1 61454AC0
 P 8850 3000
@@
 $EndComp
 $Comp
-L Device:R R31
+L sesame-fonctionnel-rescue:R-Device R31
 U 1 1 61492A34
 P 8800 4000
@@
 $EndComp
 $Comp
-L Device:R R35
+L sesame-fonctionnel-rescue:R-Device R35
 U 1 1 6149304C
 P 9450 4000
@@
 $EndComp
 $Comp
-L Device:R R33
+L sesame-fonctionnel-rescue:R-Device R33
 U 1 1 6128A052
 P 8850 2850
@@
 $EndComp
 $Comp
-L power:GND #PWR050
+L sesame-fonctionnel-rescue:GND-power #PWR050
 U 1 1 612A5111
 P 6400 3250
@@
 	6300 2300 6300 4750
 $Comp
-L power:VCC #PWR052
+L sesame-fonctionnel-rescue:VCC-power #PWR052
 U 1 1 6147E979
 P 7450 2650
@@
 $EndComp
 $Comp
-L Device:R R29
+L sesame-fonctionnel-rescue:R-Device R29
 U 1 1 61526169
 P 6600 2750
@@
 	6850 3100 6800 3100
 $Comp
-L power:VCC #PWR046
+L sesame-fonctionnel-rescue:VCC-power #PWR046
 U 1 1 6147EE29
 P 4350 2650
@@
 	5050 3200 5050 3150
 $Comp
-L power:VCC #PWR047
+L sesame-fonctionnel-rescue:VCC-power #PWR047
 U 1 1 61311635
 P 5050 3150
@@
 	5050 3350 5050 3300
 $Comp
-L power:GND #PWR048
+L sesame-fonctionnel-rescue:GND-power #PWR048
 U 1 1 6130709D
 P 5050 3350
@@
 	3650 4000 3650 3900
 $Comp
-L power:GND #PWR044
+L sesame-fonctionnel-rescue:GND-power #PWR044
 U 1 1 613BCF5A
 P 3650 4000
@@
 	4250 4150 4250 4100
 $Comp
-L power:GND #PWR045
+L sesame-fonctionnel-rescue:GND-power #PWR045
 U 1 1 613BCF4A
 P 4200 4200
@@
 	6050 1400 6050 3100
 $Comp
-L Device:R R30
+L sesame-fonctionnel-rescue:R-Device R30
 U 1 1 61353D13
 P 6600 3200
@@
 Resistor_pull
 $Comp
-L Device:R R32
+L sesame-fonctionnel-rescue:R-Device R32
 U 1 1 6149251A
 P 8800 5400
@@
 $EndComp
 $Comp
-L Device:R R36
+L sesame-fonctionnel-rescue:R-Device R36
 U 1 1 6114A712
 P 9450 5400
@@
 Connection ~ 9450 5000
 $Comp
-L power:GND #PWR055
+L sesame-fonctionnel-rescue:GND-power #PWR055
 U 1 1 613D46B1
 P 9100 3000
@@
 $EndComp
 $Comp
-L Device:R R34
+L sesame-fonctionnel-rescue:R-Device R34
 U 1 1 613D46B7
 P 9100 2850
@@
 Connection ~ 8800 5850
 $Comp
-L Connector:TestPoint TP?
+L sesame-fonctionnel-rescue:TestPoint-Connector TP?
 U 1 1 613F5D58
 P 10300 3500
@@
 	10300 3500 10575 3500
 $Comp
-L Connector:TestPoint TP?
+L sesame-fonctionnel-rescue:TestPoint-Connector TP?
 U 1 1 61400B10
 P 10300 3600
@@
 	10300 3600 10575 3600
 $Comp
-L Connector:TestPoint TP?
+L sesame-fonctionnel-rescue:TestPoint-Connector TP?
 U 1 1 61407FD3
 P 10300 5000
@@
 $EndComp
 $Comp
-L Connector:TestPoint TP?
+L sesame-fonctionnel-rescue:TestPoint-Connector TP?
 U 1 1 6140B9F0
 P 10300 4900
@@
 	10300 5000 10550 5000
 $Comp
-L Connector:TestPoint TP?
+L sesame-fonctionnel-rescue:TestPoint-Connector TP?
 U 1 1 61415864
 P 6050 1400
@@
 Connection ~ 4800 3600
 $Comp
-L Connector:TestPoint TP?
+L sesame-fonctionnel-rescue:TestPoint-Connector TP?
 U 1 1 61446F7B
 P 8250 5850
@@
 PWM_Series
 $Comp
-L Connector:TestPoint TP?
+L sesame-fonctionnel-rescue:TestPoint-Connector TP?
 U 1 1 6146B21F
 P 5900 3800
@@
 	6050 3100 6800 3100
 $Comp
-L Connector:TestPoint TP?
+L sesame-fonctionnel-rescue:TestPoint-Connector TP?
 U 1 1 6146AAD7
 P 5900 3600
