File: KICAD/DC_DC_Converter.sch (KiCad schematic (older format))
At the start: 7 parts

Commit message: mainly footprints
Parts:
- added C? (x5): 470uF, symbol Device:CP
- added C? (x3): C, symbol Device:C
- C?: value CP -> 470uF
Connections:
- wire segments 21 -> 51
Other:
- moved on the sheet: C?

Commit message: revex with jmt
Parts:
- QLP, QLS, QRP, QRS: footprint (none) -> Package_TO_SOT_SMD:TO-263-2
Other:
- note added: "Inductor between 90uH -> 125uH\nhttps://fr.rs-online.com/web/p/inductances-traversantes/1816037\nhttps://fr.rs-online.com/web/p/inductances-traversantes/1542466\nhttps://fr.rs-online.com/web/p/inductances-traversantes/1048448"
- note removed: "Bobine TBD !"
- note removed: "D2PAK"

Commit message: review w/ jmt
Parts:
- added C41, C42, C43, C44: C, symbol Device:C
- added R89, R90, R91, R92, R93, R94, R95, R96: R, symbol Device:R
- gave numbers to parts that had none: 10
- renumbered L1 to L2, QLP to QLP1, QLS to QLS1, QRP to QRP1, QRS to QRS1
Connections:
- net labels added: GND
- net labels removed: GNDPWR
- wire segments 51 -> 85
Other:
- moved on the sheet: C36, C37, C38, C39, C40, C45, C46, C47, C48, C49, L2, QLP1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

Commit message: edit footprints by jmt
Parts:
- C36, C37, C38, C47, C48, C49: footprint (none) -> Capacitor_THT:CP_Radial_D12.5mm_P5.00mm
- C39, C40, C41, C42, C43, C44, C45, C46: footprint (none) -> Capacitor_SMD:C_0805_2012Metric_Pad1.15x1.40mm_HandSolder
- R89, R90, R91, R92, R93, R94, R95, R96: footprint (none) -> Resistor_SMD:R_0805_2012Metric_Pad1.15x1.40mm_HandSolder
Changed lines of the file:
@@
 F 0 "R91" H 5270 3196 50  0000 L CNN
 F 1 "R" H 5270 3105 50  0000 L CNN
-F 2 "" V 5130 3150 50  0001 C CNN
+F 2 "Resistor_SMD:R_0805_2012Metric_Pad1.15x1.40mm_HandSolder" V 5130 3150 50  0001 C CNN
 F 3 "~" H 5200 3150 50  0001 C CNN
 	1    5200 3150
@@
 F 0 "C41" H 5315 2696 50  0000 L CNN
 F 1 "C" H 5315 2605 50  0000 L CNN
-F 2 "" H 5238 2500 50  0001 C CNN
+F 2 "Capacitor_SMD:C_0805_2012Metric_Pad1.15x1.40mm_HandSolder" H 5238 2500 50  0001 C CNN
 F 3 "~" H 5200 2650 50  0001 C CNN
 	1    5200 2650
@@
 F 0 "C46" H 8865 2796 50  0000 L CNN
 F 1 "C" H 8865 2705 50  0000 L CNN
-F 2 "" H 8788 2600 50  0001 C CNN
+F 2 "Capacitor_SMD:C_0805_2012Metric_Pad1.15x1.40mm_HandSolder" H 8788 2600 50  0001 C CNN
 F 3 "~" H 8750 2750 50  0001 C CNN
 	1    8750 2750
@@
 F 0 "C47" H 9268 2796 50  0000 L CNN
 F 1 "470uF" H 9268 2705 50  0000 L CNN
-F 2 "" H 9188 2600 50  0001 C CNN
+F 2 "Capacitor_THT:CP_Radial_D12.5mm_P5.00mm" H 9188 2600 50  0001 C CNN
 F 3 "~" H 9150 2750 50  0001 C CNN
 	1    9150 2750
@@
 F 0 "C48" H 9768 2796 50  0000 L CNN
 F 1 "470uF" H 9768 2705 50  0000 L CNN
-F 2 "" H 9688 2600 50  0001 C CNN
+F 2 "Capacitor_THT:CP_Radial_D12.5mm_P5.00mm" H 9688 2600 50  0001 C CNN
 F 3 "~" H 9650 2750 50  0001 C CNN
 	1    9650 2750
@@
 F 0 "C49" H 10268 2796 50  0000 L CNN
 F 1 "470uF" H 10268 2705 50  0000 L CNN
-F 2 "" H 10188 2600 50  0001 C CNN
+F 2 "Capacitor_THT:CP_Radial_D12.5mm_P5.00mm" H 10188 2600 50  0001 C CNN
 F 3 "~" H 10150 2750 50  0001 C CNN
 	1    10150 2750
@@
 F 0 "C45" H 8465 2796 50  0000 L CNN
 F 1 "C" H 8465 2705 50  0000 L CNN
-F 2 "" H 8388 2600 50  0001 C CNN
+F 2 "Capacitor_SMD:C_0805_2012Metric_Pad1.15x1.40mm_HandSolder" H 8388 2600 50  0001 C CNN
 F 3 "~" H 8350 2750 50  0001 C CNN
 	1    8350 2750
@@
 F 0 "R93" H 6370 3196 50  0000 L CNN
 F 1 "R" H 6370 3105 50  0000 L CNN
-F 2 "" V 6230 3150 50  0001 C CNN
+F 2 "Resistor_SMD:R_0805_2012Metric_Pad1.15x1.40mm_HandSolder" V 6230 3150 50  0001 C CNN
 F 3 "~" H 6300 3150 50  0001 C CNN
 	1    6300 3150
@@
 F 0 "C43" H 6415 2696 50  0000 L CNN
 F 1 "C" H 6415 2605 50  0000 L CNN
-F 2 "" H 6338 2500 50  0001 C CNN
+F 2 "Capacitor_SMD:C_0805_2012Metric_Pad1.15x1.40mm_HandSolder" H 6338 2500 50  0001 C CNN
 F 3 "~" H 6300 2650 50  0001 C CNN
 	1    6300 2650
@@
 F 0 "R92" H 5270 4396 50  0000 L CNN
 F 1 "R" H 5270 4305 50  0000 L CNN
-F 2 "" V 5130 4350 50  0001 C CNN
+F 2 "Resistor_SMD:R_0805_2012Metric_Pad1.15x1.40mm_HandSolder" V 5130 4350 50  0001 C CNN
 F 3 "~" H 5200 4350 50  0001 C CNN
 	1    5200 4350
@@
 F 0 "C42" H 5315 3896 50  0000 L CNN
 F 1 "C" H 5315 3805 50  0000 L CNN
-F 2 "" H 5238 3700 50  0001 C CNN
+F 2 "Capacitor_SMD:C_0805_2012Metric_Pad1.15x1.40mm_HandSolder" H 5238 3700 50  0001 C CNN
 F 3 "~" H 5200 3850 50  0001 C CNN
 	1    5200 3850
@@
 F 0 "R94" H 6370 4396 50  0000 L CNN
 F 1 "R" H 6370 4305 50  0000 L CNN
-F 2 "" V 6230 4350 50  0001 C CNN
+F 2 "Resistor_SMD:R_0805_2012Metric_Pad1.15x1.40mm_HandSolder" V 6230 4350 50  0001 C CNN
 F 3 "~" H 6300 4350 50  0001 C CNN
 	1    6300 4350
@@
 F 0 "C44" H 6415 3896 50  0000 L CNN
 F 1 "C" H 6415 3805 50  0000 L CNN
-F 2 "" H 6338 3700 50  0001 C CNN
+F 2 "Capacitor_SMD:C_0805_2012Metric_Pad1.15x1.40mm_HandSolder" H 6338 3700 50  0001 C CNN
 F 3 "~" H 6300 3850 50  0001 C CNN
 	1    6300 3850
@@
 F 0 "R90" H 4220 4496 50  0000 L CNN
 F 1 "R" H 4220 4405 50  0000 L CNN
-F 2 "" V 4080 4450 50  0001 C CNN
+F 2 "Resistor_SMD:R_0805_2012Metric_Pad1.15x1.40mm_HandSolder" V 4080 4450 50  0001 C CNN
 F 3 "~" H 4150 4450 50  0001 C CNN
 	1    4150 4450
@@
 F 0 "R96" H 7570 4496 50  0000 L CNN
 F 1 "R" H 7570 4405 50  0000 L CNN
-F 2 "" V 7430 4450 50  0001 C CNN
+F 2 "Resistor_SMD:R_0805_2012Metric_Pad1.15x1.40mm_HandSolder" V 7430 4450 50  0001 C CNN
 F 3 "~" H 7500 4450 50  0001 C CNN
 	1    7500 4450
@@
 F 0 "R89" H 4220 3296 50  0000 L CNN
 F 1 "R" H 4220 3205 50  0000 L CNN
-F 2 "" V 4080 3250 50  0001 C CNN
+F 2 "Resistor_SMD:R_0805_2012Metric_Pad1.15x1.40mm_HandSolder" V 4080 3250 50  0001 C CNN
 F 3 "~" H 4150 3250 50  0001 C CNN
 	1    4150 3250
@@
 F 0 "R95" H 7570 3296 50  0000 L CNN
 F 1 "R" H 7570 3205 50  0000 L CNN
-F 2 "" V 7430 3250 50  0001 C CNN
+F 2 "Resistor_SMD:R_0805_2012Metric_Pad1.15x1.40mm_HandSolder" V 7430 3250 50  0001 C CNN
 F 3 "~" H 7500 3250 50  0001 C CNN
 	1    7500 3250
@@
 F 0 "C40" H 3515 2796 50  0000 L CNN
 F 1 "C" H 3515 2705 50  0000 L CNN
-F 2 "" H 3438 2600 50  0001 C CNN
+F 2 "Capacitor_SMD:C_0805_2012Metric_Pad1.15x1.40mm_HandSolder" H 3438 2600 50  0001 C CNN
 F 3 "~" H 3400 2750 50  0001 C CNN
 	1    3400 2750
@@
 F 0 "C36" H 1718 2796 50  0000 L CNN
 F 1 "470uF" H 1718 2705 50  0000 L CNN
-F 2 "" H 1638 2600 50  0001 C CNN
+F 2 "Capacitor_THT:CP_Radial_D12.5mm_P5.00mm" H 1638 2600 50  0001 C CNN
 F 3 "~" H 1600 2750 50  0001 C CNN
 	1    1600 2750
@@
 F 0 "C37" H 2218 2796 50  0000 L CNN
 F 1 "470uF" H 2218 2705 50  0000 L CNN
-F 2 "" H 2138 2600 50  0001 C CNN
+F 2 "Capacitor_THT:CP_Radial_D12.5mm_P5.00mm" H 2138 2600 50  0001 C CNN
 F 3 "~" H 2100 2750 50  0001 C CNN
 	1    2100 2750
@@
 F 0 "C38" H 2718 2796 50  0000 L CNN
 F 1 "470uF" H 2718 2705 50  0000 L CNN
-F 2 "" H 2638 2600 50  0001 C CNN
+F 2 "Capacitor_THT:CP_Radial_D12.5mm_P5.00mm" H 2638 2600 50  0001 C CNN
 F 3 "~" H 2600 2750 50  0001 C CNN
 	1    2600 2750
@@
 F 0 "C39" H 3115 2796 50  0000 L CNN
 F 1 "C" H 3115 2705 50  0000 L CNN
-F 2 "" H 3038 2600 50  0001 C CNN
+F 2 "Capacitor_SMD:C_0805_2012Metric_Pad1.15x1.40mm_HandSolder" H 3038 2600 50  0001 C CNN
 F 3 "~" H 3000 2750 50  0001 C CNN
 	1    3000 2750

Commit message: route + work on djd
Parts:
- L2: footprint (none) -> Sesame_footprint:Multi-coil
Changed lines of the file:
@@
 $Descr A4 11693 8268
 encoding utf-8
-Sheet 17 17
+Sheet 16 17
 Title "SESAME"
 Date ""
@@
 F 0 "L2" H 5750 3765 50  0000 C CNN
 F 1 "INDUCTOR" H 5750 3674 50  0000 C CNN
-F 2 "" H 5750 3550 50  0001 C CNN
+F 2 "Sesame_footprint:Multi-coil" H 5750 3550 50  0001 C CNN
 F 3 "~" H 5750 3550 50  0001 C CNN
 	1    5750 3550
@@
 	-1   0    0    -1
 $EndComp
+Text Label 4600 2350 0    50   ~ 0
+VD_LS
+Text Label 7050 2350 2    50   ~ 0
+VD_RS
+Text Label 7050 3550 2    50   ~ 0
+VS_R
+Text Label 4600 3550 0    50   ~ 0
+VS_L
 $EndSCHEMATC

Commit message: added footprint for sepic coil + no more errors in netlist
Parts:
- C39, C40, C41, C42, C43, C44, C45, C46: footprint Capacitor_SMD:C_0805_2012Metric_Pad1.15x1.40mm_HandSolder -> Sesame_footprint:C_0805_2012Metric_Pad1.18x1.45mm_HandSolder
- R89, R90, R91, R92, R93, R94, R95, R96: footprint Resistor_SMD:R_0805_2012Metric_Pad1.15x1.40mm_HandSolder -> Sesame_footprint:R_0805_2012Metric_Pad1.20x1.40mm_HandSolder
Changed lines of the file:
@@
 F 0 "R91" H 5270 3196 50  0000 L CNN
 F 1 "R" H 5270 3105 50  0000 L CNN
-F 2 "Resistor_SMD:R_0805_2012Metric_Pad1.15x1.40mm_HandSolder" V 5130 3150 50  0001 C CNN
+F 2 "Sesame_footprint:R_0805_2012Metric_Pad1.20x1.40mm_HandSolder" V 5130 3150 50  0001 C CNN
 F 3 "~" H 5200 3150 50  0001 C CNN
 	1    5200 3150
@@
 F 0 "C41" H 5315 2696 50  0000 L CNN
 F 1 "C" H 5315 2605 50  0000 L CNN
-F 2 "Capacitor_SMD:C_0805_2012Metric_Pad1.15x1.40mm_HandSolder" H 5238 2500 50  0001 C CNN
+F 2 "Sesame_footprint:C_0805_2012Metric_Pad1.18x1.45mm_HandSolder" H 5238 2500 50  0001 C CNN
 F 3 "~" H 5200 2650 50  0001 C CNN
 	1    5200 2650
@@
 F 0 "C46" H 8865 2796 50  0000 L CNN
 F 1 "C" H 8865 2705 50  0000 L CNN
-F 2 "Capacitor_SMD:C_0805_2012Metric_Pad1.15x1.40mm_HandSolder" H 8788 2600 50  0001 C CNN
+F 2 "Sesame_footprint:C_0805_2012Metric_Pad1.18x1.45mm_HandSolder" H 8788 2600 50  0001 C CNN
 F 3 "~" H 8750 2750 50  0001 C CNN
 	1    8750 2750
@@
 F 0 "C45" H 8465 2796 50  0000 L CNN
 F 1 "C" H 8465 2705 50  0000 L CNN
-F 2 "Capacitor_SMD:C_0805_2012Metric_Pad1.15x1.40mm_HandSolder" H 8388 2600 50  0001 C CNN
+F 2 "Sesame_footprint:C_0805_2012Metric_Pad1.18x1.45mm_HandSolder" H 8388 2600 50  0001 C CNN
 F 3 "~" H 8350 2750 50  0001 C CNN
 	1    8350 2750
@@
 F 0 "R93" H 6370 3196 50  0000 L CNN
 F 1 "R" H 6370 3105 50  0000 L CNN
-F 2 "Resistor_SMD:R_0805_2012Metric_Pad1.15x1.40mm_HandSolder" V 6230 3150 50  0001 C CNN
+F 2 "Sesame_footprint:R_0805_2012Metric_Pad1.20x1.40mm_HandSolder" V 6230 3150 50  0001 C CNN
 F 3 "~" H 6300 3150 50  0001 C CNN
 	1    6300 3150
@@
 F 0 "C43" H 6415 2696 50  0000 L CNN
 F 1 "C" H 6415 2605 50  0000 L CNN
-F 2 "Capacitor_SMD:C_0805_2012Metric_Pad1.15x1.40mm_HandSolder" H 6338 2500 50  0001 C CNN
+F 2 "Sesame_footprint:C_0805_2012Metric_Pad1.18x1.45mm_HandSolder" H 6338 2500 50  0001 C CNN
 F 3 "~" H 6300 2650 50  0001 C CNN
 	1    6300 2650
@@
 F 0 "R92" H 5270 4396 50  0000 L CNN
 F 1 "R" H 5270 4305 50  0000 L CNN
-F 2 "Resistor_SMD:R_0805_2012Metric_Pad1.15x1.40mm_HandSolder" V 5130 4350 50  0001 C CNN
+F 2 "Sesame_footprint:R_0805_2012Metric_Pad1.20x1.40mm_HandSolder" V 5130 4350 50  0001 C CNN
 F 3 "~" H 5200 4350 50  0001 C CNN
 	1    5200 4350
@@
 F 0 "C42" H 5315 3896 50  0000 L CNN
 F 1 "C" H 5315 3805 50  0000 L CNN
-F 2 "Capacitor_SMD:C_0805_2012Metric_Pad1.15x1.40mm_HandSolder" H 5238 3700 50  0001 C CNN
+F 2 "Sesame_footprint:C_0805_2012Metric_Pad1.18x1.45mm_HandSolder" H 5238 3700 50  0001 C CNN
 F 3 "~" H 5200 3850 50  0001 C CNN
 	1    5200 3850
@@
 F 0 "R94" H 6370 4396 50  0000 L CNN
 F 1 "R" H 6370 4305 50  0000 L CNN
-F 2 "Resistor_SMD:R_0805_2012Metric_Pad1.15x1.40mm_HandSolder" V 6230 4350 50  0001 C CNN
+F 2 "Sesame_footprint:R_0805_2012Metric_Pad1.20x1.40mm_HandSolder" V 6230 4350 50  0001 C CNN
 F 3 "~" H 6300 4350 50  0001 C CNN
 	1    6300 4350
@@
 F 0 "C44" H 6415 3896 50  0000 L CNN
 F 1 "C" H 6415 3805 50  0000 L CNN
-F 2 "Capacitor_SMD:C_0805_2012Metric_Pad1.15x1.40mm_HandSolder" H 6338 3700 50  0001 C CNN
+F 2 "Sesame_footprint:C_0805_2012Metric_Pad1.18x1.45mm_HandSolder" H 6338 3700 50  0001 C CNN
 F 3 "~" H 6300 3850 50  0001 C CNN
 	1    6300 3850
@@
 F 0 "R90" H 4220 4496 50  0000 L CNN
 F 1 "R" H 4220 4405 50  0000 L CNN
-F 2 "Resistor_SMD:R_0805_2012Metric_Pad1.15x1.40mm_HandSolder" V 4080 4450 50  0001 C CNN
+F 2 "Sesame_footprint:R_0805_2012Metric_Pad1.20x1.40mm_HandSolder" V 4080 4450 50  0001 C CNN
 F 3 "~" H 4150 4450 50  0001 C CNN
 	1    4150 4450
@@
 F 0 "R96" H 7570 4496 50  0000 L CNN
 F 1 "R" H 7570 4405 50  0000 L CNN
-F 2 "Resistor_SMD:R_0805_2012Metric_Pad1.15x1.40mm_HandSolder" V 7430 4450 50  0001 C CNN
+F 2 "Sesame_footprint:R_0805_2012Metric_Pad1.20x1.40mm_HandSolder" V 7430 4450 50  0001 C CNN
 F 3 "~" H 7500 4450 50  0001 C CNN
 	1    7500 4450
@@
 F 0 "R89" H 4220 3296 50  0000 L CNN
 F 1 "R" H 4220 3205 50  0000 L CNN
-F 2 "Resistor_SMD:R_0805_2012Metric_Pad1.15x1.40mm_HandSolder" V 4080 3250 50  0001 C CNN
+F 2 "Sesame_footprint:R_0805_2012Metric_Pad1.20x1.40mm_HandSolder" V 4080 3250 50  0001 C CNN
 F 3 "~" H 4150 3250 50  0001 C CNN
 	1    4150 3250
@@
 F 0 "R95" H 7570 3296 50  0000 L CNN
 F 1 "R" H 7570 3205 50  0000 L CNN
-F 2 "Resistor_SMD:R_0805_2012Metric_Pad1.15x1.40mm_HandSolder" V 7430 3250 50  0001 C CNN
+F 2 "Sesame_footprint:R_0805_2012Metric_Pad1.20x1.40mm_HandSolder" V 7430 3250 50  0001 C CNN
 F 3 "~" H 7500 3250 50  0001 C CNN
 	1    7500 3250
@@
 F 0 "C40" H 3515 2796 50  0000 L CNN
 F 1 "C" H 3515 2705 50  0000 L CNN
-F 2 "Capacitor_SMD:C_0805_2012Metric_Pad1.15x1.40mm_HandSolder" H 3438 2600 50  0001 C CNN
+F 2 "Sesame_footprint:C_0805_2012Metric_Pad1.18x1.45mm_HandSolder" H 3438 2600 50  0001 C CNN
 F 3 "~" H 3400 2750 50  0001 C CNN
 	1    3400 2750
@@
 F 0 "C39" H 3115 2796 50  0000 L CNN
 F 1 "C" H 3115 2705 50  0000 L CNN
-F 2 "Capacitor_SMD:C_0805_2012Metric_Pad1.15x1.40mm_HandSolder" H 3038 2600 50  0001 C CNN
+F 2 "Sesame_footprint:C_0805_2012Metric_Pad1.18x1.45mm_HandSolder" H 3038 2600 50  0001 C CNN
 F 3 "~" H 3000 2750 50  0001 C CNN
 	1    3000 2750
