File: KICAD/DC_DC_Converter.sch (KiCad schematic (older format))
At the start: 27 parts

Commit message: lil cleanup on the main schematic sheet
Parts:
- C36, C37, C38, C47, C48, C49: symbol Device:CP -> sesame-fonctionnel-rescue:CP-Device
- C39, C40, C41, C42, C43, C44, C45, C46: symbol Device:C -> sesame-fonctionnel-rescue:C-Device
- L2: symbol pspice:INDUCTOR -> sesame-fonctionnel-rescue:INDUCTOR-pspice
- QLP1, QLS1, QRP1, QRS1: symbol Device:Q_NMOS_GDS -> sesame-fonctionnel-rescue:Q_NMOS_GDS-Device
- R89, R90, R91, R92, R93, R94, R95, R96: symbol Device:R -> sesame-fonctionnel-rescue:R-Device
Changed lines of the file:
@@
 VG_LP
 $Comp
-L Device:Q_NMOS_GDS QLS1
+L sesame-fonctionnel-rescue:Q_NMOS_GDS-Device QLS1
 U 1 1 610E334F
 P 4450 2950
@@
 $EndComp
 $Comp
-L pspice:INDUCTOR L2
+L sesame-fonctionnel-rescue:INDUCTOR-pspice L2
 U 1 1 610F3EF5
 P 5750 3550
@@
 	4000 3550 4150 3550
 $Comp
-L Device:R R91
+L sesame-fonctionnel-rescue:R-Device R91
 U 1 1 61ABF7A3
 P 5200 3150
@@
 $EndComp
 $Comp
-L Device:C C41
+L sesame-fonctionnel-rescue:C-Device C41
 U 1 1 61AC857C
 P 5200 2650
@@
 	4550 4350 4550 4750
 $Comp
-L Device:Q_NMOS_GDS QLP1
+L sesame-fonctionnel-rescue:Q_NMOS_GDS-Device QLP1
 U 1 1 610EEE2E
 P 4450 4150
@@
 $EndComp
 $Comp
-L Device:Q_NMOS_GDS QRP1
+L sesame-fonctionnel-rescue:Q_NMOS_GDS-Device QRP1
 U 1 1 610F2085
 P 7200 4150
@@
 VG_RS
 $Comp
-L Device:Q_NMOS_GDS QRS1
+L sesame-fonctionnel-rescue:Q_NMOS_GDS-Device QRS1
 U 1 1 610F207F
 P 7200 2950
@@
 	7600 2950 7500 2950
 $Comp
-L Device:C C46
+L sesame-fonctionnel-rescue:C-Device C46
 U 1 1 6149AEB6
 P 8750 2750
@@
 $EndComp
 $Comp
-L Device:CP C47
+L sesame-fonctionnel-rescue:CP-Device C47
 U 1 1 6149B9CD
 P 9150 2750
@@
 $EndComp
 $Comp
-L Device:CP C48
+L sesame-fonctionnel-rescue:CP-Device C48
 U 1 1 615C9A23
 P 9650 2750
@@
 $EndComp
 $Comp
-L Device:CP C49
+L sesame-fonctionnel-rescue:CP-Device C49
 U 1 1 615CA3E5
 P 10150 2750
@@
 $EndComp
 $Comp
-L Device:C C45
+L sesame-fonctionnel-rescue:C-Device C45
 U 1 1 615CB20D
 P 8350 2750
@@
 	5200 3550 5500 3550
 $Comp
-L Device:R R93
+L sesame-fonctionnel-rescue:R-Device R93
 U 1 1 61AF6D76
 P 6300 3150
@@
 $EndComp
 $Comp
-L Device:C C43
+L sesame-fonctionnel-rescue:C-Device C43
 U 1 1 61AF6D7C
 P 6300 2650
@@
 	6300 3550 6000 3550
 $Comp
-L Device:R R92
+L sesame-fonctionnel-rescue:R-Device R92
 U 1 1 61AFCB5F
 P 5200 4350
@@
 $EndComp
 $Comp
-L Device:C C42
+L sesame-fonctionnel-rescue:C-Device C42
 U 1 1 61AFCB65
 P 5200 3850
@@
 	5200 4500 5200 4750
 $Comp
-L Device:R R94
+L sesame-fonctionnel-rescue:R-Device R94
 U 1 1 61AFE399
 P 6300 4350
@@
 $EndComp
 $Comp
-L Device:C C44
+L sesame-fonctionnel-rescue:C-Device C44
 U 1 1 61AFE39F
 P 6300 3850
@@
 	6300 4750 7100 4750
 $Comp
-L Device:R R90
+L sesame-fonctionnel-rescue:R-Device R90
 U 1 1 61B03C5B
 P 4150 4450
@@
 Connection ~ 4550 4750
 $Comp
-L Device:R R96
+L sesame-fonctionnel-rescue:R-Device R96
 U 1 1 61B0B5A6
 P 7500 4450
@@
 Connection ~ 7100 4750
 $Comp
-L Device:R R89
+L sesame-fonctionnel-rescue:R-Device R89
 U 1 1 61B1964C
 P 4150 3250
@@
 	4150 2950 4250 2950
 $Comp
-L Device:R R95
+L sesame-fonctionnel-rescue:R-Device R95
 U 1 1 61B29627
 P 7500 3250
@@
 	7500 3550 7100 3550
 $Comp
-L power:GND #PWR0128
+L sesame-fonctionnel-rescue:GND-power #PWR0128
 U 1 1 61B83564
 P 8350 3150
@@
 $EndComp
 $Comp
-L power:GND #PWR0129
+L sesame-fonctionnel-rescue:GND-power #PWR0129
 U 1 1 61B83A89
 P 8750 3150
@@
 $EndComp
 $Comp
-L power:GND #PWR0130
+L sesame-fonctionnel-rescue:GND-power #PWR0130
 U 1 1 61B841A2
 P 9150 3150
@@
 $EndComp
 $Comp
-L power:GND #PWR0131
+L sesame-fonctionnel-rescue:GND-power #PWR0131
 U 1 1 61B8455E
 P 9650 3150
@@
 $EndComp
 $Comp
-L power:GND #PWR0132
+L sesame-fonctionnel-rescue:GND-power #PWR0132
 U 1 1 61B847F4
 P 10150 3150
@@
 Connection ~ 4550 2350
 $Comp
-L power:GND #PWR0122
+L sesame-fonctionnel-rescue:GND-power #PWR0122
 U 1 1 61B86FB5
 P 1600 3150
@@
 $EndComp
 $Comp
-L power:GND #PWR0123
+L sesame-fonctionnel-rescue:GND-power #PWR0123
 U 1 1 61B86FAF
 P 2100 3150
@@
 $EndComp
 $Comp
-L power:GND #PWR0124
+L sesame-fonctionnel-rescue:GND-power #PWR0124
 U 1 1 61B86FA9
 P 2600 3150
@@
 $EndComp
 $Comp
-L power:GND #PWR0125
+L sesame-fonctionnel-rescue:GND-power #PWR0125
 U 1 1 61B86FA3
 P 3000 3150
@@
 $EndComp
 $Comp
-L power:GND #PWR0126
+L sesame-fonctionnel-rescue:GND-power #PWR0126
 U 1 1 61B86F9D
 P 3400 3150
@@
 	3400 3150 3400 2900
 $Comp
-L Device:C C40
+L sesame-fonctionnel-rescue:C-Device C40
 U 1 1 616023EF
 P 3400 2750
@@
 $EndComp
 $Comp
-L Device:CP C36
+L sesame-fonctionnel-rescue:CP-Device C36
 U 1 1 616023E9
 P 1600 2750
@@
 $EndComp
 $Comp
-L Device:CP C37
+L sesame-fonctionnel-rescue:CP-Device C37
 U 1 1 616023E3
 P 2100 2750
@@
 $EndComp
 $Comp
-L Device:CP C38
+L sesame-fonctionnel-rescue:CP-Device C38
 U 1 1 616023DD
 P 2600 2750
@@
 $EndComp
 $Comp
-L Device:C C39
+L sesame-fonctionnel-rescue:C-Device C39
 U 1 1 616023D7
 P 3000 2750
@@
 VD_LS
 $Comp
-L power:GND #PWR0127
+L sesame-fonctionnel-rescue:GND-power #PWR0127
 U 1 1 61B9B9A2
 P 5750 4850

Commit message: V1.0 of the schematic
Other:
- note added: "Inductor between 90uH -> 125uH\nhttps://fr.rs-online.com/web/p/inductances-traversantes/1816037\nhttps://fr.rs-online.com/web/p/inductances-traversantes/1542466\nhttps://fr.rs-online.com/web/p/inductances-traversantes/1048448\nhttps://fr.rs-online.com/web/p/inductances-traversantes/1229231"
- note removed: "Inductor between 90uH -> 125uH\nhttps://fr.rs-online.com/web/p/inductances-traversantes/1816037\nhttps://fr.rs-online.com/web/p/inductances-traversantes/1542466\nhttps://fr.rs-online.com/web/p/inductances-traversantes/1048448"
Changed lines of the file:
@@
 $Descr A4 11693 8268
 encoding utf-8
-Sheet 16 17
+Sheet 12 17
 Title "SESAME"
-Date ""
-Rev ""
+Date "2021-09-23"
+Rev "1"
 Comp "ALEEA"
 Comment1 "Dessin : Guillaume Arthaud"
@@
 	10150 2350 9650 2350
 Text Notes 4600 1300 0    50   ~ 0
-Inductor between 90uH -> 125uH\nhttps://fr.rs-online.com/web/p/inductances-traversantes/1816037\nhttps://fr.rs-online.com/web/p/inductances-traversantes/1542466\nhttps://fr.rs-online.com/web/p/inductances-traversantes/1048448
+Inductor between 90uH -> 125uH\nhttps://fr.rs-online.com/web/p/inductances-traversantes/1816037\nhttps://fr.rs-online.com/web/p/inductances-traversantes/1542466\nhttps://fr.rs-online.com/web/p/inductances-traversantes/1048448\nhttps://fr.rs-online.com/web/p/inductances-traversantes/1229231
 Wire Wire Line
 	10150 3150 10150 2900
