File: KICAD/sesame-fonctionnel.kicad_pcb (KiCad board)
At the start: 2 copper layers, 0 parts

Commit message: added footprint lib + steps for connectors
Parts:
- added REF**: CXS70-14-C, Sesame_footprint:CXS70-14-C, F.Cu at (155.6, 93.3)
Changed lines of the file:
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@@
     (tracks 0)
     (zones 0)
-    (modules 0)
+    (modules 1)
     (nets 1)
   )
@@
     (uvia_drill 0.1)
   )
+  (module Sesame_footprint:CXS70-14-C (layer F.Cu)
+    (at 155.6 93.3)
+    (fp_text reference REF** (at 0 -13) (layer F.SilkS)
+      (effects (font (size 1 1) (thickness 0.15)))
+    )
+    (fp_text value CXS70-14-C (at 0 -11.25) (layer F.Fab)
+      (effects (font (size 1 1) (thickness 0.15)))
+    )
+    (fp_poly (pts (xy 8.35 11.3) (xy -8.35 11.3) (xy -8.35 -9.9) (xy 8.35 -9.9)) (layer F.Mask) (width 0.1))
+    (fp_poly (pts (xy 8.35 11.3) (xy -8.35 11.3) (xy -8.35 -9.9) (xy 8.35 -9.9)) (layer F.Cu) (width 0.1))
+    (fp_poly (pts (xy 8.35 11.3) (xy -8.35 11.3) (xy -8.35 -9.9) (xy 8.35 -9.9)) (layer B.Cu) (width 0.1))
+    (fp_line (start -8.35 11.3) (end 8.35 11.3) (layer Dwgs.User) (width 0.12))
+    (fp_line (start 8.35 -9.9) (end 8.35 11.3) (layer Dwgs.User) (width 0.12))
+    (fp_line (start -8.35 -9.9) (end -8.35 11.3) (layer Dwgs.User) (width 0.12))
+    (fp_line (start -8.35 -9.9) (end 8.35 -9.9) (layer Dwgs.User) (width 0.12))
+    (fp_poly (pts (xy 8.35 11.3) (xy -8.35 11.3) (xy -8.35 -9.9) (xy 8.35 -9.9)) (layer B.Mask) (width 0.1))
+    (fp_line (start -6.35 11.3) (end 6.35 11.3) (layer Dwgs.User) (width 0.12))
+    (fp_line (start 6.35 -7.9) (end 6.35 11.3) (layer Dwgs.User) (width 0.12))
+    (fp_line (start -6.35 -7.9) (end 6.35 -7.9) (layer Dwgs.User) (width 0.12))
+    (fp_line (start -6.35 -7.9) (end -6.35 11.3) (layer Dwgs.User) (width 0.12))
+    (pad "" thru_hole circle (at -3 5) (size 2 2) (drill 1) (layers *.Cu *.Mask))
+    (pad "" thru_hole circle (at 3 5) (size 2 2) (drill 1) (layers *.Cu *.Mask))
+    (pad "" thru_hole circle (at 6 -2) (size 2 2) (drill 1) (layers *.Cu *.Mask))
+    (pad "" thru_hole circle (at 6 2) (size 2 2) (drill 1) (layers *.Cu *.Mask))
+    (pad "" thru_hole circle (at 6 5) (size 2 2) (drill 1) (layers *.Cu *.Mask))
+    (pad "" thru_hole circle (at 6 8) (size 2 2) (drill 1) (layers *.Cu *.Mask))
+    (pad "" thru_hole circle (at 3 8) (size 2 2) (drill 1) (layers *.Cu *.Mask))
+    (pad "" thru_hole circle (at 0 8) (size 2 2) (drill 1) (layers *.Cu *.Mask))
+    (pad "" thru_hole circle (at -3 8) (size 2 2) (drill 1) (layers *.Cu *.Mask))
+    (pad "" thru_hole circle (at -6 8) (size 2 2) (drill 1) (layers *.Cu *.Mask))
+    (pad "" thru_hole circle (at -6 5) (size 2 2) (drill 1) (layers *.Cu *.Mask))
+    (pad "" thru_hole circle (at -6 2) (size 2 2) (drill 1) (layers *.Cu *.Mask))
+    (pad "" thru_hole circle (at -6 -2) (size 2 2) (drill 1) (layers *.Cu *.Mask))
+    (pad "" thru_hole circle (at 3 -5) (size 2 2) (drill 1) (layers *.Cu *.Mask))
+    (pad "" thru_hole circle (at -3 -5) (size 2 2) (drill 1) (layers *.Cu *.Mask))
+    (pad "" thru_hole circle (at -6 -5) (size 2 2) (drill 1) (layers *.Cu *.Mask))
+    (pad "" thru_hole circle (at 6 -5) (size 2 2) (drill 1) (layers *.Cu *.Mask))
+    (pad "" thru_hole circle (at 6 -8) (size 2 2) (drill 1) (layers *.Cu *.Mask))
+    (pad "" thru_hole circle (at 3 -8) (size 2 2) (drill 1) (layers *.Cu *.Mask))
+    (pad "" thru_hole circle (at -6 -8) (size 2 2) (drill 1) (layers *.Cu *.Mask))
+    (pad "" thru_hole circle (at -3 -8) (size 2 2) (drill 1) (layers *.Cu *.Mask))
+    (pad "" thru_hole circle (at 0 -8) (size 2 2) (drill 1) (layers *.Cu *.Mask))
+    (pad 1 thru_hole circle (at 0 0) (size 10.8 10.8) (drill 6.8) (layers *.Cu *.Mask))
+    (model STEP/CXS70-14-C.STEP
+      (offset (xyz -6.4 7.9 0))
+      (scale (xyz 1 1 1))
+      (rotate (xyz 0 0 90))
+    )
+    (model STEP/keystone-PN6095.STEP
+      (offset (xyz 1 1.25 -1))
+      (scale (xyz 1 1 1))
+      (rotate (xyz -90 0 0))
+    )
+  )
 )
