File: KICAD/alims.sch (KiCad schematic (older format))
At the start: 5 parts

Commit message: ebauche driver mos
Connections:
- net VCC renamed +7V
Other:
- note removed: "A definir"
- note removed: "A definir\n\n"
Changed lines of the file:
@@
 Comment4 ""
 $EndDescr
-Text HLabel 2200 800  0    50   Input ~ 0
-Dir
 Text HLabel 2250 1400 0    50   Input ~ 0
 LEFT
 Text HLabel 2250 1750 0    50   Input ~ 0
 RIGHT
-Text HLabel 4150 1100 2    50   Output ~ 0
-5V
 Text HLabel 6050 1950 2    50   Output ~ 0
 VREF
-Text HLabel 6050 1100 2    50   Output ~ 0
-VMOS
 Text Notes 3000 3050 0    50   ~ 0
 Gen 5v and Vref\n
@@
 	6050 1950 5950 1950
 Connection ~ 5950 1950
-$Comp
-L power:VCC #PWR0105
-U 1 1 612FE019
-P 4650 1600
-F 0 "#PWR0105" H 4650 1450 50  0001 C CNN
-F 1 "VCC" H 4665 1773 50  0000 C CNN
-F 2 "" H 4650 1600 50  0001 C CNN
-F 3 "" H 4650 1600 50  0001 C CNN
-	1    4650 1600
-	1    0    0    -1
-$EndComp
 $Comp
 L power:GND #PWR0106
@@
 Wire Wire Line
 	2850 1750 2850 1400
-$Comp
-L power:VCC #PWR0107
-U 1 1 614DE65E
-P 6000 1050
-F 0 "#PWR0107" H 6000 900 50  0001 C CNN
-F 1 "VCC" H 6015 1223 50  0000 C CNN
-F 2 "" H 6000 1050 50  0001 C CNN
-F 3 "" H 6000 1050 50  0001 C CNN
-	1    6000 1050
-	1    0    0    -1
-$EndComp
-Wire Wire Line
-	6000 1050 6000 1100
-Wire Wire Line
-	6000 1100 6050 1100
-Wire Notes Line
-	6550 750  5850 750
-Wire Notes Line
-	5850 750  5850 1300
-Wire Notes Line
-	5850 1300 6550 1300
-Wire Notes Line
-	6550 750  6550 1300
-Text Notes 6050 1300 0    50   ~ 0
-A definir
-Wire Notes Line
-	2000 700  2350 700
-Wire Notes Line
-	2350 700  2350 1000
-Wire Notes Line
-	2350 1000 2000 1000
-Wire Notes Line
-	2000 1000 2000 700
-Text Notes 2050 950  0    50   ~ 0
-A definir\n\n
 $Comp
 L Device:D_Shockley D?
@@
 Wire Wire Line
 	5950 1500 5950 1950
+$Comp
+L Sesame:+7V #PWR?
+U 1 1 612A93DA
+P 4650 1600
+F 0 "#PWR?" H 4650 1450 50  0001 C CNN
+F 1 "+7V" H 4665 1773 50  0000 C CNN
+F 2 "" H 4650 1600 50  0001 C CNN
+F 3 "" H 4650 1600 50  0001 C CNN
+	1    4650 1600
+	1    0    0    -1
+$EndComp
 $EndSCHEMATC

Commit message: a ton of new stuff. V0.8
Connections:
- net +7V renamed VCC
Changed lines of the file:
@@
 $Descr A4 11693 8268
 encoding utf-8
-Sheet 14 15
+Sheet 14 16
 Title "SESAME"
 Date ""
@@
 	5950 1500 5950 1950
 $Comp
-L Sesame:+7V #PWR?
-U 1 1 612A93DA
+L power:VCC #PWR0178
+U 1 1 6158EF67
 P 4650 1600
-F 0 "#PWR?" H 4650 1450 50  0001 C CNN
-F 1 "+7V" H 4665 1773 50  0000 C CNN
+F 0 "#PWR0178" H 4650 1450 50  0001 C CNN
+F 1 "VCC" H 4665 1773 50  0000 C CNN
 F 2 "" H 4650 1600 50  0001 C CNN
 F 3 "" H 4650 1600 50  0001 C CNN

Commit message: worked on power supply + connectors
Parts:
- removed D? (x2): D_Shockley, symbol Device:D_Shockley
- added C? (x5): C, symbol Device:C
- added D? (x3): D_Schottky, symbol Device:D_Schottky
- added L2: L_Core_Ferrite_Coupled_2_Parts, symbol Sesame:L_Core_Ferrite_Coupled_2_Parts
- added R?: R, symbol Device:R
- added R?: 1M, symbol Device:R
- added R?: 296k, symbol Device:R
- added R?: 84.5, symbol Device:R
- added U1: LT8365, symbol Sesame:LT8365
Connections:
- net GND: now also C?.1, C?.2, C?.2, C?.2, L2.3, R?.2, R?.2, U1.12 (SYNC/MODE), U1.17 (GND)
- net LEFT: now also D?.2 (A)
- net RIGHT: now also D?.2 (A)
- net VCC: now also C?.2, D?.1 (K), R?.1, U1.7 (BIAS)
- new net: C?.2, L2.2, U1.14 (SW2), U1.16 (SW1)
- new net: R?.1, U1.10 (RT)
- new net: C?.1, U1.11 (SS)
- new net: C?.1, U1.5 (INTVCC)
- new net: R?.1, U1.8 (VC)
- new net: R?.1, R?.2, U1.9 (FBX)
- new net: C?.1, D?.2 (A), L2.4
- new net: C?.1, R?.2
- new net VIN: D?.1 (K), D?.1 (K), L2.1, U1.1 (EN/UVLO), U1.3 (VIN)
Other:
- note added: "RT = 432k -> 100 kHz\nRT = 143k -> 300 kHz\nRT = 84.5k -> 500 kHz"
- note removed: "Gen 5v and Vref\n"
- note removed: "The Dir pin chose from which side the power supply is generated"
- moved on the sheet: D?, R?, U?A

Commit message: lt6015 it is
Parts:
- removed U?: MCP602, symbol Amplifier_Operational:MCP602
- added U? (x2): AD8030, symbol Sesame:AD8030
Connections:
- net VREF: now also U?.1, U?.3 (+), U?.5 (+)
- net at D?.1 (K), R?.2: now also U?.2 (-)
- new net: U?.6 (-), U?.7
Other:
- note added: "VCC = 7V\nVREF = 6V"
Changed lines of the file:
@@
 $Descr A4 11693 8268
 encoding utf-8
-Sheet 13 16
+Sheet 15 16
 Title "SESAME"
 Date ""
@@
 	0    1    1    0
 $EndComp
-$Comp
-L Amplifier_Operational:MCP602 U?
-U 1 1 6108AD98
-P 9050 2900
-F 0 "U?" H 9050 2533 50  0000 C CNN
-F 1 "MCP602" H 9050 2624 50  0000 C CNN
-F 2 "" H 9050 2900 50  0001 C CNN
-F 3 "http://ww1.microchip.com/downloads/en/DeviceDoc/21314g.pdf" H 9050 2900 50  0001 C CNN
-	1    9050 2900
-	1    0    0    1
-$EndComp
 Wire Wire Line
 	8650 2450 9450 2450
@@
 P 6050 2900
 F 0 "L2" H 6050 3050 50  0000 C CNN
-F 1 "L_Core_Ferrite_Coupled_2_Parts" V 6900 2900 50  0000 C CNN
+F 1 "L_Core_Ferrite_Coupled_2_Parts" V 6750 3000 50  0001 C CNN
 F 2 "" H 6050 3000 50  0001 C CNN
 F 3 "~" H 6050 3000 50  0001 C CNN
@@
 	-1   0    0    1
 $EndComp
-Text Notes 2650 4700 0    50   ~ 0
+Text Notes 2600 4600 0    50   ~ 0
 RT = 432k  -> 100 kHz\nRT = 143k  -> 300 kHz\nRT = 84.5k -> 500 kHz
 $Comp
@@
 	9800 2900 9450 2900
 Connection ~ 9450 2900
+Text Notes 5050 1600 0    100  ~ 0
+VCC = 7V\nVREF = 6V
+$Comp
+L Sesame:AD8030 U?
+U 1 1 615918A8
+P 9050 2900
+F 0 "U?" H 9050 3267 50  0000 C CNN
+F 1 "AD8030" H 9050 3176 50  0000 C CNN
+F 2 "" H 9050 2900 50  0001 C CNN
+F 3 "~" H 9050 2900 50  0001 C CNN
+	1    9050 2900
+	1    0    0    -1
+$EndComp
+$Comp
+L Sesame:AD8030 U?
+U 2 1 61592FA9
+P 10200 4550
+F 0 "U?" H 10200 4917 50  0000 C CNN
+F 1 "AD8030" H 10200 4826 50  0000 C CNN
+F 2 "" H 10200 4550 50  0001 C CNN
+F 3 "~" H 10200 4550 50  0001 C CNN
+	2    10200 4550
+	1    0    0    -1
+$EndComp
+$Comp
+L Sesame:VREF #PWR?
+U 1 1 61598955
+P 9800 4400
+F 0 "#PWR?" H 9800 4250 50  0001 C CNN
+F 1 "VREF" H 9815 4573 50  0000 C CNN
+F 2 "" H 9800 4400 50  0001 C CNN
+F 3 "" H 9800 4400 50  0001 C CNN
+	1    9800 4400
+	1    0    0    -1
+$EndComp
+Wire Wire Line
+	9800 4400 9800 4450
+Wire Wire Line
+	9800 4450 9900 4450
+Wire Wire Line
+	10500 4550 10600 4550
+Wire Wire Line
+	10600 4550 10600 4900
+Wire Wire Line
+	10600 4900 9800 4900
+Wire Wire Line
+	9800 4900 9800 4650
+Wire Wire Line
+	9800 4650 9900 4650
 $EndSCHEMATC

Commit message: mainly footprints
Parts:
- added C?: 100n, symbol Device:C
- added U?: AD8030, Package_SO:SO-8_3.9x4.9mm_P1.27mm, symbol Sesame:AD8030
- D? (x3): value D_Schottky -> SS36; footprint (none) -> Diode_SMD:D_SMA_Handsoldering
- U? (x2): footprint (none) -> Package_SO:SO-8_3.9x4.9mm_P1.27mm
- renumbered U1 to U?
Connections:
- net GND: now also C?.2, U?.4 (V-)
- net VCC: now also C?.1, U?.8 (V+)
Changed lines of the file:
@@
 $EndComp
 $Comp
-L Sesame:LT8365 U1
+L Sesame:LT8365 U?
 U 1 1 6123C49A
 P 4850 3400
-F 0 "U1" H 3650 3700 100 0000 L CNN
+F 0 "U?" H 3650 3700 100 0000 L CNN
 F 1 "LT8365" H 3500 3550 100 0000 L CNN
 F 2 "" H 4850 4100 100 0001 C CNN
@@
 P 6300 2650
 F 0 "D?" H 6300 2433 50  0000 C CNN
-F 1 "D_Schottky" H 6300 2524 50  0000 C CNN
-F 2 "" H 6300 2650 50  0001 C CNN
+F 1 "SS36" H 6300 2524 50  0000 C CNN
+F 2 "Diode_SMD:D_SMA_Handsoldering" H 6300 2650 50  0001 C CNN
 F 3 "~" H 6300 2650 50  0001 C CNN
 	1    6300 2650
@@
 P 3400 2500
 F 0 "D?" H 3400 2283 50  0000 C CNN
-F 1 "D_Schottky" H 3400 2374 50  0000 C CNN
-F 2 "" H 3400 2500 50  0001 C CNN
+F 1 "SS36" H 3400 2374 50  0000 C CNN
+F 2 "Diode_SMD:D_SMA_Handsoldering" H 3400 2500 50  0001 C CNN
 F 3 "~" H 3400 2500 50  0001 C CNN
 	1    3400 2500
@@
 P 3400 2850
 F 0 "D?" H 3400 2633 50  0000 C CNN
-F 1 "D_Schottky" H 3400 2724 50  0000 C CNN
-F 2 "" H 3400 2850 50  0001 C CNN
+F 1 "SS36" H 3400 2724 50  0000 C CNN
+F 2 "Diode_SMD:D_SMA_Handsoldering" H 3400 2850 50  0001 C CNN
 F 3 "~" H 3400 2850 50  0001 C CNN
 	1    3400 2850
@@
 VCC = 7V\nVREF = 6V
 $Comp
-L Sesame:AD8030 U?
-U 1 1 615918A8
-P 9050 2900
-F 0 "U?" H 9050 3267 50  0000 C CNN
-F 1 "AD8030" H 9050 3176 50  0000 C CNN
-F 2 "" H 9050 2900 50  0001 C CNN
-F 3 "~" H 9050 2900 50  0001 C CNN
-	1    9050 2900
-	1    0    0    -1
-$EndComp
-$Comp
-L Sesame:AD8030 U?
-U 2 1 61592FA9
-P 10200 4550
-F 0 "U?" H 10200 4917 50  0000 C CNN
-F 1 "AD8030" H 10200 4826 50  0000 C CNN
-F 2 "" H 10200 4550 50  0001 C CNN
-F 3 "~" H 10200 4550 50  0001 C CNN
-	2    10200 4550
-	1    0    0    -1
-$EndComp
-$Comp
 L Sesame:VREF #PWR?
 U 1 1 61598955
@@
 Wire Wire Line
 	9800 4650 9900 4650
+$Comp
+L Device:C C?
+U 1 1 6161C7DE
+P 1350 6950
+AR Path="/60F1AF26/6161C7DE" Ref="C?"  Part="1"
+AR Path="/60F1B237/6161C7DE" Ref="C?"  Part="1"
+AR Path="/60F16FAE/6161C7DE" Ref="C?"  Part="1"
+AR Path="/60F171CE/6161C7DE" Ref="C?"  Part="1"
+AR Path="/60F19D5B/6161C7DE" Ref="C?"  Part="1"
+AR Path="/60F1AA92/6161C7DE" Ref="C?"  Part="1"
+F 0 "C?" H 1465 6996 50  0000 L CNN
+F 1 "100n" H 1465 6905 50  0000 L CNN
+F 2 "" H 1388 6800 50  0001 C CNN
+F 3 "~" H 1350 6950 50  0001 C CNN
+	1    1350 6950
+	1    0    0    -1
+$EndComp
+Wire Wire Line
+	1200 6550 1200 6600
+Wire Wire Line
+	1200 6600 1050 6600
+Wire Wire Line
+	1050 6600 1050 6650
+Connection ~ 1200 6600
+Wire Wire Line
+	1050 7300 1050 7250
+$Comp
+L power:GND #PWR?
+U 1 1 6161C7E9
+P 1200 7350
+AR Path="/60F1AF26/6161C7E9" Ref="#PWR?"  Part="1"
+AR Path="/60F1B237/6161C7E9" Ref="#PWR?"  Part="1"
+AR Path="/60F16FAE/6161C7E9" Ref="#PWR?"  Part="1"
+AR Path="/60F171CE/6161C7E9" Ref="#PWR?"  Part="1"
+AR Path="/60F19D5B/6161C7E9" Ref="#PWR?"  Part="1"
+AR Path="/60F1AA92/6161C7E9" Ref="#PWR?"  Part="1"
+F 0 "#PWR?" H 1200 7100 50  0001 C CNN
+F 1 "GND" H 1205 7177 50  0000 C CNN
+F 2 "" H 1200 7350 50  0001 C CNN
+F 3 "" H 1200 7350 50  0001 C CNN
+	1    1200 7350
+	1    0    0    -1
+$EndComp
+Wire Wire Line
+	1200 7350 1200 7300
+Connection ~ 1200 7300
+Wire Wire Line
+	1200 7300 1050 7300
+Wire Wire Line
+	1350 6600 1350 6800
+Wire Wire Line
+	1200 6600 1350 6600
+Wire Wire Line
+	1350 7100 1350 7300
+Wire Wire Line
+	1200 7300 1350 7300
+$Comp
+L power:VCC #PWR?
+U 1 1 6161C7F6
+P 1200 6550
+AR Path="/60F1AF26/6161C7F6" Ref="#PWR?"  Part="1"
+AR Path="/60F1B237/6161C7F6" Ref="#PWR?"  Part="1"
+AR Path="/60F16FAE/6161C7F6" Ref="#PWR?"  Part="1"
+AR Path="/60F171CE/6161C7F6" Ref="#PWR?"  Part="1"
+AR Path="/60F19D5B/6161C7F6" Ref="#PWR?"  Part="1"
+AR Path="/60F1AA92/6161C7F6" Ref="#PWR?"  Part="1"
+F 0 "#PWR?" H 1200 6400 50  0001 C CNN
+F 1 "VCC" H 1215 6723 50  0000 C CNN
+F 2 "" H 1200 6550 50  0001 C CNN
+F 3 "" H 1200 6550 50  0001 C CNN
+	1    1200 6550
+	1    0    0    -1
+$EndComp
+$Comp
+L Sesame:AD8030 U?
+U 3 1 6161C7FC
+P 1150 6950
+AR Path="/60F1AF26/6161C7FC" Ref="U?"  Part="3"
+AR Path="/60F1B237/6161C7FC" Ref="U?"  Part="3"
+AR Path="/60F16FAE/6161C7FC" Ref="U?"  Part="3"
+AR Path="/60F171CE/6161C7FC" Ref="U?"  Part="3"
+AR Path="/60F19D5B/6161C7FC" Ref="U?"  Part="3"
+AR Path="/60F1AA92/6161C7FC" Ref="U?"  Part="3"
+F 0 "U?" H 963 6904 50  0000 R CNN
+F 1 "AD8030" H 963 6995 50  0000 R CNN
+F 2 "Package_SO:SO-8_3.9x4.9mm_P1.27mm" H 1150 6950 50  0001 C CNN
+F 3 "~" H 1150 6950 50  0001 C CNN
+	3    1150 6950
+	1    0    0    -1
+$EndComp
+$Comp
+L Sesame:AD8030 U?
+U 2 1 61592FA9
+P 10200 4550
+F 0 "U?" H 10200 4917 50  0000 C CNN
+F 1 "AD8030" H 10200 4826 50  0000 C CNN
+F 2 "Package_SO:SO-8_3.9x4.9mm_P1.27mm" H 10200 4550 50  0001 C CNN
+F 3 "~" H 10200 4550 50  0001 C CNN
+	2    10200 4550
+	1    0    0    -1
+$EndComp
+$Comp
+L Sesame:AD8030 U?
+U 1 1 615918A8
+P 9050 2900
+F 0 "U?" H 9050 3267 50  0000 C CNN
+F 1 "AD8030" H 9050 3176 50  0000 C CNN
+F 2 "Package_SO:SO-8_3.9x4.9mm_P1.27mm" H 9050 2900 50  0001 C CNN
+F 3 "~" H 9050 2900 50  0001 C CNN
+	1    9050 2900
+	1    0    0    -1
+$EndComp
 $EndSCHEMATC
