File: KICAD/alims.sch (KiCad schematic (older format))
At the start: 24 parts, among them U14 AD8030, U15 LT8365

Commit message: 0 conn. + new vref
Parts:
- removed U14: AD8030, Package_SO:SO-8_5.3x6.2mm_P1.27mm, symbol Sesame:AD8030
- gave numbers to parts that had none: 3
Connections:
- wire segments 78 -> 73
Other:
- note removed: "REF TENSION AUTRE SOLUTION\n"
- moved on the sheet: C27, R28, R83, R84
Changed lines of the file:
@@
 L power:GND #PWR0114
 U 1 1 612FEB08
-P 10500 3750
-F 0 "#PWR0114" H 10500 3500 50  0001 C CNN
-F 1 "GND" H 10505 3577 50  0000 C CNN
-F 2 "" H 10500 3750 50  0001 C CNN
-F 3 "" H 10500 3750 50  0001 C CNN
-	1    10500 3750
-	1    0    0    -1
-$EndComp
-Wire Wire Line
-	10500 2500 10500 2600
+P 9500 4000
+F 0 "#PWR0114" H 9500 3750 50  0001 C CNN
+F 1 "GND" H 9505 3827 50  0000 C CNN
+F 2 "" H 9500 4000 50  0001 C CNN
+F 3 "" H 9500 4000 50  0001 C CNN
+	1    9500 4000
+	1    0    0    -1
+$EndComp
+Wire Wire Line
+	9500 2500 9500 2600
 Wire Wire Line
 	2050 2850 2200 2850
@@
 L Device:R R83
 U 1 1 61087C02
-P 10500 2750
-F 0 "R83" H 10570 2796 50  0000 L CNN
-F 1 "R" H 10570 2705 50  0000 L CNN
-F 2 "Sesame_footprint:R_0805_2012Metric_Pad1.20x1.40mm_HandSolder" V 10430 2750 50  0001 C CNN
-F 3 "~" H 10500 2750 50  0001 C CNN
-	1    10500 2750
+P 9500 2750
+F 0 "R83" H 9570 2796 50  0000 L CNN
+F 1 "R" H 9570 2705 50  0000 L CNN
+F 2 "Sesame_footprint:R_0805_2012Metric_Pad1.20x1.40mm_HandSolder" V 9430 2750 50  0001 C CNN
+F 3 "~" H 9500 2750 50  0001 C CNN
+	1    9500 2750
 	1    0    0    -1
 $EndComp
@@
 L power:VCC #PWR0113
 U 1 1 6158EF67
-P 10500 2500
-F 0 "#PWR0113" H 10500 2350 50  0001 C CNN
-F 1 "VCC" H 10515 2673 50  0000 C CNN
-F 2 "" H 10500 2500 50  0001 C CNN
-F 3 "" H 10500 2500 50  0001 C CNN
-	1    10500 2500
+P 9500 2500
+F 0 "#PWR0113" H 9500 2350 50  0001 C CNN
+F 1 "VCC" H 9515 2673 50  0000 C CNN
+F 2 "" H 9500 2500 50  0001 C CNN
+F 3 "" H 9500 2500 50  0001 C CNN
+	1    9500 2500
 	1    0    0    -1
 $EndComp
@@
 Text Notes 2550 1350 0    100  ~ 0
 VCC = 7V\nVREF = 6V
-$Comp
-L Device:C C?
-U 1 1 6161C7DE
-P 1350 6950
-AR Path="/60F1AF26/6161C7DE" Ref="C?"  Part="1"
-AR Path="/60F1B237/6161C7DE" Ref="C?"  Part="1"
-AR Path="/60F16FAE/6161C7DE" Ref="C?"  Part="1"
-AR Path="/60F171CE/6161C7DE" Ref="C?"  Part="1"
-AR Path="/60F19D5B/6161C7DE" Ref="C?"  Part="1"
-AR Path="/60F1AA92/6161C7DE" Ref="C27"  Part="1"
-F 0 "C27" H 1465 6996 50  0000 L CNN
-F 1 "100n" H 1465 6905 50  0000 L CNN
-F 2 "Sesame_footprint:C_0805_2012Metric_Pad1.18x1.45mm_HandSolder" H 1388 6800 50  0001 C CNN
-F 3 "~" H 1350 6950 50  0001 C CNN
-	1    1350 6950
-	1    0    0    -1
-$EndComp
-Wire Wire Line
-	1200 6550 1200 6600
-Wire Wire Line
-	1200 6600 1050 6600
-Wire Wire Line
-	1050 6600 1050 6650
-Connection ~ 1200 6600
-Wire Wire Line
-	1050 7300 1050 7250
-$Comp
-L power:GND #PWR?
-U 1 1 6161C7E9
-P 1200 7350
-AR Path="/60F1AF26/6161C7E9" Ref="#PWR?"  Part="1"
-AR Path="/60F1B237/6161C7E9" Ref="#PWR?"  Part="1"
-AR Path="/60F16FAE/6161C7E9" Ref="#PWR?"  Part="1"
-AR Path="/60F171CE/6161C7E9" Ref="#PWR?"  Part="1"
-AR Path="/60F19D5B/6161C7E9" Ref="#PWR?"  Part="1"
-AR Path="/60F1AA92/6161C7E9" Ref="#PWR0101"  Part="1"
-F 0 "#PWR0101" H 1200 7100 50  0001 C CNN
-F 1 "GND" H 1205 7177 50  0000 C CNN
-F 2 "" H 1200 7350 50  0001 C CNN
-F 3 "" H 1200 7350 50  0001 C CNN
-	1    1200 7350
-	1    0    0    -1
-$EndComp
-Wire Wire Line
-	1200 7350 1200 7300
-Connection ~ 1200 7300
-Wire Wire Line
-	1200 7300 1050 7300
-Wire Wire Line
-	1350 6600 1350 6800
-Wire Wire Line
-	1200 6600 1350 6600
-Wire Wire Line
-	1350 7100 1350 7300
-Wire Wire Line
-	1200 7300 1350 7300
-$Comp
-L power:VCC #PWR?
-U 1 1 6161C7F6
-P 1200 6550
-AR Path="/60F1AF26/6161C7F6" Ref="#PWR?"  Part="1"
-AR Path="/60F1B237/6161C7F6" Ref="#PWR?"  Part="1"
-AR Path="/60F16FAE/6161C7F6" Ref="#PWR?"  Part="1"
-AR Path="/60F171CE/6161C7F6" Ref="#PWR?"  Part="1"
-AR Path="/60F19D5B/6161C7F6" Ref="#PWR?"  Part="1"
-AR Path="/60F1AA92/6161C7F6" Ref="#PWR0100"  Part="1"
-F 0 "#PWR0100" H 1200 6400 50  0001 C CNN
-F 1 "VCC" H 1215 6723 50  0000 C CNN
-F 2 "" H 1200 6550 50  0001 C CNN
-F 3 "" H 1200 6550 50  0001 C CNN
-	1    1200 6550
-	1    0    0    -1
-$EndComp
-$Comp
-L Sesame:AD8030 U?
-U 3 1 6161C7FC
-P 1150 6950
-AR Path="/60F1AF26/6161C7FC" Ref="U?"  Part="3"
-AR Path="/60F1B237/6161C7FC" Ref="U?"  Part="3"
-AR Path="/60F16FAE/6161C7FC" Ref="U?"  Part="3"
-AR Path="/60F171CE/6161C7FC" Ref="U?"  Part="3"
-AR Path="/60F19D5B/6161C7FC" Ref="U?"  Part="3"
-AR Path="/60F1AA92/6161C7FC" Ref="U14"  Part="3"
-F 0 "U14" H 963 6904 50  0000 R CNN
-F 1 "AD8030" H 963 6995 50  0000 R CNN
-F 2 "Package_SO:SO-8_5.3x6.2mm_P1.27mm" H 1150 6950 50  0001 C CNN
-F 3 "~" H 1150 6950 50  0001 C CNN
-	3    1150 6950
-	1    0    0    -1
-$EndComp
 $Comp
 L Connector:TestPoint TP?
@@
 Text Notes 4500 1950 0    100  ~ 20
 BOBINE !!!\nCondo serie
-Text Notes 8600 2300 0    100  ~ 20
-REF TENSION AUTRE SOLUTION\n
 $Comp
 L Device:CP C32
@@
 	5400 2650 5300 2650
 $Comp
-L Reference_Voltage:TL431DBZ U?
+L Reference_Voltage:TL431DBZ U16
 U 1 1 6135BA5E
-P 10500 3500
-F 0 "U?" H 10500 3385 50  0000 C CNN
-F 1 "TL431DBZ" H 10500 3294 50  0000 C CNN
-F 2 "Package_TO_SOT_SMD:SOT-23" H 10500 3350 50  0001 C CIN
-F 3 "http://www.ti.com/lit/ds/symlink/tl431.pdf" H 10500 3500 50  0001 C CIN
-	1    10500 3500
+P 9500 3500
+F 0 "U16" H 9500 3385 50  0000 C CNN
+F 1 "TL431DBZ" H 9500 3294 50  0000 C CNN
+F 2 "Package_TO_SOT_SMD:SOT-23" H 9500 3350 50  0001 C CIN
+F 3 "http://www.ti.com/lit/ds/symlink/tl431.pdf" H 9500 3500 50  0001 C CIN
+	1    9500 3500
 	0    -1   -1   0
 $EndComp
 Wire Wire Line
-	10500 2900 10500 3000
-Wire Wire Line
-	10500 3600 10500 3750
-$Comp
-L Device:R R?
+	9500 2900 9500 3000
+Wire Wire Line
+	9500 3600 9500 4000
+$Comp
+L Device:R R84
 U 1 1 61378003
-P 10000 3750
-F 0 "R?" H 10070 3796 50  0000 L CNN
-F 1 "R" H 10070 3705 50  0000 L CNN
-F 2 "Sesame_footprint:R_0805_2012Metric_Pad1.20x1.40mm_HandSolder" V 9930 3750 50  0001 C CNN
-F 3 "~" H 10000 3750 50  0001 C CNN
-	1    10000 3750
-	1    0    0    -1
-$EndComp
-$Comp
-L Device:R R?
+P 9000 3750
+F 0 "R84" H 9070 3796 50  0000 L CNN
+F 1 "R" H 9070 3705 50  0000 L CNN
+F 2 "Sesame_footprint:R_0805_2012Metric_Pad1.20x1.40mm_HandSolder" V 8930 3750 50  0001 C CNN
+F 3 "~" H 9000 3750 50  0001 C CNN
+	1    9000 3750
+	1    0    0    -1
+$EndComp
+$Comp
+L Device:R R28
 U 1 1 61379D1A
-P 10000 3250
-F 0 "R?" H 10070 3296 50  0000 L CNN
-F 1 "R" H 10070 3205 50  0000 L CNN
-F 2 "Sesame_footprint:R_0805_2012Metric_Pad1.20x1.40mm_HandSolder" V 9930 3250 50  0001 C CNN
-F 3 "~" H 10000 3250 50  0001 C CNN
-	1    10000 3250
-	1    0    0    -1
-$EndComp
-Wire Wire Line
-	10000 3600 10000 3500
-Wire Wire Line
-	10000 3500 10400 3500
-Connection ~ 10000 3500
-Wire Wire Line
-	10000 3500 10000 3400
+P 9000 3250
+F 0 "R28" H 9070 3296 50  0000 L CNN
+F 1 "R" H 9070 3205 50  0000 L CNN
+F 2 "Sesame_footprint:R_0805_2012Metric_Pad1.20x1.40mm_HandSolder" V 8930 3250 50  0001 C CNN
+F 3 "~" H 9000 3250 50  0001 C CNN
+	1    9000 3250
+	1    0    0    -1
+$EndComp
+Wire Wire Line
+	9000 3600 9000 3500
+Wire Wire Line
+	9000 3500 9400 3500
+Connection ~ 9000 3500
+Wire Wire Line
+	9000 3500 9000 3400
+$Comp
+L power:GND #PWR0112
+U 1 1 61384F17
+P 9000 4000
+F 0 "#PWR0112" H 9000 3750 50  0001 C CNN
+F 1 "GND" H 9005 3827 50  0000 C CNN
+F 2 "" H 9000 4000 50  0001 C CNN
+F 3 "" H 9000 4000 50  0001 C CNN
+	1    9000 4000
+	1    0    0    -1
+$EndComp
+Wire Wire Line
+	9000 4000 9000 3900
+Wire Wire Line
+	9000 3100 9000 3000
+Wire Wire Line
+	9000 3000 9500 3000
+Connection ~ 9500 3000
+Wire Wire Line
+	9500 3000 9500 3400
+$Comp
+L Sesame:VREF #PWR0115
+U 1 1 61391751
+P 9900 2900
+F 0 "#PWR0115" H 9900 2750 50  0001 C CNN
+F 1 "VREF" H 9915 3073 50  0000 C CNN
+F 2 "" H 9900 2900 50  0001 C CNN
+F 3 "" H 9900 2900 50  0001 C CNN
+	1    9900 2900
+	1    0    0    -1
+$EndComp
+Wire Wire Line
+	9900 2900 9900 3000
+$Comp
+L power:PWR_FLAG #FLG0101
+U 1 1 61398926
+P 10250 2900
+F 0 "#FLG0101" H 10250 2975 50  0001 C CNN
+F 1 "PWR_FLAG" H 10250 3073 50  0000 C CNN
+F 2 "" H 10250 2900 50  0001 C CNN
+F 3 "~" H 10250 2900 50  0001 C CNN
+	1    10250 2900
+	1    0    0    -1
+$EndComp
+Wire Wire Line
+	10250 2900 10250 3000
+Wire Wire Line
+	9500 3000 9900 3000
+Connection ~ 9900 3000
+Wire Wire Line
+	9900 3000 10250 3000
+$Comp
+L Device:C C?
+U 1 1 6161C7DE
+P 9900 3500
+AR Path="/60F1AF26/6161C7DE" Ref="C?"  Part="1"
+AR Path="/60F1B237/6161C7DE" Ref="C?"  Part="1"
+AR Path="/60F16FAE/6161C7DE" Ref="C?"  Part="1"
+AR Path="/60F171CE/6161C7DE" Ref="C?"  Part="1"
+AR Path="/60F19D5B/6161C7DE" Ref="C?"  Part="1"
+AR Path="/60F1AA92/6161C7DE" Ref="C27"  Part="1"
+F 0 "C27" H 10015 3546 50  0000 L CNN
+F 1 "100n" H 10015 3455 50  0000 L CNN
+F 2 "Sesame_footprint:C_0805_2012Metric_Pad1.18x1.45mm_HandSolder" H 9938 3350 50  0001 C CNN
+F 3 "~" H 9900 3500 50  0001 C CNN
+	1    9900 3500
+	1    0    0    -1
+$EndComp
 $Comp
 L power:GND #PWR?
-U 1 1 61384F17
-P 10000 4000
-F 0 "#PWR?" H 10000 3750 50  0001 C CNN
-F 1 "GND" H 10005 3827 50  0000 C CNN
-F 2 "" H 10000 4000 50  0001 C CNN
-F 3 "" H 10000 4000 50  0001 C CNN
-	1    10000 4000
-	1    0    0    -1
-$EndComp
-Wire Wire Line
-	10000 4000 10000 3900
-Wire Wire Line
-	10000 3100 10000 3000
-Wire Wire Line
-	10000 3000 10500 3000
-Connection ~ 10500 3000
-Wire Wire Line
-	10500 3000 10500 3400
-$Comp
-L Sesame:VREF #PWR?
-U 1 1 61391751
-P 10000 2900
-F 0 "#PWR?" H 10000 2750 50  0001 C CNN
-F 1 "VREF" H 10015 3073 50  0000 C CNN
-F 2 "" H 10000 2900 50  0001 C CNN
-F 3 "" H 10000 2900 50  0001 C CNN
-	1    10000 2900
-	1    0    0    -1
-$EndComp
-Wire Wire Line
-	10000 2900 10000 3000
-Connection ~ 10000 3000
+U 1 1 613C7BA8
+P 9900 4000
+F 0 "#PWR?" H 9900 3750 50  0001 C CNN
+F 1 "GND" H 9905 3827 50  0000 C CNN
+F 2 "" H 9900 4000 50  0001 C CNN
+F 3 "" H 9900 4000 50  0001 C CNN
+	1    9900 4000
+	1    0    0    -1
+$EndComp
+Wire Wire Line
+	9900 3650 9900 4000
+Wire Wire Line
+	9900 3350 9900 3000
 $EndSCHEMATC

Commit message: mod. ref rail on kicad
Parts:
- R28: value R -> 14k
- R83: value R -> 200
- R84: value R -> 10k
Other:
- note removed: "BOBINE !!!\nCondo serie"
Changed lines of the file:
@@
 P 9500 2750
 F 0 "R83" H 9570 2796 50  0000 L CNN
-F 1 "R" H 9570 2705 50  0000 L CNN
+F 1 "200" H 9570 2705 50  0000 L CNN
 F 2 "Sesame_footprint:R_0805_2012Metric_Pad1.20x1.40mm_HandSolder" V 9430 2750 50  0001 C CNN
 F 3 "~" H 9500 2750 50  0001 C CNN
@@
 $EndComp
 Connection ~ 7200 2650
-Text Notes 2550 1350 0    100  ~ 0
+Text Notes 650  900  0    100  ~ 0
 VCC = 7V\nVREF = 6V
 $Comp
@@
 Wire Wire Line
 	3350 2650 2950 2650
-Text Notes 4500 1950 0    100  ~ 20
-BOBINE !!!\nCondo serie
 $Comp
 L Device:CP C32
@@
 P 9000 3750
 F 0 "R84" H 9070 3796 50  0000 L CNN
-F 1 "R" H 9070 3705 50  0000 L CNN
+F 1 "10k" H 9070 3705 50  0000 L CNN
 F 2 "Sesame_footprint:R_0805_2012Metric_Pad1.20x1.40mm_HandSolder" V 8930 3750 50  0001 C CNN
 F 3 "~" H 9000 3750 50  0001 C CNN
@@
 P 9000 3250
 F 0 "R28" H 9070 3296 50  0000 L CNN
-F 1 "R" H 9070 3205 50  0000 L CNN
+F 1 "14k" H 9070 3205 50  0000 L CNN
 F 2 "Sesame_footprint:R_0805_2012Metric_Pad1.20x1.40mm_HandSolder" V 8930 3250 50  0001 C CNN
 F 3 "~" H 9000 3250 50  0001 C CNN

Commit message: lil cleanup on the main schematic sheet
Parts:
- C27, C28, C29, C30, C31: symbol Device:C -> sesame-fonctionnel-rescue:C-Device
- C32: symbol Device:CP -> sesame-fonctionnel-rescue:CP-Device
- D12, D13, D14: symbol Device:D_Schottky -> sesame-fonctionnel-rescue:D_Schottky-Device
- R28, R79, R80, R81, R82, R83, R84: symbol Device:R -> sesame-fonctionnel-rescue:R-Device
- TP39, TP40, TP41, TP42: symbol Connector:TestPoint -> sesame-fonctionnel-rescue:TestPoint-Connector
- U16: symbol Reference_Voltage:TL431DBZ -> sesame-fonctionnel-rescue:TL431DBZ-Reference_Voltage
Changed lines of the file:
@@
 $Descr A4 11693 8268
 encoding utf-8
-Sheet 14 17
+Sheet 11 17
 Title "SESAME"
 Date ""
@@
 RIGHT
 $Comp
-L power:GND #PWR0114
+L sesame-fonctionnel-rescue:GND-power #PWR0114
 U 1 1 612FEB08
 P 9500 4000
@@
 	2500 2500 2650 2500
 $Comp
-L Device:R R83
+L sesame-fonctionnel-rescue:R-Device R83
 U 1 1 61087C02
 P 9500 2750
@@
 $EndComp
 $Comp
-L power:VCC #PWR0113
+L sesame-fonctionnel-rescue:VCC-power #PWR0113
 U 1 1 6158EF67
 P 9500 2500
@@
 Connection ~ 4550 2650
 $Comp
-L Device:C C30
+L sesame-fonctionnel-rescue:C-Device C30
 U 1 1 61244F9E
 P 5700 2650
@@
 Connection ~ 5150 2650
 $Comp
-L Device:R R80
+L sesame-fonctionnel-rescue:R-Device R80
 U 1 1 61246D21
 P 5250 4350
@@
 	6550 3100 6550 3050
 $Comp
-L power:GND #PWR0109
+L sesame-fonctionnel-rescue:GND-power #PWR0109
 U 1 1 61259762
 P 6550 3100
@@
 	6550 2750 6550 2650
 $Comp
-L power:GND #PWR0108
+L sesame-fonctionnel-rescue:GND-power #PWR0108
 U 1 1 61253B2C
 P 6050 3100
@@
 	6050 2700 6050 2650
 $Comp
-L Device:D_Schottky D14
+L sesame-fonctionnel-rescue:D_Schottky-Device D14
 U 1 1 6124B9FF
 P 6300 2650
@@
 	7200 3200 7200 3450
 $Comp
-L Device:R R81
+L sesame-fonctionnel-rescue:R-Device R81
 U 1 1 612476CB
 P 7200 3050
@@
 	7200 3450 7200 3700
 $Comp
-L Device:R R82
+L sesame-fonctionnel-rescue:R-Device R82
 U 1 1 61247B73
 P 7200 3850
@@
 $EndComp
 $Comp
-L power:GND #PWR0110
+L sesame-fonctionnel-rescue:GND-power #PWR0110
 U 1 1 61249817
 P 7200 4150
@@
 	7200 4150 7200 4000
 $Comp
-L power:GND #PWR0105
+L sesame-fonctionnel-rescue:GND-power #PWR0105
 U 1 1 6127CD6C
 P 4850 4850
@@
 $EndComp
 $Comp
-L Device:C C29
+L sesame-fonctionnel-rescue:C-Device C29
 U 1 1 6127EBD7
 P 5250 4650
@@
 $EndComp
 $Comp
-L power:GND #PWR0106
+L sesame-fonctionnel-rescue:GND-power #PWR0106
 U 1 1 6127FC82
 P 5250 4850
@@
 $EndComp
 $Comp
-L power:GND #PWR0104
+L sesame-fonctionnel-rescue:GND-power #PWR0104
 U 1 1 612803A6
 P 4450 4850
@@
 	5250 4200 5250 4150
 $Comp
-L Device:R R79
+L sesame-fonctionnel-rescue:R-Device R79
 U 1 1 61283A99
 P 4050 4500
@@
 	4050 3750 4200 3750
 $Comp
-L Device:C C28
+L sesame-fonctionnel-rescue:C-Device C28
 U 1 1 61286334
 P 4450 4500
@@
 $EndComp
 $Comp
-L power:GND #PWR0103
+L sesame-fonctionnel-rescue:GND-power #PWR0103
 U 1 1 612874BD
 P 4050 4850
@@
 	5250 4850 5250 4800
 $Comp
-L power:GND #PWR0102
+L sesame-fonctionnel-rescue:GND-power #PWR0102
 U 1 1 612945AE
 P 3700 4850
@@
 	3700 3450 3700 4850
 $Comp
-L Device:C C31
+L sesame-fonctionnel-rescue:C-Device C31
 U 1 1 6129A654
 P 5750 4500
@@
 	5750 3750 5500 3750
 $Comp
-L power:GND #PWR0107
+L sesame-fonctionnel-rescue:GND-power #PWR0107
 U 1 1 6129CD8D
 P 5750 4850
@@
 VIN
 $Comp
-L Device:D_Schottky D12
+L sesame-fonctionnel-rescue:D_Schottky-Device D12
 U 1 1 612B6943
 P 2350 2500
@@
 $EndComp
 $Comp
-L Device:D_Schottky D13
+L sesame-fonctionnel-rescue:D_Schottky-Device D13
 U 1 1 612B7084
 P 2350 2850
@@
 RT = 432k  -> 100 kHz\nRT = 143k  -> 300 kHz\nRT = 84.5k -> 500 kHz
 $Comp
-L power:VCC #PWR0111
+L sesame-fonctionnel-rescue:VCC-power #PWR0111
 U 1 1 612BD8C1
 P 7750 2550
@@
 VCC = 7V\nVREF = 6V
 $Comp
-L Connector:TestPoint TP?
+L sesame-fonctionnel-rescue:TestPoint-Connector TP?
 U 1 1 61513B8D
 P 2950 2650
@@
 	2950 2650 2650 2650
 $Comp
-L Connector:TestPoint TP?
+L sesame-fonctionnel-rescue:TestPoint-Connector TP?
 U 1 1 61522F2C
 P 7400 2650
@@
 Connection ~ 7400 2650
 $Comp
-L Connector:TestPoint TP?
+L sesame-fonctionnel-rescue:TestPoint-Connector TP?
 U 1 1 61530DA6
 P 5400 2600
@@
 $EndComp
 $Comp
-L Connector:TestPoint TP?
+L sesame-fonctionnel-rescue:TestPoint-Connector TP?
 U 1 1 61533C44
 P 6050 2650
@@
 $EndComp
 $Comp
-L power:PWR_FLAG #FLG03
+L sesame-fonctionnel-rescue:PWR_FLAG-power #FLG03
 U 1 1 61B4926B
 P 8100 2550
@@
 Connection ~ 7750 2650
 $Comp
-L power:PWR_FLAG #FLG02
+L sesame-fonctionnel-rescue:PWR_FLAG-power #FLG02
 U 1 1 61B527B2
 P 3350 2550
@@
 	3350 2650 2950 2650
 $Comp
-L Device:CP C32
+L sesame-fonctionnel-rescue:CP-Device C32
 U 1 1 6126F44E
 P 6550 2900
@@
 	5400 2650 5300 2650
 $Comp
-L Reference_Voltage:TL431DBZ U16
+L sesame-fonctionnel-rescue:TL431DBZ-Reference_Voltage U16
 U 1 1 6135BA5E
 P 9500 3500
@@
 	9500 3600 9500 4000
 $Comp
-L Device:R R84
+L sesame-fonctionnel-rescue:R-Device R84
 U 1 1 61378003
 P 9000 3750
@@
 $EndComp
 $Comp
-L Device:R R28
+L sesame-fonctionnel-rescue:R-Device R28
 U 1 1 61379D1A
 P 9000 3250
@@
 	9000 3500 9000 3400
 $Comp
-L power:GND #PWR0112
+L sesame-fonctionnel-rescue:GND-power #PWR0112
 U 1 1 61384F17
 P 9000 4000
@@
 	9900 2900 9900 3000
 $Comp
-L power:PWR_FLAG #FLG0101
+L sesame-fonctionnel-rescue:PWR_FLAG-power #FLG0101
 U 1 1 61398926
 P 10250 2900
@@
 	9900 3000 10250 3000
 $Comp
-L Device:C C?
+L sesame-fonctionnel-rescue:C-Device C?
 U 1 1 6161C7DE
 P 9900 3500
@@
 $EndComp
 $Comp
-L power:GND #PWR0101
+L sesame-fonctionnel-rescue:GND-power #PWR0101
 U 1 1 613C7BA8
 P 9900 4000
