File: KICAD/voltage_current_sens.sch (KiCad schematic (older format))
At the start: 17 parts, among them U10 LT6016, U11 AD8030

Commit message: review w/ jmt
Parts:
- R48, R49, R50, R59, R60, R61, R62: renamed from R?; footprint Resistor_SMD:R_0805_2012Metric_Pad1.15x1.40mm_HandSolder -> (none)
- RShunt2: footprint Resistor_SMD:R_2512_6332Metric_Pad1.40x3.35mm_HandSolder -> (none)
- U8: renamed from U10; footprint Package_SO:MSOP-8_3x3mm_P0.65mm -> (none)
- U9: renamed from U11; footprint Package_SO:SO-8_3.9x4.9mm_P1.27mm -> (none)
- gave numbers to parts that had none: 7

Commit message: edit footprints by jmt
Parts:
- C19, C20: footprint (none) -> Capacitor_SMD:C_0805_2012Metric_Pad1.15x1.40mm_HandSolder
- R48, R49, R50, R59, R60, R61, R62: footprint (none) -> Resistor_SMD:R_0805_2012Metric_Pad1.15x1.40mm_HandSolder
- RShunt2: footprint (none) -> Resistor_SMD:R_2512_6332Metric_Pad1.52x3.35mm_HandSolder
- TP20, TP21, TP22: footprint (none) -> TestPoint:TestPoint_Loop_D1.80mm_Drill1.0mm_Beaded
- U8: footprint (none) -> Package_SO:MSOP-8_3x3mm_P0.65mm
- U9: footprint (none) -> Package_SO:SO-8_5.3x6.2mm_P1.27mm
Changed lines of the file:
@@
 F 0 "RShunt2" V 2143 2600 50  0000 C CNN
 F 1 "PA2512FKF070R005E" V 2234 2600 50  0000 C CNN
-F 2 "" V 2280 2600 50  0001 C CNN
+F 2 "Resistor_SMD:R_2512_6332Metric_Pad1.52x3.35mm_HandSolder" V 2280 2600 50  0001 C CNN
 F 3 "~" H 2350 2600 50  0001 C CNN
 	1    2350 2600
@@
 F 0 "R60" V 3000 3650 50  0000 C CNN
 F 1 "200" V 3100 3650 50  0000 C CNN
-F 2 "" V 2830 3650 50  0001 C CNN
+F 2 "Resistor_SMD:R_0805_2012Metric_Pad1.15x1.40mm_HandSolder" V 2830 3650 50  0001 C CNN
 F 3 "~" H 2900 3650 50  0001 C CNN
 	1    2900 3650
@@
 F 0 "R59" V 2693 3450 50  0000 C CNN
 F 1 "200" V 2784 3450 50  0000 C CNN
-F 2 "" V 2830 3450 50  0001 C CNN
+F 2 "Resistor_SMD:R_0805_2012Metric_Pad1.15x1.40mm_HandSolder" V 2830 3450 50  0001 C CNN
 F 3 "~" H 2900 3450 50  0001 C CNN
 	1    2900 3450
@@
 F 0 "R65" H 7720 3746 50  0000 L CNN
 F 1 "10k" H 7720 3655 50  0000 L CNN
-F 2 "" V 7580 3700 50  0001 C CNN
+F 2 "Resistor_SMD:R_0805_2012Metric_Pad1.15x1.40mm_HandSolder" V 7580 3700 50  0001 C CNN
 F 3 "~" H 7650 3700 50  0001 C CNN
 	1    7650 3700
@@
 F 0 "R64" H 7720 3046 50  0000 L CNN
 F 1 "90k" H 7720 2955 50  0000 L CNN
-F 2 "" V 7580 3000 50  0001 C CNN
+F 2 "Resistor_SMD:R_0805_2012Metric_Pad1.15x1.40mm_HandSolder" V 7580 3000 50  0001 C CNN
 F 3 "~" H 7650 3000 50  0001 C CNN
 	1    7650 3000
@@
 F 0 "R63" H 4120 5146 50  0000 L CNN
 F 1 "20k" H 4120 5055 50  0000 L CNN
-F 2 "" V 3980 5100 50  0001 C CNN
+F 2 "Resistor_SMD:R_0805_2012Metric_Pad1.15x1.40mm_HandSolder" V 3980 5100 50  0001 C CNN
 F 3 "~" H 4050 5100 50  0001 C CNN
 	1    4050 5100
@@
 F 0 "R61" V 2693 4550 50  0000 C CNN
 F 1 "200" V 2784 4550 50  0000 C CNN
-F 2 "" V 2830 4550 50  0001 C CNN
+F 2 "Resistor_SMD:R_0805_2012Metric_Pad1.15x1.40mm_HandSolder" V 2830 4550 50  0001 C CNN
 F 3 "~" H 2900 4550 50  0001 C CNN
 	1    2900 4550
@@
 F 0 "R62" V 3000 4750 50  0000 C CNN
 F 1 "200" V 3100 4750 50  0000 C CNN
-F 2 "" V 2830 4750 50  0001 C CNN
+F 2 "Resistor_SMD:R_0805_2012Metric_Pad1.15x1.40mm_HandSolder" V 2830 4750 50  0001 C CNN
 F 3 "~" H 2900 4750 50  0001 C CNN
 	1    2900 4750
@@
 F 0 "U11" H 8350 2800 50  0000 C CNN
 F 1 "AD8030" H 8350 2900 50  0000 C CNN
-F 2 "" H 8350 3250 50  0001 C CNN
+F 2 "Package_SO:SO-8_5.3x6.2mm_P1.27mm" H 8350 3250 50  0001 C CNN
 F 3 "~" H 8350 3250 50  0001 C CNN
 	2    8350 3250
@@
 F 0 "U11" H 5350 3400 50  0000 C CNN
 F 1 "AD8030" H 5350 3500 50  0000 C CNN
-F 2 "" H 5350 3850 50  0001 C CNN
+F 2 "Package_SO:SO-8_5.3x6.2mm_P1.27mm" H 5350 3850 50  0001 C CNN
 F 3 "~" H 5350 3850 50  0001 C CNN
 	1    5350 3850
@@
 F 0 "C21" H 1365 6996 50  0000 L CNN
 F 1 "100n" H 1365 6905 50  0000 L CNN
-F 2 "" H 1288 6800 50  0001 C CNN
+F 2 "Capacitor_SMD:C_0805_2012Metric_Pad1.15x1.40mm_HandSolder" H 1288 6800 50  0001 C CNN
 F 3 "~" H 1250 6950 50  0001 C CNN
 	1    1250 6950
@@
 F 0 "C22" H 2565 6946 50  0000 L CNN
 F 1 "100n" H 2565 6855 50  0000 L CNN
-F 2 "" H 2488 6750 50  0001 C CNN
+F 2 "Capacitor_SMD:C_0805_2012Metric_Pad1.15x1.40mm_HandSolder" H 2488 6750 50  0001 C CNN
 F 3 "~" H 2450 6900 50  0001 C CNN
 	1    2450 6900
@@
 F 0 "U11" H 2050 6850 50  0000 R CNN
 F 1 "AD8030" H 2063 6945 50  0000 R CNN
-F 2 "" H 2250 6900 50  0001 C CNN
+F 2 "Package_SO:SO-8_5.3x6.2mm_P1.27mm" H 2250 6900 50  0001 C CNN
 F 3 "~" H 2250 6900 50  0001 C CNN
 	3    2250 6900
@@
 F 0 "U10" H 3450 3917 50  0000 C CNN
 F 1 "LT6016" H 3450 3826 50  0000 C CNN
-F 2 "" H 3450 3550 50  0001 C CNN
+F 2 "Package_SO:MSOP-8_3x3mm_P0.65mm" H 3450 3550 50  0001 C CNN
 F 3 "~" H 3450 3550 50  0001 C CNN
 	1    3450 3550
@@
 F 0 "U10" H 3450 5017 50  0000 C CNN
 F 1 "LT6016" H 3450 4926 50  0000 C CNN
-F 2 "" H 3450 4650 50  0001 C CNN
+F 2 "Package_SO:MSOP-8_3x3mm_P0.65mm" H 3450 4650 50  0001 C CNN
 F 3 "~" H 3450 4650 50  0001 C CNN
 	2    3450 4650
@@
 F 0 "U10" H 650 6900 50  0000 L CNN
 F 1 "LT6016" H 600 7000 50  0000 L CNN
-F 2 "" H 1050 6950 50  0001 C CNN
+F 2 "Package_SO:MSOP-8_3x3mm_P0.65mm" H 1050 6950 50  0001 C CNN
 F 3 "~" H 1050 6950 50  0001 C CNN
 	3    1050 6950
@@
 F 0 "TP29" H 4550 4300 50  0000 L CNN
 F 1 "TP_POP" H 4600 4200 50  0000 C CNN
-F 2 "" H 4800 3950 50  0001 C CNN
+F 2 "TestPoint:TestPoint_Loop_D1.80mm_Drill1.0mm_Beaded" H 4800 3950 50  0001 C CNN
 F 3 "~" H 4800 3950 50  0001 C CNN
 	1    4600 3950
@@
 F 0 "TP31" H 9050 3600 50  0000 L CNN
 F 1 "TP_POP" H 9100 3500 50  0000 C CNN
-F 2 "" H 9300 3250 50  0001 C CNN
+F 2 "TestPoint:TestPoint_Loop_D1.80mm_Drill1.0mm_Beaded" H 9300 3250 50  0001 C CNN
 F 3 "~" H 9300 3250 50  0001 C CNN
 	1    9100 3250
@@
 F 0 "TP30" H 5850 4200 50  0000 L CNN
 F 1 "TP_POP" H 5900 4100 50  0000 C CNN
-F 2 "" H 6100 3850 50  0001 C CNN
+F 2 "TestPoint:TestPoint_Loop_D1.80mm_Drill1.0mm_Beaded" H 6100 3850 50  0001 C CNN
 F 3 "~" H 6100 3850 50  0001 C CNN
 	1    5900 3850

Commit message: route + work on djd
Connections:
- net VD_Mos: now also R59.2, R62.2, RShunt2.2; no longer R49.1, R60.2, R61.2, RShunt2.1
- net VProt: now also R49.1, R60.2, R61.2, RShunt2.1; no longer R59.2, R62.2, RShunt2.2
Changed lines of the file:
@@
 Comment4 ""
 $EndDescr
-Text HLabel 1700 2600 0    100  BiDi ~ 0
-VProt
 Wire Wire Line
 	2200 2600 2150 2600
@@
 AR Path="/60F19D5B/6109114F" Ref="RShunt2"  Part="1"
 AR Path="/60F171CE/6109114F" Ref="RShunt1"  Part="1"
-F 0 "RShunt2" V 2143 2600 50  0000 C CNN
+F 0 "RShunt1" V 2143 2600 50  0000 C CNN
 F 1 "PA2512FKF070R005E" V 2234 2600 50  0000 C CNN
 F 2 "Resistor_SMD:R_2512_6332Metric_Pad1.52x3.35mm_HandSolder" V 2280 2600 50  0001 C CNN
@@
 AR Path="/60F19D5B/61091B7C" Ref="R60"  Part="1"
 AR Path="/60F171CE/61091B7C" Ref="R45"  Part="1"
-F 0 "R60" V 3000 3650 50  0000 C CNN
+F 0 "R45" V 3000 3650 50  0000 C CNN
 F 1 "200" V 3100 3650 50  0000 C CNN
 F 2 "Resistor_SMD:R_0805_2012Metric_Pad1.15x1.40mm_HandSolder" V 2830 3650 50  0001 C CNN
@@
 AR Path="/60F19D5B/610923D6" Ref="R59"  Part="1"
 AR Path="/60F171CE/610923D6" Ref="R44"  Part="1"
-F 0 "R59" V 2693 3450 50  0000 C CNN
+F 0 "R44" V 2693 3450 50  0000 C CNN
 F 1 "200" V 2784 3450 50  0000 C CNN
 F 2 "Resistor_SMD:R_0805_2012Metric_Pad1.15x1.40mm_HandSolder" V 2830 3450 50  0001 C CNN
@@
 AR Path="/60F171CE/610DC636" Ref="R50"  Part="1"
 AR Path="/60F19D5B/610DC636" Ref="R65"  Part="1"
-F 0 "R65" H 7720 3746 50  0000 L CNN
+F 0 "R50" H 7720 3746 50  0000 L CNN
 F 1 "10k" H 7720 3655 50  0000 L CNN
 F 2 "Resistor_SMD:R_0805_2012Metric_Pad1.15x1.40mm_HandSolder" V 7580 3700 50  0001 C CNN
@@
 AR Path="/60F171CE/610DBB97" Ref="R49"  Part="1"
 AR Path="/60F19D5B/610DBB97" Ref="R64"  Part="1"
-F 0 "R64" H 7720 3046 50  0000 L CNN
+F 0 "R49" H 7720 3046 50  0000 L CNN
 F 1 "90k" H 7720 2955 50  0000 L CNN
 F 2 "Resistor_SMD:R_0805_2012Metric_Pad1.15x1.40mm_HandSolder" V 7580 3000 50  0001 C CNN
@@
 Text HLabel 9400 3250 2    50   Output ~ 0
 Voltage_Sens
-Text HLabel 9000 2600 2    100  BiDi ~ 0
+Text HLabel 1700 2600 0    100  BiDi ~ 0
 VD_Mos
 Connection ~ 7650 2600
@@
 AR Path="/60F171CE/61382079" Ref="Q4"  Part="1"
 AR Path="/60F19D5B/61382079" Ref="Q12"  Part="1"
-F 0 "Q12" H 4141 3596 50  0000 L CNN
+F 0 "Q4" H 4141 3596 50  0000 L CNN
 F 1 "BC847" H 4141 3505 50  0000 L CNN
 F 2 "Package_TO_SOT_SMD:SOT-23" H 4150 3475 50  0001 L CIN
@@
 AR Path="/60F171CE/613844DA" Ref="Q5"  Part="1"
 AR Path="/60F19D5B/613844DA" Ref="Q13"  Part="1"
-F 0 "Q13" H 4141 4696 50  0000 L CNN
+F 0 "Q5" H 4141 4696 50  0000 L CNN
 F 1 "BC847" H 4141 4605 50  0000 L CNN
 F 2 "Package_TO_SOT_SMD:SOT-23" H 4150 4575 50  0001 L CIN
@@
 AR Path="/60F171CE/6138CEF9" Ref="R48"  Part="1"
 AR Path="/60F19D5B/6138CEF9" Ref="R63"  Part="1"
-F 0 "R63" H 4120 5146 50  0000 L CNN
+F 0 "R48" H 4120 5146 50  0000 L CNN
 F 1 "20k" H 4120 5055 50  0000 L CNN
 F 2 "Resistor_SMD:R_0805_2012Metric_Pad1.15x1.40mm_HandSolder" V 3980 5100 50  0001 C CNN
@@
 AR Path="/60F19D5B/61397C3C" Ref="R61"  Part="1"
 AR Path="/60F171CE/61397C3C" Ref="R46"  Part="1"
-F 0 "R61" V 2693 4550 50  0000 C CNN
+F 0 "R46" V 2693 4550 50  0000 C CNN
 F 1 "200" V 2784 4550 50  0000 C CNN
 F 2 "Resistor_SMD:R_0805_2012Metric_Pad1.15x1.40mm_HandSolder" V 2830 4550 50  0001 C CNN
@@
 AR Path="/60F19D5B/61398F33" Ref="R62"  Part="1"
 AR Path="/60F171CE/61398F33" Ref="R47"  Part="1"
-F 0 "R62" V 3000 4750 50  0000 C CNN
+F 0 "R47" V 3000 4750 50  0000 C CNN
 F 1 "200" V 3100 4750 50  0000 C CNN
 F 2 "Resistor_SMD:R_0805_2012Metric_Pad1.15x1.40mm_HandSolder" V 2830 4750 50  0001 C CNN
@@
 AR Path="/60F171CE/6139E98B" Ref="U9"  Part="2"
 AR Path="/60F19D5B/6139E98B" Ref="U11"  Part="2"
-F 0 "U11" H 8350 2800 50  0000 C CNN
+F 0 "U9" H 8350 2800 50  0000 C CNN
 F 1 "AD8030" H 8350 2900 50  0000 C CNN
 F 2 "Package_SO:SO-8_5.3x6.2mm_P1.27mm" H 8350 3250 50  0001 C CNN
@@
 AR Path="/60F171CE/613A5251" Ref="U9"  Part="1"
 AR Path="/60F19D5B/613A5251" Ref="U11"  Part="1"
-F 0 "U11" H 5350 3400 50  0000 C CNN
+F 0 "U9" H 5350 3400 50  0000 C CNN
 F 1 "AD8030" H 5350 3500 50  0000 C CNN
 F 2 "Package_SO:SO-8_5.3x6.2mm_P1.27mm" H 5350 3850 50  0001 C CNN
@@
 AR Path="/60F171CE/613B4715" Ref="C19"  Part="1"
 AR Path="/60F19D5B/613B4715" Ref="C21"  Part="1"
-F 0 "C21" H 1365 6996 50  0000 L CNN
+F 0 "C19" H 1365 6996 50  0000 L CNN
 F 1 "100n" H 1365 6905 50  0000 L CNN
 F 2 "Capacitor_SMD:C_0805_2012Metric_Pad1.15x1.40mm_HandSolder" H 1288 6800 50  0001 C CNN
@@
 AR Path="/60F171CE/613B7585" Ref="C20"  Part="1"
 AR Path="/60F19D5B/613B7585" Ref="C22"  Part="1"
-F 0 "C22" H 2565 6946 50  0000 L CNN
+F 0 "C20" H 2565 6946 50  0000 L CNN
 F 1 "100n" H 2565 6855 50  0000 L CNN
 F 2 "Capacitor_SMD:C_0805_2012Metric_Pad1.15x1.40mm_HandSolder" H 2488 6750 50  0001 C CNN
@@
 AR Path="/60F171CE/613B75A3" Ref="U9"  Part="3"
 AR Path="/60F19D5B/613B75A3" Ref="U11"  Part="3"
-F 0 "U11" H 2050 6850 50  0000 R CNN
+F 0 "U9" H 2050 6850 50  0000 R CNN
 F 1 "AD8030" H 2063 6945 50  0000 R CNN
 F 2 "Package_SO:SO-8_5.3x6.2mm_P1.27mm" H 2250 6900 50  0001 C CNN
@@
 AR Path="/60F171CE/615B8C9F" Ref="U8"  Part="1"
 AR Path="/60F19D5B/615B8C9F" Ref="U10"  Part="1"
-F 0 "U10" H 3450 3917 50  0000 C CNN
+F 0 "U8" H 3450 3917 50  0000 C CNN
 F 1 "LT6016" H 3450 3826 50  0000 C CNN
 F 2 "Package_SO:MSOP-8_3x3mm_P0.65mm" H 3450 3550 50  0001 C CNN
@@
 AR Path="/60F171CE/615BC62A" Ref="U8"  Part="2"
 AR Path="/60F19D5B/615BC62A" Ref="U10"  Part="2"
-F 0 "U10" H 3450 5017 50  0000 C CNN
+F 0 "U8" H 3450 5017 50  0000 C CNN
 F 1 "LT6016" H 3450 4926 50  0000 C CNN
 F 2 "Package_SO:MSOP-8_3x3mm_P0.65mm" H 3450 4650 50  0001 C CNN
@@
 AR Path="/60F171CE/615BFCFC" Ref="U8"  Part="3"
 AR Path="/60F19D5B/615BFCFC" Ref="U10"  Part="3"
-F 0 "U10" H 650 6900 50  0000 L CNN
+F 0 "U8" H 650 6900 50  0000 L CNN
 F 1 "LT6016" H 600 7000 50  0000 L CNN
 F 2 "Package_SO:MSOP-8_3x3mm_P0.65mm" H 1050 6950 50  0001 C CNN
@@
 AR Path="/60F171CE/6153C862" Ref="TP20"  Part="1"
 AR Path="/60F19D5B/6153C862" Ref="TP29"  Part="1"
-F 0 "TP29" H 4550 4300 50  0000 L CNN
+F 0 "TP20" H 4550 4300 50  0000 L CNN
 F 1 "TP_POP" H 4600 4200 50  0000 C CNN
 F 2 "TestPoint:TestPoint_Loop_D1.80mm_Drill1.0mm_Beaded" H 4800 3950 50  0001 C CNN
@@
 AR Path="/60F171CE/61544B27" Ref="TP22"  Part="1"
 AR Path="/60F19D5B/61544B27" Ref="TP31"  Part="1"
-F 0 "TP31" H 9050 3600 50  0000 L CNN
+F 0 "TP22" H 9050 3600 50  0000 L CNN
 F 1 "TP_POP" H 9100 3500 50  0000 C CNN
 F 2 "TestPoint:TestPoint_Loop_D1.80mm_Drill1.0mm_Beaded" H 9300 3250 50  0001 C CNN
@@
 AR Path="/60F171CE/6154A16C" Ref="TP21"  Part="1"
 AR Path="/60F19D5B/6154A16C" Ref="TP30"  Part="1"
-F 0 "TP30" H 5850 4200 50  0000 L CNN
+F 0 "TP21" H 5850 4200 50  0000 L CNN
 F 1 "TP_POP" H 5900 4100 50  0000 C CNN
 F 2 "TestPoint:TestPoint_Loop_D1.80mm_Drill1.0mm_Beaded" H 6100 3850 50  0001 C CNN
@@
 Wire Wire Line
 	5900 3850 5700 3850
+Text HLabel 9000 2600 2    100  BiDi ~ 0
+VProt
 $EndSCHEMATC
