File: KICAD/voltage_current_sens.sch (KiCad schematic (older format))
At the start: 17 parts, among them Q4 BC847, Q5 BC847, U8 LT6016, U9 AD8030

Commit message: lil cleanup on the main schematic sheet
Parts:
- C19, C20: symbol Device:C -> sesame-fonctionnel-rescue:C-Device
- Q4, Q5: symbol Transistor_BJT:BC847 -> sesame-fonctionnel-rescue:BC847-Transistor_BJT
- R48, R49, R50, R59, R60, R61, R62, RShunt2: symbol Device:R -> sesame-fonctionnel-rescue:R-Device
- TP20, TP21, TP22: symbol Connector:TestPoint -> sesame-fonctionnel-rescue:TestPoint-Connector
Changed lines of the file:
@@
 	2150 2600 1700 2600
 $Comp
-L Device:R RShunt2
+L sesame-fonctionnel-rescue:R-Device RShunt2
 U 1 1 6109114F
 P 2350 2600
@@
 $EndComp
 $Comp
-L Device:R R60
+L sesame-fonctionnel-rescue:R-Device R60
 U 1 1 61091B7C
 P 2900 3650
@@
 $EndComp
 $Comp
-L Device:R R59
+L sesame-fonctionnel-rescue:R-Device R59
 U 1 1 610923D6
 P 2900 3450
@@
 	7650 3900 7650 3850
 $Comp
-L power:GND #PWR068
+L sesame-fonctionnel-rescue:GND-power #PWR068
 U 1 1 610DEA27
 P 7650 3900
@@
 	7650 2850 7650 2600
 $Comp
-L Device:R R50
+L sesame-fonctionnel-rescue:R-Device R50
 U 1 1 610DC636
 P 7650 3700
@@
 $EndComp
 $Comp
-L Device:R R49
+L sesame-fonctionnel-rescue:R-Device R49
 U 1 1 610DBB97
 P 7650 3000
@@
 	2550 3650 2550 4550
 $Comp
-L Transistor_BJT:BC847 Q4
+L sesame-fonctionnel-rescue:BC847-Transistor_BJT Q4
 U 1 1 61382079
 P 3950 3550
@@
 $EndComp
 $Comp
-L Transistor_BJT:BC847 Q5
+L sesame-fonctionnel-rescue:BC847-Transistor_BJT Q5
 U 1 1 613844DA
 P 3950 4650
@@
 	3100 4550 3150 4550
 $Comp
-L Device:R R48
+L sesame-fonctionnel-rescue:R-Device R48
 U 1 1 6138CEF9
 P 4050 5100
@@
 	4050 4900 4050 4950
 $Comp
-L power:GND #PWR067
+L sesame-fonctionnel-rescue:GND-power #PWR067
 U 1 1 61391300
 P 4050 5350
@@
 	4050 5350 4050 5250
 $Comp
-L Device:R R61
+L sesame-fonctionnel-rescue:R-Device R61
 U 1 1 61397C3C
 P 2900 4550
@@
 $EndComp
 $Comp
-L Device:R R62
+L sesame-fonctionnel-rescue:R-Device R62
 U 1 1 61398F33
 P 2900 4750
@@
 Current_Sens
 $Comp
-L Device:C C?
+L sesame-fonctionnel-rescue:C-Device C?
 U 1 1 613B4715
 P 1250 6950
@@
 	950  7300 950  7250
 $Comp
-L power:GND #PWR?
+L sesame-fonctionnel-rescue:GND-power #PWR?
 U 1 1 613B4720
 P 1100 7350
@@
 	1100 7300 1250 7300
 $Comp
-L power:VCC #PWR?
+L sesame-fonctionnel-rescue:VCC-power #PWR?
 U 1 1 613B472D
 P 1100 6550
@@
 OP Amp supply
 $Comp
-L Device:C C?
+L sesame-fonctionnel-rescue:C-Device C?
 U 1 1 613B7585
 P 2450 6900
@@
 	2150 7250 2150 7200
 $Comp
-L power:GND #PWR?
+L sesame-fonctionnel-rescue:GND-power #PWR?
 U 1 1 613B7590
 P 2300 7300
@@
 	2300 7250 2450 7250
 $Comp
-L power:VCC #PWR?
+L sesame-fonctionnel-rescue:VCC-power #PWR?
 U 1 1 613B759D
 P 2300 6500
@@
 	550  7700 2850 7700
 $Comp
-L Connector:TestPoint TP?
+L sesame-fonctionnel-rescue:TestPoint-Connector TP?
 U 1 1 6153C862
 P 4600 3950
@@
 $EndComp
 $Comp
-L Connector:TestPoint TP?
+L sesame-fonctionnel-rescue:TestPoint-Connector TP?
 U 1 1 61544B27
 P 9100 3250
@@
 	9100 3250 8700 3250
 $Comp
-L Connector:TestPoint TP?
+L sesame-fonctionnel-rescue:TestPoint-Connector TP?
 U 1 1 6154A16C
 P 5900 3850
