File: KICAD/Mos_Drivers.sch (KiCad schematic (older format))
At the start: 14 parts

Commit message: revex with jmt
Other:
- note added: "ucc27284-q1\n"
Changed lines of the file:
@@
 $Descr A4 11693 8268
 encoding utf-8
-Sheet 14 16
+Sheet 15 16
 Title "SESAME"
 Date ""
@@
 	1    0    0    -1
 $EndComp
+Text Notes 4150 1400 0    50   ~ 0
+ucc27284-q1\n
 $EndSCHEMATC

Commit message: minor cleanup
Parts:
- gave numbers to parts that had none: 1
Other:
- note added: "u9\n"
Changed lines of the file:
@@
 $Descr A4 11693 8268
 encoding utf-8
-Sheet 15 16
+Sheet 13 16
 Title "SESAME"
 Date ""
@@
 Candidats potentiels:\nMCP14628\nhttps://www.microchip.com/en-us/parametric-search.html/385\n-> UCC27284 (pas sourcable)\nBesoin: \nHalfBridge driver\nPWM & ~PWM~\nRapidité < 100ns\nAlim 7v\n(Pas cher)\nChez RS\nCourant de grille vers 2.5 - 3 A\nEnable\nMode DC !!
 $Comp
-L Driver_FET:UCC27714D U?
+L Driver_FET:UCC27714D U8
 U 1 1 612B940B
 P 4450 2550
-F 0 "U?" H 4100 3200 50  0000 C CNN
+F 0 "U8" H 4100 3200 50  0000 C CNN
 F 1 "UCC27714D" H 4100 3100 50  0000 C CNN
 F 2 "Package_SO:SOIC-14_3.9x8.7mm_P1.27mm" H 4450 2550 50  0001 C CNN
@@
 Text Notes 4150 1400 0    50   ~ 0
 ucc27284-q1\n
+Text Notes 4700 3850 0    50   ~ 0
+u9\n
 $EndSCHEMATC

Commit message: drivers draft + clean and minors changes
Parts:
- removed C?: 100n, symbol Device:C
- removed R?: 1k, symbol Device:R
- removed U8: UCC27714D, Package_SO:SOIC-14_3.9x8.7mm_P1.27mm, symbol Driver_FET:UCC27714D
- added C?: C, symbol Device:C
- added D? (x2): D_Schottky, symbol Device:D_Schottky
- added D? (x2): D, symbol Device:D
- added R? (x4): R, symbol Device:R
- added TP? (x6): TP_POP, symbol Connector:TestPoint
- added U? (x2): UCC27284-Q1, Package_SO:SOIC-8_3.9x4.9mm_P1.27mm, symbol Sesame:UCC27284-Q1
Connections:
- net labels removed: Enable, Enable_Softstart
- wire segments 39 -> 64
Other:
- note removed: "Candidats potentiels:\nMCP14628\nhttps://www.microchip.com/en-us/parametric-search.html/385\n-> UCC27284 (pas sourcable)\nBesoin: \nHalfBridge driver\nPWM & ~PWM~\nRapidité < 100ns\nAlim 7v\n(Pas cher)\nChez RS\nCourant de grille vers 2.5 - 3 A\nEnable\nMode DC !!"
- note removed: "Driver demi-Pont en H"
- note removed: "au plus vite (juste apres le triangle)\nenv 0.1ms"
- note removed: "choisir capacité + empreinte"
- note removed: "u9\n"
- note removed: "ucc27284-q1\n"
- moved on the sheet: C?, D?, R?

Commit message: driver + clean clean clean
Parts:
- removed C?: 100n, symbol Device:C
- removed C?: C, symbol Device:C
- removed D? (x3): D_Schottky, symbol Device:D_Schottky
- removed D? (x4): D, symbol Device:D
- removed R? (x8): R, symbol Device:R
- removed TP? (x3): TP_POP, symbol Connector:TestPoint
- removed U?: UCC27284-Q1, Package_SO:SOIC-8_3.9x4.9mm_P1.27mm, symbol Sesame:UCC27284-Q1
- added D? (x3): SS36, Diode_SMD:D_SMA_Handsoldering, symbol Device:D_Schottky
- added R? (x4): TBD, Resistor_SMD:R_0805_2012Metric_Pad1.15x1.40mm_HandSolder, symbol Device:R
- D?: value D_Schottky -> SS36; footprint (none) -> Diode_SMD:D_SMA_Handsoldering
- gave numbers to parts that had none: 1
Connections:
- net labels added: Driver_P, Driver_S, VG_P, VG_S, VS
- net labels removed: Driver_LP, Driver_LS, Driver_RP, Driver_RS, VG_LP, VG_LS, VG_RP, VG_RS, VS_L, VS_R
- wire segments 64 -> 32
Other:
- moved on the sheet: C?, D?, TP?, U9

Commit message: review w/ jmt
Parts:
- removed C?: C, symbol Device:C
- removed D?: SS36, Diode_SMD:D_SMA_Handsoldering, symbol Device:D_Schottky
- removed R? (x2): TBD, Resistor_SMD:R_0805_2012Metric_Pad1.15x1.40mm_HandSolder, symbol Device:R
- added C24: 100n, symbol Device:C
- added C25: 1u, symbol Device:CP
- added D11: SS36, Diode_SMD:D_SMA_Handsoldering, symbol Device:D_Schottky
- added R67: 1, symbol Device:R
- added R69: 5, symbol Device:R
- R66: renamed from R?; value TBD -> 1; footprint Resistor_SMD:R_0805_2012Metric_Pad1.15x1.40mm_HandSolder -> (none)
- R68: renamed from R?; value TBD -> 5; footprint Resistor_SMD:R_0805_2012Metric_Pad1.15x1.40mm_HandSolder -> (none)
- U12: renamed from U8; footprint Package_SO:SOIC-8_3.9x4.9mm_P1.27mm -> (none)
- gave numbers to parts that had none: 7
Connections:
- net VG_P: now also D11.2 (A), R69.2
- net VS: now also C24.2, C25.2
- net at U12.2 (HB): now also C24.1, C25.1
- net at D9.1 (K), U12.8 (LO): now also R67.2, R69.1
- new net: D11.1 (K), R67.1
Other:
- note added: "ajouter power pad\nVerifier que le driver peut tenir l’etat DC"
- moved on the sheet: D15, D16, D17, R85, R87, TP45, TP46, TP47, U17

Commit message: edit footprints by jmt
Parts:
- C23, C24, C25: footprint (none) -> Capacitor_SMD:C_0805_2012Metric_Pad1.15x1.40mm_HandSolder
- R66, R67, R68, R69: footprint (none) -> Resistor_SMD:R_0805_2012Metric_Pad1.15x1.40mm_HandSolder
- TP32, TP33, TP34: footprint (none) -> TestPoint:TestPoint_Loop_D1.80mm_Drill1.0mm_Beaded
- U12: footprint (none) -> Package_SO:SOIC-8_3.9x4.9mm_P1.27mm
Changed lines of the file:
@@
 F 0 "C33" H 965 7146 50  0000 L CNN
 F 1 "100n" H 965 7055 50  0000 L CNN
-F 2 "" H 888 6950 50  0001 C CNN
+F 2 "Capacitor_SMD:C_0805_2012Metric_Pad1.15x1.40mm_HandSolder" H 888 6950 50  0001 C CNN
 F 3 "~" H 850 7100 50  0001 C CNN
 	1    850  7100
@@
 F 0 "TP46" H 8250 3850 50  0000 L CNN
 F 1 "TP_POP" H 8300 3750 50  0000 C CNN
-F 2 "" H 8300 3650 50  0001 C CNN
+F 2 "TestPoint:TestPoint_Loop_D1.80mm_Drill1.0mm_Beaded" H 8300 3650 50  0001 C CNN
 F 3 "~" H 8300 3650 50  0001 C CNN
 	1    8100 3650
@@
 F 0 "TP47" H 8250 4150 50  0000 L CNN
 F 1 "TP_POP" H 8300 4050 50  0000 C CNN
-F 2 "" H 8300 3950 50  0001 C CNN
+F 2 "TestPoint:TestPoint_Loop_D1.80mm_Drill1.0mm_Beaded" H 8300 3950 50  0001 C CNN
 F 3 "~" H 8300 3950 50  0001 C CNN
 	1    8100 3950
@@
 F 0 "TP45" H 8250 3150 50  0000 L CNN
 F 1 "TP_POP" H 8300 3050 50  0000 C CNN
-F 2 "" H 8300 2950 50  0001 C CNN
+F 2 "TestPoint:TestPoint_Loop_D1.80mm_Drill1.0mm_Beaded" H 8300 2950 50  0001 C CNN
 F 3 "~" H 8300 2950 50  0001 C CNN
 	1    8100 2950
@@
 F 0 "U17" H 4000 4250 50  0000 C CNN
 F 1 "UCC27284-Q1" H 4000 4150 50  0000 C CNN
-F 2 "" H 4400 3450 50  0001 C CNN
+F 2 "Package_SO:SOIC-8_3.9x4.9mm_P1.27mm" H 4400 3450 50  0001 C CNN
 F 3 "" H 4400 3450 50  0001 C CNN
 	1    4400 3450
@@
 F 0 "R85" V 6943 2950 50  0000 C CNN
 F 1 "1" V 7034 2950 50  0000 C CNN
-F 2 "" V 7080 2950 50  0001 C CNN
+F 2 "Resistor_SMD:R_0805_2012Metric_Pad1.15x1.40mm_HandSolder" V 7080 2950 50  0001 C CNN
 F 3 "~" H 7150 2950 50  0001 C CNN
 	1    7150 2950
@@
 F 0 "R87" V 7093 3150 50  0000 C CNN
 F 1 "5" V 7184 3150 50  0000 C CNN
-F 2 "" V 7230 3150 50  0001 C CNN
+F 2 "Resistor_SMD:R_0805_2012Metric_Pad1.15x1.40mm_HandSolder" V 7230 3150 50  0001 C CNN
 F 3 "~" H 7300 3150 50  0001 C CNN
 	1    7300 3150
@@
 F 0 "C35" H 5818 3496 50  0000 L CNN
 F 1 "1u" H 5818 3405 50  0000 L CNN
-F 2 "" H 5738 3300 50  0001 C CNN
+F 2 "Capacitor_SMD:C_0805_2012Metric_Pad1.15x1.40mm_HandSolder" H 5738 3300 50  0001 C CNN
 F 3 "~" H 5700 3450 50  0001 C CNN
 	1    5700 3450
@@
 F 0 "R86" V 6943 3950 50  0000 C CNN
 F 1 "1" V 7034 3950 50  0000 C CNN
-F 2 "" V 7080 3950 50  0001 C CNN
+F 2 "Resistor_SMD:R_0805_2012Metric_Pad1.15x1.40mm_HandSolder" V 7080 3950 50  0001 C CNN
 F 3 "~" H 7150 3950 50  0001 C CNN
 	1    7150 3950
@@
 F 0 "R88" V 7093 4150 50  0000 C CNN
 F 1 "5" V 7184 4150 50  0000 C CNN
-F 2 "" V 7230 4150 50  0001 C CNN
+F 2 "Resistor_SMD:R_0805_2012Metric_Pad1.15x1.40mm_HandSolder" V 7230 4150 50  0001 C CNN
 F 3 "~" H 7300 4150 50  0001 C CNN
 	1    7300 4150
@@
 F 0 "C34" H 5315 3496 50  0000 L CNN
 F 1 "100n" H 5315 3405 50  0000 L CNN
-F 2 "" H 5238 3300 50  0001 C CNN
+F 2 "Capacitor_SMD:C_0805_2012Metric_Pad1.15x1.40mm_HandSolder" H 5238 3300 50  0001 C CNN
 F 3 "~" H 5200 3450 50  0001 C CNN
 	1    5200 3450

Commit message: route + work on djd
Changed lines of the file:
@@
 $Descr A4 11693 8268
 encoding utf-8
-Sheet 16 17
+Sheet 12 17
 Title "SESAME"
 Date ""
@@
 AR Path="/61996C9F/612BC387" Ref="C?"  Part="1"
 AR Path="/619A00BB/612BC387" Ref="C33"  Part="1"
-F 0 "C33" H 965 7146 50  0000 L CNN
+F 0 "C23" H 965 7146 50  0000 L CNN
 F 1 "100n" H 965 7055 50  0000 L CNN
 F 2 "Capacitor_SMD:C_0805_2012Metric_Pad1.15x1.40mm_HandSolder" H 888 6950 50  0001 C CNN
@@
 AR Path="/61996C9F/612C31FB" Ref="D?"  Part="1"
 AR Path="/619A00BB/612C31FB" Ref="D15"  Part="1"
-F 0 "D15" V 6004 3380 50  0000 L CNN
+F 0 "D8" V 6004 3380 50  0000 L CNN
 F 1 "SS36" V 6095 3380 50  0000 L CNN
 F 2 "Diode_SMD:D_SMA_Handsoldering" H 6050 3300 50  0001 C CNN
@@
 AR Path="/61996C9F/6154F3B3" Ref="TP?"  Part="1"
 AR Path="/619A00BB/6154F3B3" Ref="TP46"  Part="1"
-F 0 "TP46" H 8250 3850 50  0000 L CNN
+F 0 "TP33" H 8250 3850 50  0000 L CNN
 F 1 "TP_POP" H 8300 3750 50  0000 C CNN
 F 2 "TestPoint:TestPoint_Loop_D1.80mm_Drill1.0mm_Beaded" H 8300 3650 50  0001 C CNN
@@
 AR Path="/61996C9F/61556ADA" Ref="TP?"  Part="1"
 AR Path="/619A00BB/61556ADA" Ref="TP47"  Part="1"
-F 0 "TP47" H 8250 4150 50  0000 L CNN
+F 0 "TP34" H 8250 4150 50  0000 L CNN
 F 1 "TP_POP" H 8300 4050 50  0000 C CNN
 F 2 "TestPoint:TestPoint_Loop_D1.80mm_Drill1.0mm_Beaded" H 8300 3950 50  0001 C CNN
@@
 AR Path="/61996C9F/61556D55" Ref="TP?"  Part="1"
 AR Path="/619A00BB/61556D55" Ref="TP45"  Part="1"
-F 0 "TP45" H 8250 3150 50  0000 L CNN
+F 0 "TP32" H 8250 3150 50  0000 L CNN
 F 1 "TP_POP" H 8300 3050 50  0000 C CNN
 F 2 "TestPoint:TestPoint_Loop_D1.80mm_Drill1.0mm_Beaded" H 8300 2950 50  0001 C CNN
@@
 AR Path="/61996C9F/615F8500" Ref="U?"  Part="1"
 AR Path="/619A00BB/615F8500" Ref="U17"  Part="1"
-F 0 "U17" H 4000 4250 50  0000 C CNN
+F 0 "U12" H 4000 4250 50  0000 C CNN
 F 1 "UCC27284-Q1" H 4000 4150 50  0000 C CNN
 F 2 "Package_SO:SOIC-8_3.9x4.9mm_P1.27mm" H 4400 3450 50  0001 C CNN
@@
 AR Path="/61996C9F/617A570A" Ref="D?"  Part="1"
 AR Path="/619A00BB/617A570A" Ref="D16"  Part="1"
-F 0 "D16" V 6004 4280 50  0000 L CNN
+F 0 "D9" V 6004 4280 50  0000 L CNN
 F 1 "SS36" V 6095 4280 50  0000 L CNN
 F 2 "Diode_SMD:D_SMA_Handsoldering" H 6050 4200 50  0001 C CNN
@@
 AR Path="/61996C9F/617B4129" Ref="D?"  Part="1"
 AR Path="/619A00BB/617B4129" Ref="D17"  Part="1"
-F 0 "D17" H 7450 3167 50  0000 C CNN
+F 0 "D10" H 7450 3167 50  0000 C CNN
 F 1 "SS36" H 7450 3076 50  0000 C CNN
 F 2 "Diode_SMD:D_SMA_Handsoldering" H 7450 2950 50  0001 C CNN
@@
 AR Path="/61996C9F/617C4D4F" Ref="R?"  Part="1"
 AR Path="/619A00BB/617C4D4F" Ref="R85"  Part="1"
-F 0 "R85" V 6943 2950 50  0000 C CNN
+F 0 "R66" V 6943 2950 50  0000 C CNN
 F 1 "1" V 7034 2950 50  0000 C CNN
 F 2 "Resistor_SMD:R_0805_2012Metric_Pad1.15x1.40mm_HandSolder" V 7080 2950 50  0001 C CNN
@@
 AR Path="/61996C9F/617CA6D6" Ref="R?"  Part="1"
 AR Path="/619A00BB/617CA6D6" Ref="R87"  Part="1"
-F 0 "R87" V 7093 3150 50  0000 C CNN
+F 0 "R68" V 7093 3150 50  0000 C CNN
 F 1 "5" V 7184 3150 50  0000 C CNN
 F 2 "Resistor_SMD:R_0805_2012Metric_Pad1.15x1.40mm_HandSolder" V 7230 3150 50  0001 C CNN
@@
 AR Path="/60F19D6C/619F44C6" Ref="C25"  Part="1"
 AR Path="/619A00BB/619F44C6" Ref="C35"  Part="1"
-F 0 "C35" H 5818 3496 50  0000 L CNN
+F 0 "C25" H 5818 3496 50  0000 L CNN
 F 1 "1u" H 5818 3405 50  0000 L CNN
 F 2 "Capacitor_SMD:C_0805_2012Metric_Pad1.15x1.40mm_HandSolder" H 5738 3300 50  0001 C CNN
@@
 AR Path="/61996C9F/61A058A4" Ref="D?"  Part="1"
 AR Path="/619A00BB/61A058A4" Ref="D18"  Part="1"
-F 0 "D18" H 7450 4167 50  0000 C CNN
+F 0 "D11" H 7450 4167 50  0000 C CNN
 F 1 "SS36" H 7450 4076 50  0000 C CNN
 F 2 "Diode_SMD:D_SMA_Handsoldering" H 7450 3950 50  0001 C CNN
@@
 AR Path="/61996C9F/61A058AA" Ref="R?"  Part="1"
 AR Path="/619A00BB/61A058AA" Ref="R86"  Part="1"
-F 0 "R86" V 6943 3950 50  0000 C CNN
+F 0 "R67" V 6943 3950 50  0000 C CNN
 F 1 "1" V 7034 3950 50  0000 C CNN
 F 2 "Resistor_SMD:R_0805_2012Metric_Pad1.15x1.40mm_HandSolder" V 7080 3950 50  0001 C CNN
@@
 AR Path="/61996C9F/61A058B0" Ref="R?"  Part="1"
 AR Path="/619A00BB/61A058B0" Ref="R88"  Part="1"
-F 0 "R88" V 7093 4150 50  0000 C CNN
+F 0 "R69" V 7093 4150 50  0000 C CNN
 F 1 "5" V 7184 4150 50  0000 C CNN
 F 2 "Resistor_SMD:R_0805_2012Metric_Pad1.15x1.40mm_HandSolder" V 7230 4150 50  0001 C CNN
@@
 AR Path="/61996C9F/61A06D05" Ref="C?"  Part="1"
 AR Path="/619A00BB/61A06D05" Ref="C34"  Part="1"
-F 0 "C34" H 5315 3496 50  0000 L CNN
+F 0 "C24" H 5315 3496 50  0000 L CNN
 F 1 "100n" H 5315 3405 50  0000 L CNN
 F 2 "Capacitor_SMD:C_0805_2012Metric_Pad1.15x1.40mm_HandSolder" H 5238 3300 50  0001 C CNN
