File: KICAD/Mos_Drivers.sch (KiCad schematic (older format))
At the start: 24 parts, among them U12 UCC27284-Q1

Commit message: lil cleanup on the main schematic sheet
Parts:
- C23, C24, C52: symbol Device:C -> sesame-fonctionnel-rescue:C-Device
- C25, C50: symbol Device:CP -> sesame-fonctionnel-rescue:CP-Device
- D10, D11, D20, D21, D8, D9: symbol Device:D_Schottky -> sesame-fonctionnel-rescue:D_Schottky-Device
- D19: symbol Device:D_Zener -> sesame-fonctionnel-rescue:D_Zener-Device
- JP19: symbol Jumper:Jumper_2_Open -> sesame-fonctionnel-rescue:Jumper_2_Open-Jumper
- R66, R67, R68, R69, R97: symbol Device:R -> sesame-fonctionnel-rescue:R-Device
- TP32, TP33, TP34, TP43, TP48: symbol Connector:TestPoint -> sesame-fonctionnel-rescue:TestPoint-Connector
Changed lines of the file:
@@
 Driver_P
 $Comp
-L Device:C C23
+L sesame-fonctionnel-rescue:C-Device C23
 U 1 1 612BC387
 P 850 7100
@@
 $EndComp
 $Comp
-L power:GND #PWR082
+L sesame-fonctionnel-rescue:GND-power #PWR082
 U 1 1 612BD1C9
 P 1350 7250
@@
 $EndComp
 $Comp
-L power:GND #PWR084
+L sesame-fonctionnel-rescue:GND-power #PWR084
 U 1 1 612BD72C
 P 3400 5600
@@
 	5950 5400 5950 5500
 $Comp
-L power:GND #PWR085
+L sesame-fonctionnel-rescue:GND-power #PWR085
 U 1 1 612C2683
 P 5950 5800
@@
 $EndComp
 $Comp
-L Device:D_Schottky D8
+L sesame-fonctionnel-rescue:D_Schottky-Device D8
 U 1 1 612C31FB
 P 5950 4750
@@
 	600  6650 600  7650
 $Comp
-L power:VCC #PWR081
+L sesame-fonctionnel-rescue:VCC-power #PWR081
 U 1 1 6157FC90
 P 850 6950
@@
 $EndComp
 $Comp
-L Connector:TestPoint TP?
+L sesame-fonctionnel-rescue:TestPoint-Connector TP?
 U 1 1 6154F3B3
 P 8000 5100
@@
 	7550 5400 8000 5400
 $Comp
-L Connector:TestPoint TP?
+L sesame-fonctionnel-rescue:TestPoint-Connector TP?
 U 1 1 61556ADA
 P 8000 5400
@@
 $EndComp
 $Comp
-L power:VCC #PWR083
+L sesame-fonctionnel-rescue:VCC-power #PWR083
 U 1 1 615FA578
 P 3400 4200
@@
 $EndComp
 $Comp
-L Device:D_Schottky D9
+L sesame-fonctionnel-rescue:D_Schottky-Device D9
 U 1 1 617A570A
 P 5950 5650
@@
 $EndComp
 $Comp
-L Device:R R?
+L sesame-fonctionnel-rescue:R-Device R?
 U 1 1 617C4D4F
 P 7050 4400
@@
 	4200 5100 4700 5100
 $Comp
-L Device:CP C25
+L sesame-fonctionnel-rescue:CP-Device C25
 U 1 1 619F44C6
 P 4700 4900
@@
 	6850 5600 7050 5600
 $Comp
-L Device:D_Schottky D11
+L sesame-fonctionnel-rescue:D_Schottky-Device D11
 U 1 1 61A058A4
 P 7350 5400
@@
 $EndComp
 $Comp
-L Device:R R?
+L sesame-fonctionnel-rescue:R-Device R?
 U 1 1 61A058AA
 P 7050 5400
@@
 $EndComp
 $Comp
-L Device:R R?
+L sesame-fonctionnel-rescue:R-Device R?
 U 1 1 61A058B0
 P 7200 5600
@@
 $EndComp
 $Comp
-L Device:C C24
+L sesame-fonctionnel-rescue:C-Device C24
 U 1 1 61A06D05
 P 4200 4900
@@
 $EndComp
 $Comp
-L Device:CP C50
+L sesame-fonctionnel-rescue:CP-Device C50
 U 1 1 6128010B
 P 1350 7100
@@
 $EndComp
 $Comp
-L power:GND #PWR030
+L sesame-fonctionnel-rescue:GND-power #PWR030
 U 1 1 61281713
 P 850 7250
@@
 $EndComp
 $Comp
-L power:VCC #PWR0134
+L sesame-fonctionnel-rescue:VCC-power #PWR0134
 U 1 1 61281BBD
 P 1350 6950
@@
 Connection ~ 5950 5100
 $Comp
-L Device:R R?
+L sesame-fonctionnel-rescue:R-Device R?
 U 1 1 617CA6D6
 P 7200 4600
@@
 $EndComp
 $Comp
-L Device:D_Schottky D10
+L sesame-fonctionnel-rescue:D_Schottky-Device D10
 U 1 1 617B4129
 P 7350 4400
@@
 	7350 4600 7550 4600
 $Comp
-L Device:D_Schottky D21
+L sesame-fonctionnel-rescue:D_Schottky-Device D21
 U 1 1 6131353D
 P 8250 2550
@@
 	8850 2900 9150 2900
 $Comp
-L power:VCC #PWR0137
+L sesame-fonctionnel-rescue:VCC-power #PWR0137
 U 1 1 61318078
 P 8250 2300
@@
 	8250 2300 8250 2400
 $Comp
-L Device:D_Schottky D20
+L sesame-fonctionnel-rescue:D_Schottky-Device D20
 U 1 1 6131B437
 P 7350 2900
@@
 Connection ~ 8250 2900
 $Comp
-L Device:R R?
+L sesame-fonctionnel-rescue:R-Device R?
 U 1 1 6131E68D
 P 6950 2900
@@
 	7100 2900 7200 2900
 $Comp
-L Device:D_Zener D?
+L sesame-fonctionnel-rescue:D_Zener-Device D?
 U 1 1 6132C328
 P 5100 4900
@@
 Charge pump circuit
 $Comp
-L Device:C C52
+L sesame-fonctionnel-rescue:C-Device C52
 U 1 1 61341879
 P 8700 2900
@@
 Connection ~ 5100 2900
 $Comp
-L Connector:TestPoint TP?
+L sesame-fonctionnel-rescue:TestPoint-Connector TP?
 U 1 1 613ADBCD
 P 7600 2800
@@
 	7550 4400 8000 4400
 $Comp
-L Connector:TestPoint TP?
+L sesame-fonctionnel-rescue:TestPoint-Connector TP?
 U 1 1 61556D55
 P 8000 4350
@@
 $EndComp
 $Comp
-L Connector:TestPoint TP?
+L sesame-fonctionnel-rescue:TestPoint-Connector TP?
 U 1 1 613E88B5
 P 5100 2850
@@
 Connection ~ 5100 4700
 $Comp
-L Jumper:Jumper_2_Open JP19
+L sesame-fonctionnel-rescue:Jumper_2_Open-Jumper JP19
 U 1 1 615D1D25
 P 8250 3700

Commit message: V1.0 of the schematic
Parts:
- U12: footprint Package_SO:SOIC-8_3.9x4.9mm_P1.27mm -> Sesame_footprint:SOIC-8_3.9x4.9mm_P1.27mm
Changed lines of the file:
@@
 Sheet 10 17
 Title "SESAME"
-Date ""
-Rev ""
+Date "2021-09-23"
+Rev "1"
 Comp "ALEEA"
 Comment1 ""
@@
 F 0 "U12" H 3000 5700 50  0000 C CNN
 F 1 "UCC27284-Q1" H 3000 5600 50  0000 C CNN
-F 2 "Package_SO:SOIC-8_3.9x4.9mm_P1.27mm" H 3400 4900 50  0001 C CNN
+F 2 "Sesame_footprint:SOIC-8_3.9x4.9mm_P1.27mm" H 3400 4900 50  0001 C CNN
 F 3 "" H 3400 4900 50  0001 C CNN
 	1    3400 4900

Commit message: added gitignore and docs need cleenup
Changed lines of the file:
@@
 Comment4 ""
 $EndDescr
-Text HLabel 9200 5400 2    50   Output ~ 0
+Text HLabel 8650 5400 2    50   Output ~ 0
 VG_P
 Text HLabel 2600 4800 0    50   Input ~ 0
@@
 AR Path="/61996C9F/612BD1C9" Ref="#PWR?"  Part="1"
 AR Path="/619A00BB/612BD1C9" Ref="#PWR0118"  Part="1"
-F 0 "#PWR0118" H 1350 7000 50  0001 C CNN
+F 0 "#PWR082" H 1350 7000 50  0001 C CNN
 F 1 "GND" H 1355 7077 50  0000 C CNN
 F 2 "" H 1350 7250 50  0001 C CNN
@@
 AR Path="/61996C9F/612BD72C" Ref="#PWR?"  Part="1"
 AR Path="/619A00BB/612BD72C" Ref="#PWR0120"  Part="1"
-F 0 "#PWR0120" H 3400 5350 50  0001 C CNN
+F 0 "#PWR084" H 3400 5350 50  0001 C CNN
 F 1 "GND" H 3405 5427 50  0000 C CNN
 F 2 "" H 3400 5600 50  0001 C CNN
@@
 AR Path="/61996C9F/612C2683" Ref="#PWR?"  Part="1"
 AR Path="/619A00BB/612C2683" Ref="#PWR0121"  Part="1"
-F 0 "#PWR0121" H 5950 5550 50  0001 C CNN
+F 0 "#PWR085" H 5950 5550 50  0001 C CNN
 F 1 "GND" H 5955 5627 50  0000 C CNN
 F 2 "" H 5950 5800 50  0001 C CNN
@@
 $EndComp
 Connection ~ 5950 5400
-Text HLabel 9200 4400 2    50   Output ~ 0
+Text HLabel 8650 4400 2    50   Output ~ 0
 VG_S
 Wire Wire Line
@@
 AR Path="/61996C9F/6157FC90" Ref="#PWR?"  Part="1"
 AR Path="/619A00BB/6157FC90" Ref="#PWR0117"  Part="1"
-F 0 "#PWR0117" H 850 6800 50  0001 C CNN
+F 0 "#PWR081" H 850 6800 50  0001 C CNN
 F 1 "VCC" H 865 7123 50  0000 C CNN
 F 2 "" H 850 6950 50  0001 C CNN
@@
 Connection ~ 8000 5400
 Wire Wire Line
-	8000 5400 9200 5400
+	8000 5400 8650 5400
 Wire Wire Line
 	3850 5400 5950 5400
@@
 	5950 5100 5950 4900
 Wire Wire Line
-	8000 5100 9200 5100
+	8000 5100 8650 5100
 Connection ~ 7550 4400
 Wire Wire Line
@@
 AR Path="/61996C9F/615FA578" Ref="#PWR?"  Part="1"
 AR Path="/619A00BB/615FA578" Ref="#PWR0119"  Part="1"
-F 0 "#PWR0119" H 3400 4050 50  0001 C CNN
+F 0 "#PWR083" H 3400 4050 50  0001 C CNN
 F 1 "VCC" H 3415 4373 50  0000 C CNN
 F 2 "" H 3400 4200 50  0001 C CNN
@@
 AR Path="/61996C9F/61281713" Ref="#PWR?"  Part="1"
 AR Path="/619A00BB/61281713" Ref="#PWR0135"  Part="1"
-F 0 "#PWR0135" H 850 7000 50  0001 C CNN
+F 0 "#PWR030" H 850 7000 50  0001 C CNN
 F 1 "GND" H 855 7077 50  0000 C CNN
 F 2 "" H 850 7250 50  0001 C CNN
@@
 AR Path="/61996C9F/61281BBD" Ref="#PWR?"  Part="1"
 AR Path="/619A00BB/61281BBD" Ref="#PWR0136"  Part="1"
-F 0 "#PWR0136" H 1350 6800 50  0001 C CNN
+F 0 "#PWR0134" H 1350 6800 50  0001 C CNN
 F 1 "VCC" H 1365 7123 50  0000 C CNN
 F 2 "" H 1350 6950 50  0001 C CNN
@@
 	1    0    0    -1
 $EndComp
-Text HLabel 9200 5100 2    50   UnSpc ~ 0
+Text HLabel 8650 5100 2    50   UnSpc ~ 0
 VS
 Text HLabel 9150 2900 2    50   UnSpc ~ 0
@@
 AR Path="/60F19D6C/61318078" Ref="#PWR0137"  Part="1"
 AR Path="/619A00BB/61318078" Ref="#PWR0138"  Part="1"
-F 0 "#PWR0138" H 8250 2150 50  0001 C CNN
+F 0 "#PWR0137" H 8250 2150 50  0001 C CNN
 F 1 "VCC" H 8265 2473 50  0000 C CNN
 F 2 "" H 8250 2300 50  0001 C CNN
@@
 Connection ~ 8000 4400
 Wire Wire Line
-	8000 4400 9200 4400
+	8000 4400 8650 4400
 Wire Wire Line
 	7550 4400 8000 4400
@@
 Wire Wire Line
 	6450 2900 6800 2900
+$Comp
+L sesame-fonctionnel-rescue:Q_NMOS_GDS-Device QLS?
+U 1 1 619F66B1
+P 9700 4400
+AR Path="/60F18239/619F66B1" Ref="QLS?"  Part="1"
+AR Path="/60F19D6C/619F66B1" Ref="#Q?"  Part="1"
+AR Path="/619A00BB/619F66B1" Ref="#Q?"  Part="1"
+F 0 "#Q?" H 9905 4446 50  0000 L CNN
+F 1 "TK65G10N1" H 9905 4355 50  0000 L CNN
+F 2 "Package_TO_SOT_SMD:TO-263-2" H 9900 4500 50  0001 C CNN
+F 3 "https://docs.rs-online.com/a1f4/0900766b816230a5.pdf" H 9700 4400 50  0001 C CNN
+	1    9700 4400
+	1    0    0    -1
+$EndComp
+$Comp
+L sesame-fonctionnel-rescue:Q_NMOS_GDS-Device QLP?
+U 1 1 619F66BB
+P 9700 5450
+AR Path="/60F18239/619F66BB" Ref="QLP?"  Part="1"
+AR Path="/60F19D6C/619F66BB" Ref="#Q?"  Part="1"
+AR Path="/619A00BB/619F66BB" Ref="#Q?"  Part="1"
+F 0 "#Q?" H 9905 5496 50  0000 L CNN
+F 1 "TK65G10N1" H 9905 5405 50  0000 L CNN
+F 2 "Package_TO_SOT_SMD:TO-263-2" H 9900 5550 50  0001 C CNN
+F 3 "https://docs.rs-online.com/a1f4/0900766b816230a5.pdf" H 9700 5450 50  0001 C CNN
+	1    9700 5450
+	1    0    0    -1
+$EndComp
 $EndSCHEMATC
