File: KICAD/PROTECT.sch (KiCad schematic (older format))
At the start: 10 parts

Commit message: Stef merge
Parts:
- added TP? (x2): TP_POP, symbol Connector:TestPoint
- R? (x4): footprint Resistor_SMD:R_0805_2012Metric_Pad1.20x1.40mm_HandSolder -> Resistor_SMD:R_0805_2012Metric
Connections:
- wire segments 27 -> 29
Other:
- moved on the sheet: D?, Q?, R?
Changed lines of the file:
@@
 Comment4 ""
 $EndDescr
-Text HLabel 4150 2850 0    100  BiDi ~ 0
+Text HLabel 3750 2850 0    100  BiDi ~ 0
 IN_OUT_PWR
-Text HLabel 8300 2850 2    100  BiDi ~ 0
+Text HLabel 8600 2850 2    100  BiDi ~ 0
 VProt
 $Comp
 L Device:Q_PMOS_GDS Q?
 U 1 1 610FCCAA
-P 4650 2950
+P 4250 2950
 AR Path="/614794AE/610FCCAA" Ref="Q?"  Part="1"
 AR Path="/61456C6A/610FCCAA" Ref="Q?"  Part="1"
-F 0 "Q?" V 4992 2950 50  0000 C CNN
-F 1 "SQM120" V 4901 2950 50  0000 C CNN
-F 2 "Package_TO_SOT_SMD:TO-263-2" H 4850 3050 50  0001 C CNN
-F 3 "https://www.mouser.fr/datasheet/2/427/sqm120p10-10m1l-1766828.pdf" H 4650 2950 50  0001 C CNN
-	1    4650 2950
+F 0 "Q?" V 4592 2950 50  0000 C CNN
+F 1 "SQM120" V 4501 2950 50  0000 C CNN
+F 2 "Package_TO_SOT_SMD:TO-263-2" H 4450 3050 50  0001 C CNN
+F 3 "https://www.mouser.fr/datasheet/2/427/sqm120p10-10m1l-1766828.pdf" H 4250 2950 50  0001 C CNN
+	1    4250 2950
 	0    -1   -1   0
 $EndComp
@@
 L Device:D_Zener D?
 U 1 1 61100A0F
-P 4950 3100
+P 4550 3100
 AR Path="/614794AE/61100A0F" Ref="D?"  Part="1"
 AR Path="/61456C6A/61100A0F" Ref="D?"  Part="1"
-F 0 "D?" V 4904 3180 50  0000 L CNN
-F 1 "MMSZ5245" V 4995 3180 50  0000 L CNN
-F 2 "Diode_SMD:D_SOD-123" H 4950 3100 50  0001 C CNN
-F 3 "https://docs.rs-online.com/0640/0900766b814f560f.pdf" H 4950 3100 50  0001 C CNN
-	1    4950 3100
+F 0 "D?" V 4504 3180 50  0000 L CNN
+F 1 "MMSZ5245" V 4595 3180 50  0000 L CNN
+F 2 "Diode_SMD:D_SOD-123" H 4550 3100 50  0001 C CNN
+F 3 "https://docs.rs-online.com/0640/0900766b814f560f.pdf" H 4550 3100 50  0001 C CNN
+	1    4550 3100
 	0    1    1    0
 $EndComp
@@
 L Device:R R?
 U 1 1 61102FC8
-P 4650 3700
+P 4250 3700
 AR Path="/614794AE/61102FC8" Ref="R?"  Part="1"
 AR Path="/61456C6A/61102FC8" Ref="R?"  Part="1"
-F 0 "R?" H 4720 3746 50  0000 L CNN
-F 1 "330k" H 4720 3655 50  0000 L CNN
-F 2 "Resistor_SMD:R_0805_2012Metric_Pad1.20x1.40mm_HandSolder" V 4580 3700 50  0001 C CNN
-F 3 "~" H 4650 3700 50  0001 C CNN
-	1    4650 3700
-	1    0    0    -1
-$EndComp
-Wire Wire Line
-	4950 3250 4950 3350
-Wire Wire Line
-	4950 3350 4650 3350
-Wire Wire Line
-	4650 3350 4650 3150
-Wire Wire Line
-	4650 3550 4650 3350
-Connection ~ 4650 3350
+F 0 "R?" H 4320 3746 50  0000 L CNN
+F 1 "330k" H 4320 3655 50  0000 L CNN
+F 2 "Resistor_SMD:R_0805_2012Metric" V 4180 3700 50  0001 C CNN
+F 3 "~" H 4250 3700 50  0001 C CNN
+	1    4250 3700
+	1    0    0    -1
+$EndComp
+Wire Wire Line
+	4550 3250 4550 3350
+Wire Wire Line
+	4550 3350 4250 3350
+Wire Wire Line
+	4250 3350 4250 3150
+Wire Wire Line
+	4250 3550 4250 3350
+Connection ~ 4250 3350
 $Comp
 L power:GNDPWR #PWR0121
 U 1 1 61104B6E
-P 4650 4050
+P 4250 4050
 AR Path="/614794AE/61104B6E" Ref="#PWR0121"  Part="1"
 AR Path="/61456C6A/61104B6E" Ref="#PWR0124"  Part="1"
-F 0 "#PWR0124" H 4650 3850 50  0001 C CNN
-F 1 "GNDPWR" H 4654 3896 50  0000 C CNN
-F 2 "" H 4650 4000 50  0001 C CNN
-F 3 "" H 4650 4000 50  0001 C CNN
-	1    4650 4050
-	1    0    0    -1
-$EndComp
-Wire Wire Line
-	4650 4050 4650 3850
-Wire Wire Line
-	4150 2850 4450 2850
-Wire Notes Line
-	4300 2500 5500 2500
+F 0 "#PWR0121" H 4250 3850 50  0001 C CNN
+F 1 "GNDPWR" H 4254 3896 50  0000 C CNN
+F 2 "" H 4250 4000 50  0001 C CNN
+F 3 "" H 4250 4000 50  0001 C CNN
+	1    4250 4050
+	1    0    0    -1
+$EndComp
+Wire Wire Line
+	4250 4050 4250 3850
+Wire Wire Line
+	3750 2850 4050 2850
+Wire Notes Line
+	3900 2500 5100 2500
 $Comp
 L Transistor_BJT:BC857 Q?
@@
 F 0 "R?" H 5970 3146 50  0000 L CNN
 F 1 "100k" H 5970 3055 50  0000 L CNN
-F 2 "Resistor_SMD:R_0805_2012Metric_Pad1.20x1.40mm_HandSolder" V 5830 3100 50  0001 C CNN
+F 2 "Resistor_SMD:R_0805_2012Metric" V 5830 3100 50  0001 C CNN
 F 3 "~" H 5900 3100 50  0001 C CNN
 	1    5900 3100
@@
 F 0 "R?" V 6043 3300 50  0000 C CNN
 F 1 "100k" V 6134 3300 50  0000 C CNN
-F 2 "Resistor_SMD:R_0805_2012Metric_Pad1.20x1.40mm_HandSolder" V 6180 3300 50  0001 C CNN
+F 2 "Resistor_SMD:R_0805_2012Metric" V 6180 3300 50  0001 C CNN
 F 3 "~" H 6250 3300 50  0001 C CNN
 	1    6250 3300
@@
 F 0 "R?" H 7870 3896 50  0000 L CNN
 F 1 "1M" H 7870 3805 50  0000 L CNN
-F 2 "Resistor_SMD:R_0805_2012Metric_Pad1.20x1.40mm_HandSolder" V 7730 3850 50  0001 C CNN
+F 2 "Resistor_SMD:R_0805_2012Metric" V 7730 3850 50  0001 C CNN
 F 3 "~" H 7800 3850 50  0001 C CNN
 	1    7800 3850
@@
 AR Path="/614794AE/6111576B" Ref="#PWR0122"  Part="1"
 AR Path="/61456C6A/6111576B" Ref="#PWR0125"  Part="1"
-F 0 "#PWR0125" H 7800 3850 50  0001 C CNN
+F 0 "#PWR0122" H 7800 3850 50  0001 C CNN
 F 1 "GNDPWR" H 7804 3896 50  0000 C CNN
 F 2 "" H 7800 4000 50  0001 C CNN
@@
 Text Notes 5650 4400 0    50   ~ 0
 Protection sur-tensions
-Text Notes 4350 4400 0    50   ~ 0
+Text Notes 3950 4400 0    50   ~ 0
 Protection Inversion polarité
 Wire Notes Line
-	5500 4450 4300 4450
-Wire Notes Line
-	5500 2500 5500 4450
-Wire Notes Line
-	4300 2500 4300 4450
-Wire Wire Line
-	8300 2850 8000 2850
-Wire Wire Line
-	4850 2850 4950 2850
-Wire Wire Line
-	4950 2950 4950 2850
-Connection ~ 4950 2850
-Wire Wire Line
-	4950 2850 5900 2850
+	5100 4450 3900 4450
+Wire Notes Line
+	5100 2500 5100 4450
+Wire Notes Line
+	3900 2500 3900 4450
+Wire Wire Line
+	8600 2850 8400 2850
+Wire Wire Line
+	4450 2850 4550 2850
+Wire Wire Line
+	4550 2950 4550 2850
+Connection ~ 4550 2850
+Wire Wire Line
+	4550 2850 5350 2850
 Connection ~ 5900 3300
 Wire Wire Line
@@
 AR Path="/614794AE/611168C4" Ref="#PWR0123"  Part="1"
 AR Path="/61456C6A/611168C4" Ref="#PWR0126"  Part="1"
-F 0 "#PWR0126" H 5900 3850 50  0001 C CNN
+F 0 "#PWR0123" H 5900 3850 50  0001 C CNN
 F 1 "GNDPWR" H 5904 3896 50  0000 C CNN
 F 2 "" H 5900 4000 50  0001 C CNN
@@
 	0    1    1    0
 $EndComp
+$Comp
+L Connector:TestPoint TP?
+U 1 1 612D3587
+P 5350 2850
+AR Path="/614794AE/612D3587" Ref="TP?"  Part="1"
+AR Path="/61456C6A/612D3587" Ref="TP?"  Part="1"
+F 0 "TP?" H 5300 3100 50  0000 L CNN
+F 1 "TP_POP" H 5350 2750 50  0000 C CNN
+F 2 "" H 5550 2850 50  0001 C CNN
+F 3 "~" H 5550 2850 50  0001 C CNN
+	1    5350 2850
+	1    0    0    -1
+$EndComp
+Connection ~ 5350 2850
+Wire Wire Line
+	5350 2850 5900 2850
+$Comp
+L Connector:TestPoint TP?
+U 1 1 612DA888
+P 8400 2850
+AR Path="/614794AE/612DA888" Ref="TP?"  Part="1"
+AR Path="/61456C6A/612DA888" Ref="TP?"  Part="1"
+F 0 "TP?" H 8350 3100 50  0000 L CNN
+F 1 "TP_POP" H 8400 2750 50  0000 C CNN
+F 2 "" H 8600 2850 50  0001 C CNN
+F 3 "~" H 8600 2850 50  0001 C CNN
+	1    8400 2850
+	1    0    0    -1
+$EndComp
+Connection ~ 8400 2850
+Wire Wire Line
+	8000 2850 8400 2850
 $EndSCHEMATC

Commit message: drivers draft + clean and minors changes
Parts:
- added TP?: TP_POP, symbol Connector:TestPoint
- R? (x3): footprint Resistor_SMD:R_0805_2012Metric -> Resistor_SMD:R_0805_2012Metric_Pad1.15x1.40mm_HandSolder
Connections:
- wire segments 29 -> 30
Changed lines of the file:
@@
 $Descr A4 11693 8268
 encoding utf-8
-Sheet 10 16
+Sheet 9 16
 Title ""
 Date ""
@@
 Comment4 ""
 $EndDescr
-Text HLabel 3750 2850 0    100  BiDi ~ 0
+Text HLabel 3350 2850 0    100  BiDi ~ 0
 IN_OUT_PWR
 Text HLabel 8600 2850 2    100  BiDi ~ 0
@@
 AR Path="/614794AE/61104B6E" Ref="#PWR0121"  Part="1"
 AR Path="/61456C6A/61104B6E" Ref="#PWR0124"  Part="1"
-F 0 "#PWR0121" H 4250 3850 50  0001 C CNN
+F 0 "#PWR0124" H 4250 3850 50  0001 C CNN
 F 1 "GNDPWR" H 4254 3896 50  0000 C CNN
 F 2 "" H 4250 4000 50  0001 C CNN
@@
 Wire Wire Line
 	4250 4050 4250 3850
-Wire Wire Line
-	3750 2850 4050 2850
 Wire Notes Line
 	3900 2500 5100 2500
@@
 F 0 "R?" H 5970 3146 50  0000 L CNN
 F 1 "100k" H 5970 3055 50  0000 L CNN
-F 2 "Resistor_SMD:R_0805_2012Metric" V 5830 3100 50  0001 C CNN
+F 2 "Resistor_SMD:R_0805_2012Metric_Pad1.15x1.40mm_HandSolder" V 5830 3100 50  0001 C CNN
 F 3 "~" H 5900 3100 50  0001 C CNN
 	1    5900 3100
@@
 F 0 "R?" V 6043 3300 50  0000 C CNN
 F 1 "100k" V 6134 3300 50  0000 C CNN
-F 2 "Resistor_SMD:R_0805_2012Metric" V 6180 3300 50  0001 C CNN
+F 2 "Resistor_SMD:R_0805_2012Metric_Pad1.15x1.40mm_HandSolder" V 6180 3300 50  0001 C CNN
 F 3 "~" H 6250 3300 50  0001 C CNN
 	1    6250 3300
@@
 F 0 "R?" H 7870 3896 50  0000 L CNN
 F 1 "1M" H 7870 3805 50  0000 L CNN
-F 2 "Resistor_SMD:R_0805_2012Metric" V 7730 3850 50  0001 C CNN
+F 2 "Resistor_SMD:R_0805_2012Metric_Pad1.15x1.40mm_HandSolder" V 7730 3850 50  0001 C CNN
 F 3 "~" H 7800 3850 50  0001 C CNN
 	1    7800 3850
@@
 AR Path="/614794AE/6111576B" Ref="#PWR0122"  Part="1"
 AR Path="/61456C6A/6111576B" Ref="#PWR0125"  Part="1"
-F 0 "#PWR0122" H 7800 3850 50  0001 C CNN
+F 0 "#PWR0125" H 7800 3850 50  0001 C CNN
 F 1 "GNDPWR" H 7804 3896 50  0000 C CNN
 F 2 "" H 7800 4000 50  0001 C CNN
@@
 AR Path="/614794AE/611168C4" Ref="#PWR0123"  Part="1"
 AR Path="/61456C6A/611168C4" Ref="#PWR0126"  Part="1"
-F 0 "#PWR0123" H 5900 3850 50  0001 C CNN
+F 0 "#PWR0126" H 5900 3850 50  0001 C CNN
 F 1 "GNDPWR" H 5904 3896 50  0000 C CNN
 F 2 "" H 5900 4000 50  0001 C CNN
@@
 Wire Wire Line
 	8000 2850 8400 2850
+$Comp
+L Connector:TestPoint TP?
+U 1 1 614EA2DB
+P 3650 2850
+AR Path="/614794AE/614EA2DB" Ref="TP?"  Part="1"
+AR Path="/61456C6A/614EA2DB" Ref="TP?"  Part="1"
+F 0 "TP?" H 3600 3100 50  0000 L CNN
+F 1 "TP_POP" H 3650 2750 50  0000 C CNN
+F 2 "" H 3850 2850 50  0001 C CNN
+F 3 "~" H 3850 2850 50  0001 C CNN
+	1    3650 2850
+	1    0    0    -1
+$EndComp
+Wire Wire Line
+	3350 2850 3650 2850
+Connection ~ 3650 2850
+Wire Wire Line
+	3650 2850 4050 2850
 $EndSCHEMATC

Commit message: driver + clean clean clean
Connections:
- net labels added: IO_PWR
- net labels removed: IN_OUT_PWR
Changed lines of the file:
@@
 $Descr A4 11693 8268
 encoding utf-8
-Sheet 9 16
+Sheet 10 17
 Title ""
 Date ""
@@
 $EndDescr
 Text HLabel 3350 2850 0    100  BiDi ~ 0
-IN_OUT_PWR
+IO_PWR
 Text HLabel 8600 2850 2    100  BiDi ~ 0
 VProt
@@
 AR Path="/614794AE/610FCCAA" Ref="Q?"  Part="1"
 AR Path="/61456C6A/610FCCAA" Ref="Q?"  Part="1"
+AR Path="/618D2416/610FCCAA" Ref="Q?"  Part="1"
 F 0 "Q?" V 4592 2950 50  0000 C CNN
 F 1 "SQM120" V 4501 2950 50  0000 C CNN
@@
 AR Path="/614794AE/610FED91" Ref="Q?"  Part="1"
 AR Path="/61456C6A/610FED91" Ref="Q?"  Part="1"
+AR Path="/618D2416/610FED91" Ref="Q?"  Part="1"
 F 0 "Q?" V 8142 2950 50  0000 C CNN
 F 1 "SQM120" V 8051 2950 50  0000 C CNN
@@
 AR Path="/614794AE/61100A0F" Ref="D?"  Part="1"
 AR Path="/61456C6A/61100A0F" Ref="D?"  Part="1"
+AR Path="/618D2416/61100A0F" Ref="D?"  Part="1"
 F 0 "D?" V 4504 3180 50  0000 L CNN
 F 1 "MMSZ5245" V 4595 3180 50  0000 L CNN
@@
 AR Path="/614794AE/61102FC8" Ref="R?"  Part="1"
 AR Path="/61456C6A/61102FC8" Ref="R?"  Part="1"
+AR Path="/618D2416/61102FC8" Ref="R?"  Part="1"
 F 0 "R?" H 4320 3746 50  0000 L CNN
 F 1 "330k" H 4320 3655 50  0000 L CNN
@@
 AR Path="/614794AE/61104B6E" Ref="#PWR0121"  Part="1"
 AR Path="/61456C6A/61104B6E" Ref="#PWR0124"  Part="1"
-F 0 "#PWR0124" H 4250 3850 50  0001 C CNN
+AR Path="/618D2416/61104B6E" Ref="#PWR?"  Part="1"
+F 0 "#PWR?" H 4250 3850 50  0001 C CNN
 F 1 "GNDPWR" H 4254 3896 50  0000 C CNN
 F 2 "" H 4250 4000 50  0001 C CNN
@@
 AR Path="/614794AE/6110710F" Ref="Q?"  Part="1"
 AR Path="/61456C6A/6110710F" Ref="Q?"  Part="1"
+AR Path="/618D2416/6110710F" Ref="Q?"  Part="1"
 F 0 "Q?" H 6791 3346 50  0000 L CNN
 F 1 "BC857" H 6791 3255 50  0000 L CNN
@@
 AR Path="/614794AE/61107DEE" Ref="D?"  Part="1"
 AR Path="/61456C6A/61107DEE" Ref="D?"  Part="1"
+AR Path="/618D2416/61107DEE" Ref="D?"  Part="1"
 F 0 "D?" V 7204 3280 50  0000 L CNN
 F 1 "MMSZ5245" V 7295 3280 50  0000 L CNN
@@
 AR Path="/614794AE/611083FB" Ref="R?"  Part="1"
 AR Path="/61456C6A/611083FB" Ref="R?"  Part="1"
+AR Path="/618D2416/611083FB" Ref="R?"  Part="1"
 F 0 "R?" H 5970 3146 50  0000 L CNN
 F 1 "100k" H 5970 3055 50  0000 L CNN
@@
 AR Path="/614794AE/6110B925" Ref="R?"  Part="1"
 AR Path="/61456C6A/6110B925" Ref="R?"  Part="1"
+AR Path="/618D2416/6110B925" Ref="R?"  Part="1"
 F 0 "R?" V 6043 3300 50  0000 C CNN
 F 1 "100k" V 6134 3300 50  0000 C CNN
@@
 AR Path="/614794AE/61115761" Ref="R?"  Part="1"
 AR Path="/61456C6A/61115761" Ref="R?"  Part="1"
+AR Path="/618D2416/61115761" Ref="R?"  Part="1"
 F 0 "R?" H 7870 3896 50  0000 L CNN
 F 1 "1M" H 7870 3805 50  0000 L CNN
@@
 AR Path="/614794AE/6111576B" Ref="#PWR0122"  Part="1"
 AR Path="/61456C6A/6111576B" Ref="#PWR0125"  Part="1"
-F 0 "#PWR0125" H 7800 3850 50  0001 C CNN
+AR Path="/618D2416/6111576B" Ref="#PWR?"  Part="1"
+F 0 "#PWR?" H 7800 3850 50  0001 C CNN
 F 1 "GNDPWR" H 7804 3896 50  0000 C CNN
 F 2 "" H 7800 4000 50  0001 C CNN
@@
 AR Path="/614794AE/611168C4" Ref="#PWR0123"  Part="1"
 AR Path="/61456C6A/611168C4" Ref="#PWR0126"  Part="1"
-F 0 "#PWR0126" H 5900 3850 50  0001 C CNN
+AR Path="/618D2416/611168C4" Ref="#PWR?"  Part="1"
+F 0 "#PWR?" H 5900 3850 50  0001 C CNN
 F 1 "GNDPWR" H 5904 3896 50  0000 C CNN
 F 2 "" H 5900 4000 50  0001 C CNN
@@
 AR Path="/614794AE/61107C25" Ref="D?"  Part="1"
 AR Path="/61456C6A/61107C25" Ref="D?"  Part="1"
+AR Path="/618D2416/61107C25" Ref="D?"  Part="1"
 F 0 "D?" V 5854 3780 50  0000 L CNN
 F 1 "MMSZ5262" V 5945 3780 50  0000 L CNN
@@
 AR Path="/614794AE/612D3587" Ref="TP?"  Part="1"
 AR Path="/61456C6A/612D3587" Ref="TP?"  Part="1"
+AR Path="/618D2416/612D3587" Ref="TP?"  Part="1"
 F 0 "TP?" H 5300 3100 50  0000 L CNN
 F 1 "TP_POP" H 5350 2750 50  0000 C CNN
@@
 AR Path="/614794AE/612DA888" Ref="TP?"  Part="1"
 AR Path="/61456C6A/612DA888" Ref="TP?"  Part="1"
+AR Path="/618D2416/612DA888" Ref="TP?"  Part="1"
 F 0 "TP?" H 8350 3100 50  0000 L CNN
 F 1 "TP_POP" H 8400 2750 50  0000 C CNN
@@
 AR Path="/614794AE/614EA2DB" Ref="TP?"  Part="1"
 AR Path="/61456C6A/614EA2DB" Ref="TP?"  Part="1"
+AR Path="/618D2416/614EA2DB" Ref="TP?"  Part="1"
 F 0 "TP?" H 3600 3100 50  0000 L CNN
 F 1 "TP_POP" H 3650 2750 50  0000 C CNN
