File: KICAD/Int_Ext_Config.sch (KiCad schematic (older format))
At the start: 9 parts, among them J9 Conn_02x16_Odd_Even

Commit message: lil cleanup on the main schematic sheet
Parts:
- J9: symbol Connector_Generic:Conn_02x16_Odd_Even -> sesame-fonctionnel-rescue:Conn_02x16_Odd_Even-Connector_Generic
- JP10, JP11, JP12, JP13, JP14: symbol Device:Jumper_NC_Dual -> sesame-fonctionnel-rescue:Jumper_NC_Dual-Device
- R76, R77, R78: symbol Device:R -> sesame-fonctionnel-rescue:R-Device
Changed lines of the file:
@@
 Voltage_Sens_R
 $Comp
-L power:VCC #PWR092
+L sesame-fonctionnel-rescue:VCC-power #PWR092
 U 1 1 6133D413
 P 2050 3850
@@
 CC_CV_Mode
 $Comp
-L power:GND #PWR091
+L sesame-fonctionnel-rescue:GND-power #PWR091
 U 1 1 6134A761
 P 1150 5600
@@
 Ext_Rearm
 $Comp
-L power:GND #PWR096
+L sesame-fonctionnel-rescue:GND-power #PWR096
 U 1 1 61386A80
 P 2900 3200
@@
 $EndComp
 $Comp
-L Device:Jumper_NC_Dual JP13
+L sesame-fonctionnel-rescue:Jumper_NC_Dual-Device JP13
 U 1 1 61386A86
 P 3350 3100
@@
 $EndComp
 $Comp
-L power:VCC #PWR097
+L sesame-fonctionnel-rescue:VCC-power #PWR097
 U 1 1 61386A8C
 P 3800 3050
@@
 	2900 3100 3100 3100
 $Comp
-L Device:R R77
+L sesame-fonctionnel-rescue:R-Device R77
 U 1 1 61386A97
 P 3350 3450
@@
 	3350 3700 3350 3600
 $Comp
-L power:GND #PWR098
+L sesame-fonctionnel-rescue:GND-power #PWR098
 U 1 1 6138E72F
 P 4100 3200
@@
 $EndComp
 $Comp
-L Device:Jumper_NC_Dual JP14
+L sesame-fonctionnel-rescue:Jumper_NC_Dual-Device JP14
 U 1 1 6138E735
 P 4550 3100
@@
 $EndComp
 $Comp
-L power:VCC #PWR099
+L sesame-fonctionnel-rescue:VCC-power #PWR099
 U 1 1 6138E73B
 P 5000 3050
@@
 	4100 3100 4300 3100
 $Comp
-L Device:R R78
+L sesame-fonctionnel-rescue:R-Device R78
 U 1 1 6138E745
 P 4550 3450
@@
 Connection ~ 4550 3700
 $Comp
-L Device:Jumper_NC_Dual JP11
+L sesame-fonctionnel-rescue:Jumper_NC_Dual-Device JP11
 U 1 1 6139D414
 P 9200 3100
@@
 ~INT_PWM_Freewheel
 $Comp
-L Device:Jumper_NC_Dual JP10
+L sesame-fonctionnel-rescue:Jumper_NC_Dual-Device JP10
 U 1 1 613A5DB8
 P 7300 3100
@@
 	10000 3100 10000 5500
 $Comp
-L Connector_Generic:Conn_02x16_Odd_Even J9
+L sesame-fonctionnel-rescue:Conn_02x16_Odd_Even-Connector_Generic J9
 U 1 1 61332892
 P 1450 4700
@@
 	5250 3200 5250 3100
 $Comp
-L power:GND #PWR0116
+L sesame-fonctionnel-rescue:GND-power #PWR0116
 U 1 1 6143326D
 P 5250 3200
@@
 	5700 3300 5700 3200
 $Comp
-L Device:R R76
+L sesame-fonctionnel-rescue:R-Device R76
 U 1 1 6137F2F0
 P 5700 3450
@@
 	6150 3050 6150 3100
 $Comp
-L power:VCC #PWR095
+L sesame-fonctionnel-rescue:VCC-power #PWR095
 U 1 1 6136D0ED
 P 6150 3050
@@
 $EndComp
 $Comp
-L Device:Jumper_NC_Dual JP12
+L sesame-fonctionnel-rescue:Jumper_NC_Dual-Device JP12
 U 1 1 61366A29
 P 5700 3100
