File: KICAD/PID.sch (KiCad schematic (older format))
At the start: 23 parts, among them U1 AD8030

Commit message: V1.0 of the schematic
Parts:
- U1: footprint Package_SO:SO-8_5.3x6.2mm_P1.27mm -> Sesame_footprint:SO-8_5.3x6.2mm_P1.27mm
Changed lines of the file:
@@
 Sheet 15 17
 Title "SESAME"
-Date ""
-Rev ""
+Date "2021-09-23"
+Rev "1"
 Comp "ALEEA"
 Comment1 "Dessin : Kevin & Sarah & Guillaume Arthaud"
@@
 F 0 "U1" H 1063 6804 50  0000 R CNN
 F 1 "AD8030" H 1063 6895 50  0000 R CNN
-F 2 "Package_SO:SO-8_5.3x6.2mm_P1.27mm" H 1250 6850 50  0001 C CNN
+F 2 "Sesame_footprint:SO-8_5.3x6.2mm_P1.27mm" H 1250 6850 50  0001 C CNN
 F 3 "~" H 1250 6850 50  0001 C CNN
 	3    1250 6850
@@
 F 0 "U1" H 7250 2833 50  0000 C CNN
 F 1 "AD8030" H 7250 2924 50  0000 C CNN
-F 2 "Package_SO:SO-8_5.3x6.2mm_P1.27mm" H 7250 3200 50  0001 C CNN
+F 2 "Sesame_footprint:SO-8_5.3x6.2mm_P1.27mm" H 7250 3200 50  0001 C CNN
 F 3 "~" H 7250 3200 50  0001 C CNN
 	1    7250 3200
