File: KICAD/dual_LT6105/dual_LT6105.kicad_sch (KiCad schematic)
At the start: 12 parts, among them J1 Conn_01x01, J2 Conn_01x01, J3 Conn_01x01, J4 Conn_01x01, J5 Conn_01x01, J6 Conn_01x01, J7 Conn_01x01, J8 Conn_01x01, U1 LT6105, U2 LT6105

Commit message: added gitignore and docs need cleenup
Other:
- moved on the sheet: J3, J4, J5, J6, J7, J8, R1, U1, U2

Commit message: added datasheets + test bench first version
Other:
- company: (none) -> ALEEA
- title: (none) -> Dual LT6105
- moved on the sheet: J3, J4, J5, J6, J7, J8, R1, U1, U2
